File: module-tester-board.sch (KiCad schematic (older format))
At the start: 20 parts, among them J1 Conn_01x08_Male, J4 Conn_01x04_Male, SW1 SW_SPST, U1 LT8330, U4 MCP2515-EST, U5 ATA6560,1

Commit message: Version 0.0.2
Schematic to be Reviewed
Parts:
- added C? (x2): 15p, Capacitor_SMD:C_0603_1608Metric, symbol Device:C_Small
- added C?: 100uF, symbol Device:C
- added D?: 1N4007, symbol Device:D
- added R1: 1k, Resistor_SMD:R_0603_1608Metric, symbol Device:R
- added R?: 1k, symbol Device:R
- added R?: 100k, symbol Device:R
- added Y?: 20MHz, symbol Device:Crystal
Connections:
- net labels added: +5V, INT, RX0, RX1, Reset, TX0, TX1, TX2
- wire segments 88 -> 116
- no-connect marks 0 -> 14
Other:
- note added: "!R1 may or may not need to be populated!"
- note added: "48V Voltage Regulator"
- note added: "CAN"
- note added: "Nano"
- note added: "Pin Out and Switches"
- note added: "Reset for CAN"

Commit message: Version 0.0.3
Fixed red lines
Parts:
- R1: value 1k -> 1M
Connections:
- net labels removed: 5V, FBX
- wire segments 116 -> 117
- no-connect marks 14 -> 13
Other:
- note added: "48V Regulator"
- note added: "Arduino Nano"
- note added: "CAN Communication using MCP2515 and ATA6560"
- note added: "R5485 Header and Selection Switches"
- note added: "Reset for MCP2515"
- note removed: "48V Voltage Regulator"
- note removed: "CAN"
- note removed: "Nano"
- note removed: "Pin Out and Switches"
- note removed: "Reset for CAN"

Commit message: 0.0.3 cleanup and change power symbols
Parts:
- U5: symbol URT_cache:ATA6560,1 -> ATA6560_1:ATA6560,1
Connections:
- net labels added: +48V
- net labels removed: 48V
- wire segments 117 -> 115
Other:
- note added: "Main uC\n"
Changed lines of the file:
@@
 Sheet 1 1
 Title "module-tester-board"
-Date "2018-09-16"
-Rev "0.0.3"
+Date "2018-09-17"
+Rev "0.0.4"
 Comp "Missouri University of Science and Technology - Underwater Robotics Team"
 Comment1 "Board for testing ROV modules away from ROV."
@@
 $EndComp
 $Comp
-L URT_cache:ATA6560,1 U5
+L ATA6560_1:ATA6560,1 U5
 U 1 1 5B822EF5
 P 9550 3000
@@
 L power:+12V #PWR?
 U 1 1 5B9166AE
-P 6200 6550
-F 0 "#PWR?" H 6200 6400 50  0001 C CNN
-F 1 "+12V" H 6200 6700 50  0000 C CNN
-F 2 "" H 6200 6550 50  0001 C CNN
-F 3 "" H 6200 6550 50  0001 C CNN
-	1    6200 6550
+P 6100 6550
+F 0 "#PWR?" H 6100 6400 50  0001 C CNN
+F 1 "+12V" H 6100 6700 50  0000 C CNN
+F 2 "" H 6100 6550 50  0001 C CNN
+F 3 "" H 6100 6550 50  0001 C CNN
+	1    6100 6550
 	1    0    0    -1
 $EndComp
@@
 	1    0    0    -1
 $EndComp
-Text GLabel 6350 6650 1    50   Input ~ 0
-48V
-Text GLabel 12000 7050 1    50   Input ~ 0
-48V
 $Comp
 L power:GND #PWR?
@@
 	1    0    0    -1
 $EndComp
-Wire Wire Line
-	11700 7500 12450 7500
-Wire Wire Line
-	11700 7400 12450 7400
-Wire Wire Line
-	11600 7400 11700 7400
-Wire Wire Line
-	11600 7500 11700 7500
-Wire Wire Line
-	11500 7500 11600 7500
 Connection ~ 11700 7300
 Wire Wire Line
@@
 Wire Wire Line
 	6350 7400 6350 7950
-Wire Wire Line
-	6350 6850 6350 6650
 Connection ~ 6350 6850
 Wire Wire Line
@@
 Text Notes 9800 8300 0    100  Italic 0
 R5485 Header and Selection Switches
-Text Notes 3000 4900 0    100  Italic 0
+Text Notes 2950 4800 0    100  Italic 0
 Arduino Nano
 Text Notes 6550 4600 0    100  Italic 0
@@
 	13050 4600 15000 4600
 Wire Notes Line
-	4350 1850 2600 1850
-Wire Notes Line
 	2600 4950 4350 4950
 Wire Notes Line
@@
 Wire Notes Line
 	9500 6750 13100 6750
-Connection ~ 11600 7500
 Wire Wire Line
 	11600 7500 11600 7700
-Connection ~ 11700 7400
 Wire Wire Line
 	11700 7400 11700 7500
-Connection ~ 11700 7500
 Wire Wire Line
 	11700 7500 11700 7700
@@
 Wire Wire Line
 	3750 7000 3750 7100
-Connection ~ 6200 7000
-Wire Wire Line
-	6200 7000 6200 6550
+Wire Wire Line
+	6100 7000 6100 6550
 Wire Wire Line
 	6150 7950 6350 7950
@@
 Connection ~ 4900 7500
 Wire Wire Line
-	3750 7000 6200 7000
+	3750 7000 6100 7000
 Wire Wire Line
 	3750 7400 4950 7400
@@
 Wire Notes Line
 	13050 2650 13050 4600
+$Comp
+L power:+48V #PWR?
+U 1 1 5BA0A724
+P 6350 6550
+F 0 "#PWR?" H 6350 6400 50  0001 C CNN
+F 1 "+48V" H 6350 6700 50  0000 C CNN
+F 2 "" H 6350 6550 50  0001 C CNN
+F 3 "" H 6350 6550 50  0001 C CNN
+	1    6350 6550
+	1    0    0    -1
+$EndComp
+Connection ~ 6100 7000
+Wire Wire Line
+	6100 7000 6200 7000
+Wire Wire Line
+	6350 6550 6350 6850
+$Comp
+L power:+48V #PWR?
+U 1 1 5BA1B324
+P 12000 7050
+F 0 "#PWR?" H 12000 6900 50  0001 C CNN
+F 1 "+48V" H 12000 7200 50  0000 C CNN
+F 2 "" H 12000 7050 50  0001 C CNN
+F 3 "" H 12000 7050 50  0001 C CNN
+	1    12000 7050
+	1    0    0    -1
+$EndComp
+Wire Wire Line
+	11500 7500 12450 7500
+Wire Wire Line
+	11600 7400 12450 7400
+Text Notes 3300 4950 0    50   Italic 0
+Main uC\n
+Wire Notes Line
+	4350 1850 2600 1850
 $EndSCHEMATC

Commit message: Footprint changes and Zener to Schottky
Parts:
- removed D1: D_Zener, Diode_SMD:D_0603_1608Metric, symbol Device:D_Zener
- added D1: D_Schottky, Diode_SMD:D_SOD-123F, symbol Device:D_Schottky
- C7: renamed from C?; footprint (none) -> Capacitor_THT:C_Disc_D5.0mm_W2.5mm_P2.50mm
- D2: renamed from D?; footprint (none) -> Diode_SMD:D_0603_1608Metric
- R6: renamed from R?; footprint (none) -> Resistor_SMD:R_0603_1608Metric
- R7: renamed from R?; value 100k -> 10k; footprint (none) -> Resistor_SMD:R_0603_1608Metric
- U5: symbol ATA6560_1:ATA6560,1 -> URT_cache:ATA6560,1
- Y1: renamed from Y?; footprint (none) -> Crystal:Crystal_SMD_0603-2Pin_6.0x3.5mm
- gave numbers to parts that had none: 14

Commit message: 0.0.7 change reset RC circuit
Parts:
- C7: value 100uF -> 1uF
- R6: value 1k -> 100k
- U5: symbol URT_cache:ATA6560,1 -> ATA6560_1:ATA6560,1
Changed lines of the file:
@@
 Title "module-tester-board"
 Date "2018-09-26"
-Rev "0.0.6"
+Rev "0.0.7"
 Comp "Missouri University of Science and Technology - Underwater Robotics Team"
 Comment1 "Board for testing ROV modules away from ROV."
@@
 $EndComp
 $Comp
-L URT_cache:ATA6560,1 U5
+L ATA6560_1:ATA6560,1 U5
 U 1 1 5B822EF5
 P 9550 3000
@@
 P 13850 3250
 F 0 "R6" H 13920 3296 50  0000 L CNN
-F 1 "1k" H 13920 3205 50  0000 L CNN
+F 1 "100k" H 13920 3205 50  0000 L CNN
 F 2 "Resistor_SMD:R_0603_1608Metric" V 13780 3250 50  0001 C CNN
 F 3 "~" H 13850 3250 50  0001 C CNN
@@
 P 13850 3700
 F 0 "C7" H 13965 3746 50  0000 L CNN
-F 1 "100uF" H 13965 3655 50  0000 L CNN
+F 1 "1uF" H 13965 3655 50  0000 L CNN
 F 2 "Capacitor_THT:C_Disc_D5.0mm_W2.5mm_P2.50mm" H 13888 3550 50  0001 C CNN
 F 3 "~" H 13850 3700 50  0001 C CNN
