File: module-tester-board.sch (KiCad schematic (older format))
At the start: 28 parts, among them J1 Conn_01x08_Male, J4 Conn_01x04_Male, SW1 SW_SPST, SW2 SW_SPST, SW3 SW_SPST, SW4 SW_SPST, U1 LT8330, U4 MCP2515-EST, U5 ATA6560,1, Y1 20MHz

Commit message: 0.0.9 Add Barrel Jack
Parts:
- added J2: Barrel_Jack, PJ-037A:CUI_PJ-037A, symbol Connector:Barrel_Jack
- U5: symbol ATA6560_1:ATA6560,1 -> URT_cache:ATA6560,1
Connections:
- wire segments 115 -> 119
Other:
- note added: "12V Barrel Jack"
Changed lines of the file:
@@
 Sheet 1 1
 Title "module-tester-board"
-Date "2018-09-27"
-Rev "0.0.8"
+Date "2018-09-30"
+Rev "0.0.9"
 Comp "Missouri University of Science and Technology - Underwater Robotics Team"
 Comment1 "Board for testing ROV modules away from ROV."
@@
 $EndComp
 $Comp
-L ATA6560_1:ATA6560,1 U5
+L URT_cache:ATA6560,1 U5
 U 1 1 5B822EF5
 P 9550 3000
@@
 	-1   0    0    1
 $EndComp
+$Comp
+L Connector:Barrel_Jack J2
+U 1 1 5BB1A586
+P 14500 6000
+F 0 "J2" H 14555 6325 50  0000 C CNN
+F 1 "Barrel_Jack" H 14555 6234 50  0000 C CNN
+F 2 "PJ-037A:CUI_PJ-037A" H 14550 5960 50  0001 C CNN
+F 3 "~" H 14550 5960 50  0001 C CNN
+	1    14500 6000
+	1    0    0    -1
+$EndComp
+$Comp
+L power:+12V #PWR01
+U 1 1 5BB1AACD
+P 14950 5850
+F 0 "#PWR01" H 14950 5700 50  0001 C CNN
+F 1 "+12V" H 14950 6000 50  0000 C CNN
+F 2 "" H 14950 5850 50  0001 C CNN
+F 3 "" H 14950 5850 50  0001 C CNN
+	1    14950 5850
+	1    0    0    -1
+$EndComp
+Wire Wire Line
+	14950 5850 14950 5900
+Wire Wire Line
+	14950 5900 14800 5900
+Wire Wire Line
+	14800 6100 14950 6100
+Wire Wire Line
+	14950 6100 14950 6150
+$Comp
+L power:GND #PWR02
+U 1 1 5BB26857
+P 14950 6150
+F 0 "#PWR02" H 14950 5900 50  0001 C CNN
+F 1 "GND" H 14955 5977 50  0000 C CNN
+F 2 "" H 14950 6150 50  0001 C CNN
+F 3 "" H 14950 6150 50  0001 C CNN
+	1    14950 6150
+	1    0    0    -1
+$EndComp
+Wire Notes Line
+	15100 5550 15100 6650
+Wire Notes Line
+	13850 6650 13850 5550
+Text Notes 13850 6600 0    100  ~ 0
+12V Barrel Jack
+Wire Notes Line
+	15100 6650 13850 6650
+Wire Notes Line
+	13850 5550 15100 5550
 $EndSCHEMATC

Commit message: 0.0.10 Switched switches, footprints, and start Board layout
Parts:
- removed SW1, SW2, SW3, SW4: SW_SPST, Button_Switch_THT:SW_DIP_SPSTx04_Slide_9.78x12.34mm_W7.62mm_P2.54mm, symbol Switch:SW_SPST
- added SW1: SW_DIP_x04, Button_Switch_THT:SW_DIP_SPSTx04_Slide_9.78x12.34mm_W7.62mm_P2.54mm, symbol Switch:SW_DIP_x04
- C7: footprint Capacitor_THT:C_Disc_D5.0mm_W2.5mm_P2.50mm -> Capacitor_SMD:C_0603_1608Metric
Connections:
- wire segments 119 -> 116
Changed lines of the file:
@@
 Title "module-tester-board"
 Date "2018-09-30"
-Rev "0.0.9"
+Rev "0.0.10"
 Comp "Missouri University of Science and Technology - Underwater Robotics Team"
 Comment1 "Board for testing ROV modules away from ROV."
@@
 L Connector:Conn_01x04_Male J4
 U 1 1 5B823405
-P 11500 7900
-F 0 "J4" V 11350 7850 50  0000 C CNN
-F 1 "Conn_01x04_Male" V 11450 7850 50  0000 C CNN
-F 2 "Connector_PinHeader_2.54mm:PinHeader_1x04_P2.54mm_Vertical" H 11500 7900 50  0001 C CNN
-F 3 "~" H 11500 7900 50  0001 C CNN
-	1    11500 7900
-	0    -1   -1   0
+P 11600 7900
+F 0 "J4" V 11450 7850 50  0000 C CNN
+F 1 "Conn_01x04_Male" V 11550 7850 50  0000 C CNN
+F 2 "Connector_PinHeader_2.54mm:PinHeader_1x04_P2.54mm_Vertical" H 11600 7900 50  0001 C CNN
+F 3 "~" H 11600 7900 50  0001 C CNN
+	1    11600 7900
+	0    1    -1   0
 $EndComp
 $Comp
@@
 L Connector:Conn_01x08_Male J1
 U 1 1 5B833C38
-P 12650 7500
-F 0 "J1" V 12400 7450 50  0000 C CNN
-F 1 "Conn_01x08_Male" V 12550 7450 50  0000 C CNN
-F 2 "Connector_PinHeader_2.54mm:PinHeader_1x08_P2.54mm_Vertical" H 12650 7500 50  0001 C CNN
-F 3 "~" H 12650 7500 50  0001 C CNN
-	1    12650 7500
-	-1   0    0    1
+P 12650 7400
+F 0 "J1" V 12400 7350 50  0000 C CNN
+F 1 "Conn_01x08_Male" V 12550 7350 50  0000 C CNN
+F 2 "Connector_PinHeader_2.54mm:PinHeader_1x08_P2.54mm_Vertical" H 12650 7400 50  0001 C CNN
+F 3 "~" H 12650 7400 50  0001 C CNN
+	1    12650 7400
+	-1   0    0    -1
 $EndComp
 Wire Wire Line
@@
 Wire Wire Line
 	6150 7850 6150 7950
-$Comp
-L Switch:SW_SPST SW1
-U 1 1 5B890B45
-P 10650 7150
-F 0 "SW1" H 10200 7150 50  0000 C CNN
-F 1 "SW_SPST" H 9900 7150 50  0000 C CNN
-F 2 "Button_Switch_THT:SW_DIP_SPSTx04_Slide_9.78x12.34mm_W7.62mm_P2.54mm" H 10650 7150 50  0001 C CNN
-F 3 "" H 10650 7150 50  0001 C CNN
-	1    10650 7150
-	1    0    0    -1
-$EndComp
-$Comp
-L Switch:SW_SPST SW2
-U 1 1 5B8959F9
-P 10650 7300
-F 0 "SW2" H 10200 7300 50  0000 C CNN
-F 1 "SW_SPST" H 9900 7300 50  0000 C CNN
-F 2 "Button_Switch_THT:SW_DIP_SPSTx04_Slide_9.78x12.34mm_W7.62mm_P2.54mm" H 10650 7300 50  0001 C CNN
-F 3 "" H 10650 7300 50  0001 C CNN
-	1    10650 7300
-	1    0    0    -1
-$EndComp
-$Comp
-L Switch:SW_SPST SW3
-U 1 1 5B895A49
-P 10650 7450
-F 0 "SW3" H 10100 7450 50  0000 C CNN
-F 1 "SW_SPST" H 9800 7450 50  0000 C CNN
-F 2 "Button_Switch_THT:SW_DIP_SPSTx04_Slide_9.78x12.34mm_W7.62mm_P2.54mm" H 10650 7450 50  0001 C CNN
-F 3 "" H 10650 7450 50  0001 C CNN
-	1    10650 7450
-	1    0    0    -1
-$EndComp
-$Comp
-L Switch:SW_SPST SW4
-U 1 1 5B895AAF
-P 10650 7600
-F 0 "SW4" H 10100 7600 50  0000 C CNN
-F 1 "SW_SPST" H 9800 7600 50  0000 C CNN
-F 2 "Button_Switch_THT:SW_DIP_SPSTx04_Slide_9.78x12.34mm_W7.62mm_P2.54mm" H 10650 7600 50  0001 C CNN
-F 3 "" H 10650 7600 50  0001 C CNN
-	1    10650 7600
-	1    0    0    -1
-$EndComp
 Wire Wire Line
 	3500 4500 3500 4450
@@
 Text GLabel 3000 3350 0    50   Input ~ 0
 PWM0
-Text GLabel 10450 7450 0    50   Input ~ 0
+Text GLabel 10250 7500 0    50   Input ~ 0
 PWM0
 Text GLabel 3000 3450 0    50   Input ~ 0
 PWM1
-Text GLabel 10450 7600 0    50   Input ~ 0
+Text GLabel 10250 7600 0    50   Input ~ 0
 PWM1
-Text GLabel 10450 7150 0    50   Input ~ 0
+Text GLabel 10250 7300 0    50   Input ~ 0
 A0
 Text GLabel 4000 3450 2    50   Input ~ 0
 A0
-Text GLabel 10450 7300 0    50   Input ~ 0
+Text GLabel 10250 7400 0    50   Input ~ 0
 A1
 Text GLabel 4000 3550 2    50   Input ~ 0
@@
 $EndComp
 Wire Wire Line
-	10850 7450 11500 7450
-Wire Wire Line
-	11500 7450 11500 7500
-Wire Wire Line
-	11600 7300 11600 7400
-Wire Wire Line
-	10850 7300 11600 7300
-Wire Wire Line
-	11700 7150 11700 7300
-Wire Wire Line
-	10850 7150 11700 7150
+	10850 7500 11500 7500
 Wire Wire Line
 	12450 7300 11700 7300
@@
 	1    0    0    -1
 $EndComp
-Connection ~ 11700 7300
 Wire Wire Line
 	11700 7300 11700 7400
-Connection ~ 11600 7400
 Wire Wire Line
 	11600 7400 11600 7500
@@
 F 0 "C7" H 13965 3746 50  0000 L CNN
 F 1 "1uF" H 13965 3655 50  0000 L CNN
-F 2 "Capacitor_THT:C_Disc_D5.0mm_W2.5mm_P2.50mm" H 13888 3550 50  0001 C CNN
+F 2 "Capacitor_SMD:C_0603_1608Metric" H 13888 3550 50  0001 C CNN
 F 3 "~" H 13850 3700 50  0001 C CNN
 	1    13850 3700
@@
 Wire Notes Line
 	13850 5550 15100 5550
+$Comp
+L Switch:SW_DIP_x04 SW1
+U 1 1 5BB6B3B3
+P 10550 7500
+F 0 "SW1" H 10550 7967 50  0000 C CNN
+F 1 "SW_DIP_x04" H 10550 7876 50  0000 C CNN
+F 2 "Button_Switch_THT:SW_DIP_SPSTx04_Slide_9.78x12.34mm_W7.62mm_P2.54mm" H 10550 7500 50  0001 C CNN
+F 3 "" H 10550 7500 50  0001 C CNN
+	1    10550 7500
+	1    0    0    -1
+$EndComp
+Wire Wire Line
+	11700 7300 10850 7300
+Connection ~ 11700 7300
+Wire Wire Line
+	10850 7400 11600 7400
+Connection ~ 11600 7400
 $EndSCHEMATC
