File: Gimble Goblin.sch (KiCad schematic (older format))
At the start: 6 parts

Commit message: 0.0.1
First complete (?) schematic
Parts:
- added C? (x2): 15p, Capacitor_SMD:C_0603_1608Metric, symbol Device:C_Small
- added R? (x2): 10k, Resistor_SMD:R_0603_1608Metric, symbol Device:R
- added R?: 1M, Resistor_SMD:R_0603_1608Metric, symbol Device:R
- added U?: MCP2515-EST, Package_SO:TSSOP-20_4.4x6.5mm_P0.65mm, symbol Interface_CAN_LIN:MCP2515-EST
- added U?: ATA6560,1, Package_SO:SOIC-8_3.9x4.9mm_P1.27mm, symbol URT_cache:ATA6560,1
- added Y?: 20MHz, Crystal:Crystal_SMD_0603-2Pin_6.0x3.5mm, symbol Device:Crystal
Connections:
- net labels added: CANH, CANL, GND, INT, RX0, RX1, Reset, SCK, SI, SO, SS, TX0, TX1, TX2
- wire segments 0 -> 91
- no-connect marks 0 -> 1
Other:
- note added: "CAN Communication using MCP2515 and ATA6560"
- moved on the sheet: J?
