File: ProofOfConceptBoardV1.sch (KiCad schematic (older format))
At the start: 20 parts

Commit message: 0.0.2 Fixed Last Commit. Uploaded Schematic for Review.
Parts:
- added 100uF?, 15pF? (x2): C, symbol Device:C
- added 10k? (x3), 1K?, 1M?: R, symbol Device:R
- added 20MHz?: Crystal, symbol Device:Crystal
- added A?: Arduino_Nano_v3.x, Module:Arduino_Nano, symbol MCU_Module:Arduino_Nano_v3.x
- added A?: ATA6560, symbol ATA6560:ATA6560
- added D? (x2): LED, symbol Device:LED
- added D?: DIODE, symbol pspice:DIODE
- added R? (x2): 220, symbol Device:R
- added TP? (x2): TestPoint, symbol Connector:TestPoint
- added U?: MCP2515-EST, Package_SO:TSSOP-20_4.4x6.5mm_P0.65mm, symbol Interface_CAN_LIN:MCP2515-EST
- renumbered 3uF to 100uF, 1M to 1K
Connections:
- net labels added: CANRX_2, CANTX_2, INT0_2, INT1_2, INTMCP_2, MISO_2, MOSI_2, OSC1_2, OSC2_2, SCK_2, SS_2, TBUF0_2, TBUF1_2, TBUF2_2
- wire segments 53 -> 102
- no-connect marks 6 -> 26
Other:
- note added: "ATA6560. Mirrored on Other Side.\nReceiver for message received by devices on CAN BUS line"
- note added: "ATA6560\nReceiver for message received by devices on CAN BUS line"
- note added: "Arduino Nano. Mirrored on other Side\nCoordinates when and how the CAN system\noperates, transmit, and receive."
- note added: "Arduino Nano\nCoordinates when and how the CAN system\noperates, transmit, and receive."
- note added: "MCP1252 Oscillator Circuit, Mirrored on Other Side\n"
- note added: "MCP1252 Oscillator Circuit\n"
- note added: "MCP1252. Mirrored on Other Side\nCAN interface for messages from\nand to the Arduino controller and CAN BUS line."
- note added: "MCP1252\nCAN interface for messages from\nand to the Arduino controller and CAN BUS line."
- note removed: "I don't know what else we might need to attach so left analog and digital pins alone\n"
- moved on the sheet: 100uF, 15pF, 20MHz, C?, D?, TP?, U?

Commit message: 0.0.3
Schematic Fixes + PCB Layout
Parts:
- removed TP? (x2): TestPoint, symbol Connector:TestPoint
- A3, A4: renamed from A?; footprint (none) -> Package_SO:SOIC-8_3.9x4.9mm_P1.27mm
- C1: renamed from C?; value 22uF -> 100uF; footprint (none) -> Capacitor_THT:CP_Radial_D5.0mm_P2.00mm
- C2, C4: renamed from 15pF; value C -> 15pF; footprint (none) -> Capacitor_SMD:C_0603_1608Metric
- C3, C5: renamed from 15pF?; value C -> 15pF; footprint (none) -> Capacitor_SMD:C_0603_1608Metric
- C6: renamed from 100uF; value C -> 1uF; footprint (none) -> Capacitor_SMD:C_0603_1608Metric
- C7: renamed from 100uF?; value C -> 1uF; footprint (none) -> Capacitor_SMD:C_0603_1608Metric
- Crystal1: renamed from 20MHz; value Crystal -> 20MHz; footprint (none) -> Crystal:Crystal_SMD_0603-2Pin_6.0x3.5mm
- Crystal2: renamed from 20MHz?; value Crystal -> 20 MHz; footprint (none) -> Crystal:Crystal_SMD_0603-2Pin_6.0x3.5mm
- D1, D2, D3, D4: renamed from D?; footprint (none) -> LED_SMD:LED_Cree-XQ
- D5, D6: renamed from D?; footprint (none) -> Diode_SMD:D_0603_1608Metric
- R1, R2, R3, R4: renamed from R?; footprint (none) -> Resistor_SMD:R_0603_1608Metric
- R10: renamed from 1K?; value R -> 100k; footprint (none) -> Resistor_SMD:R_0603_1608Metric
- R11, R13, R14, R8: renamed from 10k?; value R -> 10k; footprint (none) -> Resistor_SMD:R_0603_1608Metric
- R12, R7: renamed from 10k; value R -> 10k; footprint (none) -> Resistor_SMD:R_0603_1608Metric
- R5: renamed from 1M; value R -> 1M; footprint (none) -> Resistor_SMD:R_0603_1608Metric
- R6: renamed from 1M?; value R -> 1M; footprint (none) -> Resistor_SMD:R_0603_1608Metric
- R9: renamed from 1K; value R -> 100k; footprint (none) -> Resistor_SMD:R_0603_1608Metric
- TP1, TP2: renamed from TP?; footprint (none) -> TestPoint:TestPoint_THTPad_1.0x1.0mm_Drill0.5mm
- gave numbers to parts that had none: 4
Connections:
- net labels added: VCC
- net labels removed: +3.3V
- wire segments 102 -> 100
- no-connect marks 26 -> 28
Other:
- moved on the sheet: C1, C2, C3, C4, C5, Crystal1, Crystal2

Commit message: 0.0.5 Changes to board after review. Also with og backup.  Sch changes
Parts:
- added C10, C11, C12, C8, C9: 100nF, Capacitor_SMD:C_0603_1608Metric, symbol Device:C
- C1: value 100uF -> 100nF; footprint Capacitor_THT:CP_Radial_D5.0mm_P2.00mm -> Capacitor_SMD:C_0603_1608Metric
Changed lines of the file:
@@
-$EndComp
-$Comp
-L power:+5V #PWR015
-U 1 1 5B873C91
-P 5800 900
-F 0 "#PWR015" H 5800 750 50  0001 C CNN
-F 1 "+5V" H 5900 950 50  0000 C CNN
-F 2 "" H 5800 900 50  0001 C CNN
-F 3 "" H 5800 900 50  0001 C CNN
-	1    5800 900
-	1    0    0    -1
-$EndComp
-$Comp
-L Device:C C1
-U 1 1 5B873D56
-P 5800 1050
-F 0 "C1" H 5915 1096 50  0000 L CNN
-F 1 "100uF" H 5915 1005 50  0000 L CNN
-F 2 "Capacitor_THT:CP_Radial_D5.0mm_P2.00mm" H 5838 900 50  0001 C CNN
-F 3 "~" H 5800 1050 50  0001 C CNN
-	1    5800 1050
-	1    0    0    -1
-$EndComp
-$Comp
-L power:GNDREF #PWR016
-U 1 1 5B873DA0
-P 5800 1200
-F 0 "#PWR016" H 5800 950 50  0001 C CNN
-F 1 "GNDREF" H 6000 1150 50  0000 C CNN
-F 2 "" H 5800 1200 50  0001 C CNN
-F 3 "" H 5800 1200 50  0001 C CNN
-	1    5800 1200
-	1    0    0    -1
 $EndComp
 $Comp
@@
 Wire Notes Line
 	450  5100 16550 5100
+$Comp
+L power:+5V #PWR0101
+U 1 1 5BDA9632
+P 3900 1750
+F 0 "#PWR0101" H 3900 1600 50  0001 C CNN
+F 1 "+5V" H 4000 1800 50  0000 C CNN
+F 2 "" H 3900 1750 50  0001 C CNN
+F 3 "" H 3900 1750 50  0001 C CNN
+	1    3900 1750
+	1    0    0    -1
+$EndComp
+$Comp
+L Device:C C1
+U 1 1 5BDA9638
+P 3900 1900
+F 0 "C1" H 4015 1946 50  0000 L CNN
+F 1 "100nF" H 4015 1855 50  0000 L CNN
+F 2 "Capacitor_SMD:C_0603_1608Metric" H 3938 1750 50  0001 C CNN
+F 3 "~" H 3900 1900 50  0001 C CNN
+	1    3900 1900
+	1    0    0    -1
+$EndComp
+$Comp
+L power:GNDREF #PWR0102
+U 1 1 5BDA963F
+P 3900 2050
+F 0 "#PWR0102" H 3900 1800 50  0001 C CNN
+F 1 "GNDREF" H 4100 2000 50  0000 C CNN
+F 2 "" H 3900 2050 50  0001 C CNN
+F 3 "" H 3900 2050 50  0001 C CNN
+	1    3900 2050
+	1    0    0    -1
+$EndComp
+$Comp
+L power:+5V #PWR0103
+U 1 1 5BDAC127
+P 10400 1150
+F 0 "#PWR0103" H 10400 1000 50  0001 C CNN
+F 1 "+5V" H 10500 1200 50  0000 C CNN
+F 2 "" H 10400 1150 50  0001 C CNN
+F 3 "" H 10400 1150 50  0001 C CNN
+	1    10400 1150
+	1    0    0    -1
+$EndComp
+$Comp
+L Device:C C9
+U 1 1 5BDAC12D
+P 10400 1300
+F 0 "C9" H 10515 1346 50  0000 L CNN
+F 1 "100nF" H 10515 1255 50  0000 L CNN
+F 2 "Capacitor_SMD:C_0603_1608Metric" H 10438 1150 50  0001 C CNN
+F 3 "~" H 10400 1300 50  0001 C CNN
+	1    10400 1300
+	1    0    0    -1
+$EndComp
+$Comp
+L power:GNDREF #PWR0104
+U 1 1 5BDAC134
+P 10400 1450
+F 0 "#PWR0104" H 10400 1200 50  0001 C CNN
+F 1 "GNDREF" H 10600 1400 50  0000 C CNN
+F 2 "" H 10400 1450 50  0001 C CNN
+F 3 "" H 10400 1450 50  0001 C CNN
+	1    10400 1450
+	1    0    0    -1
+$EndComp
+$Comp
+L power:+5V #PWR0105
+U 1 1 5BDAED22
+P 3950 5750
+F 0 "#PWR0105" H 3950 5600 50  0001 C CNN
+F 1 "+5V" H 4050 5800 50  0000 C CNN
+F 2 "" H 3950 5750 50  0001 C CNN
+F 3 "" H 3950 5750 50  0001 C CNN
+	1    3950 5750
+	1    0    0    -1
+$EndComp
+$Comp
+L Device:C C8
+U 1 1 5BDAED28
+P 3950 5900
+F 0 "C8" H 4065 5946 50  0000 L CNN
+F 1 "100nF" H 4065 5855 50  0000 L CNN
+F 2 "Capacitor_SMD:C_0603_1608Metric" H 3988 5750 50  0001 C CNN
+F 3 "~" H 3950 5900 50  0001 C CNN
+	1    3950 5900
+	1    0    0    -1
+$EndComp
+$Comp
+L power:GNDREF #PWR0106
+U 1 1 5BDAED2F
+P 3950 6050
+F 0 "#PWR0106" H 3950 5800 50  0001 C CNN
+F 1 "GNDREF" H 4150 6000 50  0000 C CNN
+F 2 "" H 3950 6050 50  0001 C CNN
+F 3 "" H 3950 6050 50  0001 C CNN
+	1    3950 6050
+	1    0    0    -1
+$EndComp
+$Comp
+L power:+5V #PWR0107
+U 1 1 5BDB185D
+P 10900 5700
+F 0 "#PWR0107" H 10900 5550 50  0001 C CNN
+F 1 "+5V" H 11000 5750 50  0000 C CNN
+F 2 "" H 10900 5700 50  0001 C CNN
+F 3 "" H 10900 5700 50  0001 C CNN
+	1    10900 5700
+	1    0    0    -1
+$EndComp
+$Comp
+L Device:C C10
+U 1 1 5BDB1863
+P 10900 5850
+F 0 "C10" H 11015 5896 50  0000 L CNN
+F 1 "100nF" H 11015 5805 50  0000 L CNN
+F 2 "Capacitor_SMD:C_0603_1608Metric" H 10938 5700 50  0001 C CNN
+F 3 "~" H 10900 5850 50  0001 C CNN
+	1    10900 5850
+	1    0    0    -1
+$EndComp
+$Comp
+L power:GNDREF #PWR0108
+U 1 1 5BDB186A
+P 10900 6000
+F 0 "#PWR0108" H 10900 5750 50  0001 C CNN
+F 1 "GNDREF" H 11100 5950 50  0000 C CNN
+F 2 "" H 10900 6000 50  0001 C CNN
+F 3 "" H 10900 6000 50  0001 C CNN
+	1    10900 6000
+	1    0    0    -1
+$EndComp
+$Comp
+L power:+5V #PWR0109
+U 1 1 5BDBA8F9
+P 13500 6250
+F 0 "#PWR0109" H 13500 6100 50  0001 C CNN
+F 1 "+5V" H 13600 6300 50  0000 C CNN
+F 2 "" H 13500 6250 50  0001 C CNN
+F 3 "" H 13500 6250 50  0001 C CNN
+	1    13500 6250
+	1    0    0    -1
+$EndComp
+$Comp
+L Device:C C12
+U 1 1 5BDBA8FF
+P 13500 6400
+F 0 "C12" H 13615 6446 50  0000 L CNN
+F 1 "100nF" H 13615 6355 50  0000 L CNN
+F 2 "Capacitor_SMD:C_0603_1608Metric" H 13538 6250 50  0001 C CNN
+F 3 "~" H 13500 6400 50  0001 C CNN
+	1    13500 6400
+	1    0    0    -1
+$EndComp
+$Comp
+L power:GNDREF #PWR0110
+U 1 1 5BDBA906
+P 13500 6550
+F 0 "#PWR0110" H 13500 6300 50  0001 C CNN
+F 1 "GNDREF" H 13700 6500 50  0000 C CNN
+F 2 "" H 13500 6550 50  0001 C CNN
+F 3 "" H 13500 6550 50  0001 C CNN
+	1    13500 6550
+	1    0    0    -1
+$EndComp
+$Comp
+L power:+5V #PWR0111
+U 1 1 5BDBD491
+P 13350 1550
+F 0 "#PWR0111" H 13350 1400 50  0001 C CNN
+F 1 "+5V" H 13450 1600 50  0000 C CNN
+F 2 "" H 13350 1550 50  0001 C CNN
+F 3 "" H 13350 1550 50  0001 C CNN
+	1    13350 1550
+	1    0    0    -1
+$EndComp
+$Comp
+L Device:C C11
+U 1 1 5BDBD497
+P 13350 1700
+F 0 "C11" H 13465 1746 50  0000 L CNN
+F 1 "100nF" H 13465 1655 50  0000 L CNN
+F 2 "Capacitor_SMD:C_0603_1608Metric" H 13388 1550 50  0001 C CNN
+F 3 "~" H 13350 1700 50  0001 C CNN
+	1    13350 1700
+	1    0    0    -1
+$EndComp
+$Comp
+L power:GNDREF #PWR0112
+U 1 1 5BDBD49E
+P 13350 1850
+F 0 "#PWR0112" H 13350 1600 50  0001 C CNN
+F 1 "GNDREF" H 13550 1800 50  0000 C CNN
+F 2 "" H 13350 1850 50  0001 C CNN
+F 3 "" H 13350 1850 50  0001 C CNN
+	1    13350 1850
+	1    0    0    -1
+$EndComp
 $EndSCHEMATC
