File: ProofOfConceptBoardV1Safety.sch (KiCad schematic (older format))
At the start: 42 parts, among them U1 MCP2515-EST, U2 MCP2515-EST

Commit message: 0.0.5 Changes to board after review. Also with og backup.  Sch changes
Parts:
- removed C10, C11, C12, C8, C9: 100nF, Capacitor_SMD:C_0603_1608Metric, symbol Device:C
- C1: value 100nF -> 100uF; footprint Capacitor_SMD:C_0603_1608Metric -> Capacitor_THT:CP_Radial_D5.0mm_P2.00mm
Changed lines of the file:
@@
+$EndComp
+$Comp
+L power:+5V #PWR015
+U 1 1 5B873C91
+P 5250 1350
+F 0 "#PWR015" H 5250 1200 50  0001 C CNN
+F 1 "+5V" H 5350 1400 50  0000 C CNN
+F 2 "" H 5250 1350 50  0001 C CNN
+F 3 "" H 5250 1350 50  0001 C CNN
+	1    5250 1350
+	1    0    0    -1
+$EndComp
+$Comp
+L Device:C C1
+U 1 1 5B873D56
+P 5250 1500
+F 0 "C1" H 5365 1546 50  0000 L CNN
+F 1 "100uF" H 5365 1455 50  0000 L CNN
+F 2 "Capacitor_THT:CP_Radial_D5.0mm_P2.00mm" H 5288 1350 50  0001 C CNN
+F 3 "~" H 5250 1500 50  0001 C CNN
+	1    5250 1500
+	1    0    0    -1
+$EndComp
+$Comp
+L power:GNDREF #PWR016
+U 1 1 5B873DA0
+P 5250 1650
+F 0 "#PWR016" H 5250 1400 50  0001 C CNN
+F 1 "GNDREF" H 5450 1600 50  0000 C CNN
+F 2 "" H 5250 1650 50  0001 C CNN
+F 3 "" H 5250 1650 50  0001 C CNN
+	1    5250 1650
+	1    0    0    -1
 $EndComp
 $Comp
@@
 Wire Notes Line
 	450  5100 16550 5100
-$Comp
-L power:+5V #PWR0101
-U 1 1 5BDA9632
-P 3900 1750
-F 0 "#PWR0101" H 3900 1600 50  0001 C CNN
-F 1 "+5V" H 4000 1800 50  0000 C CNN
-F 2 "" H 3900 1750 50  0001 C CNN
-F 3 "" H 3900 1750 50  0001 C CNN
-	1    3900 1750
-	1    0    0    -1
-$EndComp
-$Comp
-L Device:C C1
-U 1 1 5BDA9638
-P 3900 1900
-F 0 "C1" H 4015 1946 50  0000 L CNN
-F 1 "100nF" H 4015 1855 50  0000 L CNN
-F 2 "Capacitor_SMD:C_0603_1608Metric" H 3938 1750 50  0001 C CNN
-F 3 "~" H 3900 1900 50  0001 C CNN
-	1    3900 1900
-	1    0    0    -1
-$EndComp
-$Comp
-L power:GNDREF #PWR0102
-U 1 1 5BDA963F
-P 3900 2050
-F 0 "#PWR0102" H 3900 1800 50  0001 C CNN
-F 1 "GNDREF" H 4100 2000 50  0000 C CNN
-F 2 "" H 3900 2050 50  0001 C CNN
-F 3 "" H 3900 2050 50  0001 C CNN
-	1    3900 2050
-	1    0    0    -1
-$EndComp
-$Comp
-L power:+5V #PWR0103
-U 1 1 5BDAC127
-P 10400 1150
-F 0 "#PWR0103" H 10400 1000 50  0001 C CNN
-F 1 "+5V" H 10500 1200 50  0000 C CNN
-F 2 "" H 10400 1150 50  0001 C CNN
-F 3 "" H 10400 1150 50  0001 C CNN
-	1    10400 1150
-	1    0    0    -1
-$EndComp
-$Comp
-L Device:C C9
-U 1 1 5BDAC12D
-P 10400 1300
-F 0 "C9" H 10515 1346 50  0000 L CNN
-F 1 "100nF" H 10515 1255 50  0000 L CNN
-F 2 "Capacitor_SMD:C_0603_1608Metric" H 10438 1150 50  0001 C CNN
-F 3 "~" H 10400 1300 50  0001 C CNN
-	1    10400 1300
-	1    0    0    -1
-$EndComp
-$Comp
-L power:GNDREF #PWR0104
-U 1 1 5BDAC134
-P 10400 1450
-F 0 "#PWR0104" H 10400 1200 50  0001 C CNN
-F 1 "GNDREF" H 10600 1400 50  0000 C CNN
-F 2 "" H 10400 1450 50  0001 C CNN
-F 3 "" H 10400 1450 50  0001 C CNN
-	1    10400 1450
-	1    0    0    -1
-$EndComp
-$Comp
-L power:+5V #PWR0105
-U 1 1 5BDAED22
-P 3950 5750
-F 0 "#PWR0105" H 3950 5600 50  0001 C CNN
-F 1 "+5V" H 4050 5800 50  0000 C CNN
-F 2 "" H 3950 5750 50  0001 C CNN
-F 3 "" H 3950 5750 50  0001 C CNN
-	1    3950 5750
-	1    0    0    -1
-$EndComp
-$Comp
-L Device:C C8
-U 1 1 5BDAED28
-P 3950 5900
-F 0 "C8" H 4065 5946 50  0000 L CNN
-F 1 "100nF" H 4065 5855 50  0000 L CNN
-F 2 "Capacitor_SMD:C_0603_1608Metric" H 3988 5750 50  0001 C CNN
-F 3 "~" H 3950 5900 50  0001 C CNN
-	1    3950 5900
-	1    0    0    -1
-$EndComp
-$Comp
-L power:GNDREF #PWR0106
-U 1 1 5BDAED2F
-P 3950 6050
-F 0 "#PWR0106" H 3950 5800 50  0001 C CNN
-F 1 "GNDREF" H 4150 6000 50  0000 C CNN
-F 2 "" H 3950 6050 50  0001 C CNN
-F 3 "" H 3950 6050 50  0001 C CNN
-	1    3950 6050
-	1    0    0    -1
-$EndComp
-$Comp
-L power:+5V #PWR0107
-U 1 1 5BDB185D
-P 10900 5700
-F 0 "#PWR0107" H 10900 5550 50  0001 C CNN
-F 1 "+5V" H 11000 5750 50  0000 C CNN
-F 2 "" H 10900 5700 50  0001 C CNN
-F 3 "" H 10900 5700 50  0001 C CNN
-	1    10900 5700
-	1    0    0    -1
-$EndComp
-$Comp
-L Device:C C10
-U 1 1 5BDB1863
-P 10900 5850
-F 0 "C10" H 11015 5896 50  0000 L CNN
-F 1 "100nF" H 11015 5805 50  0000 L CNN
-F 2 "Capacitor_SMD:C_0603_1608Metric" H 10938 5700 50  0001 C CNN
-F 3 "~" H 10900 5850 50  0001 C CNN
-	1    10900 5850
-	1    0    0    -1
-$EndComp
-$Comp
-L power:GNDREF #PWR0108
-U 1 1 5BDB186A
-P 10900 6000
-F 0 "#PWR0108" H 10900 5750 50  0001 C CNN
-F 1 "GNDREF" H 11100 5950 50  0000 C CNN
-F 2 "" H 10900 6000 50  0001 C CNN
-F 3 "" H 10900 6000 50  0001 C CNN
-	1    10900 6000
-	1    0    0    -1
-$EndComp
-$Comp
-L power:+5V #PWR0109
-U 1 1 5BDBA8F9
-P 13500 6250
-F 0 "#PWR0109" H 13500 6100 50  0001 C CNN
-F 1 "+5V" H 13600 6300 50  0000 C CNN
-F 2 "" H 13500 6250 50  0001 C CNN
-F 3 "" H 13500 6250 50  0001 C CNN
-	1    13500 6250
-	1    0    0    -1
-$EndComp
-$Comp
-L Device:C C12
-U 1 1 5BDBA8FF
-P 13500 6400
-F 0 "C12" H 13615 6446 50  0000 L CNN
-F 1 "100nF" H 13615 6355 50  0000 L CNN
-F 2 "Capacitor_SMD:C_0603_1608Metric" H 13538 6250 50  0001 C CNN
-F 3 "~" H 13500 6400 50  0001 C CNN
-	1    13500 6400
-	1    0    0    -1
-$EndComp
-$Comp
-L power:GNDREF #PWR0110
-U 1 1 5BDBA906
-P 13500 6550
-F 0 "#PWR0110" H 13500 6300 50  0001 C CNN
-F 1 "GNDREF" H 13700 6500 50  0000 C CNN
-F 2 "" H 13500 6550 50  0001 C CNN
-F 3 "" H 13500 6550 50  0001 C CNN
-	1    13500 6550
-	1    0    0    -1
-$EndComp
-$Comp
-L power:+5V #PWR0111
-U 1 1 5BDBD491
-P 13350 1550
-F 0 "#PWR0111" H 13350 1400 50  0001 C CNN
-F 1 "+5V" H 13450 1600 50  0000 C CNN
-F 2 "" H 13350 1550 50  0001 C CNN
-F 3 "" H 13350 1550 50  0001 C CNN
-	1    13350 1550
-	1    0    0    -1
-$EndComp
-$Comp
-L Device:C C11
-U 1 1 5BDBD497
-P 13350 1700
-F 0 "C11" H 13465 1746 50  0000 L CNN
-F 1 "100nF" H 13465 1655 50  0000 L CNN
-F 2 "Capacitor_SMD:C_0603_1608Metric" H 13388 1550 50  0001 C CNN
-F 3 "~" H 13350 1700 50  0001 C CNN
-	1    13350 1700
-	1    0    0    -1
-$EndComp
-$Comp
-L power:GNDREF #PWR0112
-U 1 1 5BDBD49E
-P 13350 1850
-F 0 "#PWR0112" H 13350 1600 50  0001 C CNN
-F 1 "GNDREF" H 13550 1800 50  0000 C CNN
-F 2 "" H 13350 1850 50  0001 C CNN
-F 3 "" H 13350 1850 50  0001 C CNN
-	1    13350 1850
-	1    0    0    -1
-$EndComp
 $EndSCHEMATC
