File: ProgrammerBoard.sch (KiCad schematic (older format))
At the start: 11 parts

Commit message: Picked out parts
Parts:
- removed D? (x2): SFH460, Package_TO_SOT_THT:TO-18-2_Window, symbol LED:SFH460
- added RX: Blue, symbol Device:LED
- added TX: Green, symbol Device:LED
- C1: renamed from C?; value C -> 100nF
- F1: value Fuse -> 500mA
- J?: value Conn_01x08_Male -> 8_Pin
- R1, R2: renamed from R?; value R -> 1K
- R100: renamed from R?; value R -> R3
- R100: renamed from R?; value R -> R4
- gave numbers to parts that had none: 1
Connections:
- net labels added: GNDREF
- net labels removed: VCC
- wire segments 35 -> 45
- no-connect marks 12 -> 15
Other:
- moved on the sheet: C1, J?, R2
Changed lines of the file:
@@
 $EndDescr
 $Comp
-L Interface_USB:FT232RL U?
+L Interface_USB:FT232RL IC1
 U 1 1 5B7F2CF3
 P 3450 2850
-F 0 "U?" H 3450 4028 50  0000 C CNN
-F 1 "FT232RL" H 3450 3937 50  0000 C CNN
+F 0 "IC1" H 2900 3850 50  0000 C CNN
+F 1 "FT232RL" H 3000 3750 50  0000 C CNN
 F 2 "Package_SO:SSOP-28_5.3x10.2mm_P0.65mm" H 3450 2850 50  0001 C CNN
 F 3 "http://www.ftdichip.com/Products/ICs/FT232RL.htm" H 3450 2850 50  0001 C CNN
@@
 P 2250 2250
 F 0 "F1" V 2053 2250 50  0000 C CNN
-F 1 "Fuse" V 2144 2250 50  0000 C CNN
+F 1 "500mA" V 2144 2250 50  0000 C CNN
 F 2 "" V 2180 2250 50  0001 C CNN
 F 3 "~" H 2250 2250 50  0001 C CNN
@@
 Wire Wire Line
 	2050 2250 2100 2250
-$Comp
-L power:VCC #PWR?
-U 1 1 5B7F3986
-P 2400 2100
-F 0 "#PWR?" H 2400 1950 50  0001 C CNN
-F 1 "VCC" H 2417 2273 50  0000 C CNN
-F 2 "" H 2400 2100 50  0001 C CNN
-F 3 "" H 2400 2100 50  0001 C CNN
-	1    2400 2100
-	1    0    0    -1
-$EndComp
-Wire Wire Line
-	2400 2250 2400 2100
 $Comp
 L power:Earth #PWR?
@@
 L power:Earth #PWR?
 U 1 1 5B7F436B
-P 3950 3900
-F 0 "#PWR?" H 3950 3650 50  0001 C CNN
-F 1 "Earth" H 3950 3750 50  0001 C CNN
-F 2 "" H 3950 3900 50  0001 C CNN
-F 3 "~" H 3950 3900 50  0001 C CNN
-	1    3950 3900
-	0    -1   -1   0
+P 3950 4050
+F 0 "#PWR?" H 3950 3800 50  0001 C CNN
+F 1 "Earth" H 3950 3900 50  0001 C CNN
+F 2 "" H 3950 4050 50  0001 C CNN
+F 3 "~" H 3950 4050 50  0001 C CNN
+	1    3950 4050
+	1    0    0    -1
 $EndComp
 Wire Wire Line
@@
 	3650 3850 3650 3900
 Connection ~ 3650 3900
-Wire Wire Line
-	3650 3900 3950 3900
 $Comp
 L power:Earth #PWR?
 U 1 1 5B7F45BE
-P 2350 3550
-F 0 "#PWR?" H 2350 3300 50  0001 C CNN
-F 1 "Earth" H 2350 3400 50  0001 C CNN
-F 2 "" H 2350 3550 50  0001 C CNN
-F 3 "~" H 2350 3550 50  0001 C CNN
-	1    2350 3550
-	0    1    1    0
+P 2350 3750
+F 0 "#PWR?" H 2350 3500 50  0001 C CNN
+F 1 "Earth" H 2350 3600 50  0001 C CNN
+F 2 "" H 2350 3750 50  0001 C CNN
+F 3 "~" H 2350 3750 50  0001 C CNN
+	1    2350 3750
+	1    0    0    -1
 $EndComp
 Wire Wire Line
 	2650 3550 2350 3550
-$Comp
-L power:+5V #PWR?
-U 1 1 5B7F5269
-P 3550 1550
-F 0 "#PWR?" H 3550 1400 50  0001 C CNN
-F 1 "+5V" H 3565 1723 50  0000 C CNN
-F 2 "" H 3550 1550 50  0001 C CNN
-F 3 "" H 3550 1550 50  0001 C CNN
-	1    3550 1550
-	1    0    0    -1
-$EndComp
-Wire Wire Line
-	3550 1850 3550 1550
 $Comp
 L power:+5V #PWR?
@@
 	1    0    0    -1
 $EndComp
-Wire Wire Line
-	3350 1850 3350 1700
-$Comp
-L Device:C C?
+$Comp
+L Device:C C1
 U 1 1 5B7F5A97
-P 4650 2350
-F 0 "C?" V 4398 2350 50  0000 C CNN
-F 1 "C" V 4489 2350 50  0000 C CNN
-F 2 "" H 4688 2200 50  0001 C CNN
-F 3 "~" H 4650 2350 50  0001 C CNN
-	1    4650 2350
-	1    0    0    -1
-$EndComp
-Text Notes 4650 2300 1    50   ~ 0
+P 4800 2350
+F 0 "C1" V 4548 2350 50  0000 C CNN
+F 1 "100nF" V 4639 2350 50  0000 C CNN
+F 2 "" H 4838 2200 50  0001 C CNN
+F 3 "~" H 4800 2350 50  0001 C CNN
+	1    4800 2350
+	1    0    0    -1
+$EndComp
+Text Notes 4800 2300 1    50   ~ 0
 RESET
 $Comp
-L Device:R R?
+L Device:R R1
 U 1 1 5B7F5F0D
 P 5600 2900
-F 0 "R?" H 5670 2946 50  0000 L CNN
-F 1 "R" H 5670 2855 50  0000 L CNN
+F 0 "R1" H 5670 2946 50  0000 L CNN
+F 1 "1K" H 5670 2855 50  0000 L CNN
 F 2 "" V 5530 2900 50  0001 C CNN
 F 3 "~" H 5600 2900 50  0001 C CNN
@@
 $EndComp
 $Comp
-L Device:R R?
+L Device:R R2
 U 1 1 5B7F5F7D
-P 6500 2900
-F 0 "R?" H 6570 2946 50  0000 L CNN
-F 1 "R" H 6570 2855 50  0000 L CNN
-F 2 "" V 6430 2900 50  0001 C CNN
-F 3 "~" H 6500 2900 50  0001 C CNN
-	1    6500 2900
+P 5950 2900
+F 0 "R2" H 6020 2946 50  0000 L CNN
+F 1 "1K" H 6020 2855 50  0000 L CNN
+F 2 "" V 5880 2900 50  0001 C CNN
+F 3 "~" H 5950 2900 50  0001 C CNN
+	1    5950 2900
 	1    0    0    -1
 $EndComp
@@
 	5600 3150 5600 3050
 Wire Wire Line
-	4250 3250 6500 3250
-Wire Wire Line
-	6500 3250 6500 3050
-$Comp
-L LED:SFH460 D?
-U 1 1 5B7F6806
-P 5600 2300
-F 0 "D?" V 5504 2452 50  0000 L CNN
-F 1 "SFH460" V 5595 2452 50  0000 L CNN
-F 2 "Package_TO_SOT_THT:TO-18-2_Window" H 5600 2475 50  0001 C CNN
-F 3 "http://www.osram-os.com/Graphics/XPic6/00029609_0.pdf/SFh%20460.pdf" H 5550 2300 50  0001 C CNN
-	1    5600 2300
-	0    -1   -1   0
-$EndComp
-$Comp
-L LED:SFH460 D?
-U 1 1 5B7F6875
-P 6500 2300
-F 0 "D?" V 6404 2452 50  0000 L CNN
-F 1 "SFH460" V 6495 2452 50  0000 L CNN
-F 2 "Package_TO_SOT_THT:TO-18-2_Window" H 6500 2475 50  0001 C CNN
-F 3 "http://www.osram-os.com/Graphics/XPic6/00029609_0.pdf/SFh%20460.pdf" H 6450 2300 50  0001 C CNN
-	1    6500 2300
-	0    -1   -1   0
-$EndComp
+	5950 3250 5950 3050
 Wire Wire Line
 	5600 2750 5600 2500
 Wire Wire Line
-	6500 2750 6500 2500
+	5950 2750 5950 2500
 $Comp
 L power:+5V #PWR?
@@
 L power:+5V #PWR?
 U 1 1 5B7F6CC2
-P 6500 1850
-F 0 "#PWR?" H 6500 1700 50  0001 C CNN
-F 1 "+5V" H 6515 2023 50  0000 C CNN
-F 2 "" H 6500 1850 50  0001 C CNN
-F 3 "" H 6500 1850 50  0001 C CNN
-	1    6500 1850
+P 5950 1850
+F 0 "#PWR?" H 5950 1700 50  0001 C CNN
+F 1 "+5V" H 5965 2023 50  0000 C CNN
+F 2 "" H 5950 1850 50  0001 C CNN
+F 3 "" H 5950 1850 50  0001 C CNN
+	1    5950 1850
 	1    0    0    -1
 $EndComp
@@
 	5600 2200 5600 1850
 Wire Wire Line
-	6500 2200 6500 1850
+	5950 2200 5950 1850
 $Comp
 L Connector:Conn_01x08_Male J?
 U 1 1 5B875270
-P 5050 1550
-F 0 "J?" H 5156 2028 50  0000 C CNN
-F 1 "Conn_01x08_Male" H 5156 1937 50  0000 C CNN
-F 2 "" H 5050 1550 50  0001 C CNN
-F 3 "~" H 5050 1550 50  0001 C CNN
-	1    5050 1550
+P 5250 1550
+F 0 "J?" H 5400 2050 50  0000 C CNN
+F 1 "8_Pin" H 5350 1950 50  0000 C CNN
+F 2 "" H 5250 1550 50  0001 C CNN
+F 3 "~" H 5250 1550 50  0001 C CNN
+	1    5250 1550
 	-1   0    0    1
 $EndComp
@@
 	3250 3900 3450 3900
 Wire Wire Line
-	4850 1650 4650 1650
-Wire Wire Line
-	4850 1750 4650 1750
-Wire Wire Line
 	4350 2250 4250 2250
 $Comp
-L Device:R R?
+L Device:R R100
 U 1 1 5B87B2E1
 P 4500 1750
-F 0 "R?" V 4293 1750 50  0000 C CNN
-F 1 "R" V 4384 1750 50  0000 C CNN
+F 0 "R100" V 4600 1750 50  0000 C CNN
+F 1 "R3" V 4700 1750 50  0000 C CNN
 F 2 "" V 4430 1750 50  0001 C CNN
 F 3 "~" H 4500 1750 50  0001 C CNN
@@
 $EndComp
 $Comp
-L Device:R R?
+L Device:R R100
 U 1 1 5B87B57E
 P 4500 1650
-F 0 "R?" V 4293 1650 50  0000 C CNN
-F 1 "R" V 4384 1650 50  0000 C CNN
+F 0 "R100" V 4293 1650 50  0000 C CNN
+F 1 "R4" V 4384 1650 50  0000 C CNN
 F 2 "" V 4430 1650 50  0001 C CNN
 F 3 "~" H 4500 1650 50  0001 C CNN
@@
 	4350 1650 4250 1650
 Wire Wire Line
-	4650 2550 4650 2500
-Wire Wire Line
-	4250 2550 4650 2550
-Wire Wire Line
-	4650 2200 4650 1850
-Wire Wire Line
-	4650 1850 4850 1850
-Wire Wire Line
-	4350 1750 4350 2250
+	4800 2550 4800 2500
+Wire Wire Line
+	4800 2200 4800 1850
 Wire Wire Line
 	4250 1650 4250 2150
@@
 NoConn ~ 4250 3450
 NoConn ~ 4250 3550
+Wire Wire Line
+	3650 3900 3950 3900
+Wire Wire Line
+	3950 4050 3950 3900
+Wire Wire Line
+	2350 3750 2350 3550
+$Comp
+L Device:LED TX
+U 1 1 5B9A0C7A
+P 5950 2350
+F 0 "TX" V 5988 2233 50  0000 R CNN
+F 1 "Green" V 5897 2233 50  0000 R CNN
+F 2 "" H 5950 2350 50  0001 C CNN
+F 3 "~" H 5950 2350 50  0001 C CNN
+	1    5950 2350
+	0    -1   -1   0
+$EndComp
+$Comp
+L Device:LED RX
+U 1 1 5B9A36D9
+P 5600 2350
+F 0 "RX" V 5650 2250 50  0000 R CNN
+F 1 "Blue" V 5550 2250 50  0000 R CNN
+F 2 "" H 5600 2350 50  0001 C CNN
+F 3 "~" H 5600 2350 50  0001 C CNN
+	1    5600 2350
+	0    -1   -1   0
+$EndComp
+Wire Wire Line
+	1650 2850 1650 2900
+Wire Wire Line
+	1650 2900 1750 2900
+Connection ~ 1750 2900
+Wire Wire Line
+	3350 1800 3550 1800
+Wire Wire Line
+	3550 1800 3550 1850
+Connection ~ 3350 1800
+Wire Wire Line
+	3350 1800 3350 1700
+Wire Wire Line
+	3350 1850 3350 1800
+$Comp
+L power:+5V #PWR?
+U 1 1 5BA3C5A4
+P 4850 1100
+F 0 "#PWR?" H 4850 950 50  0001 C CNN
+F 1 "+5V" H 4865 1273 50  0000 C CNN
+F 2 "" H 4850 1100 50  0001 C CNN
+F 3 "" H 4850 1100 50  0001 C CNN
+	1    4850 1100
+	1    0    0    -1
+$EndComp
+Wire Wire Line
+	4850 1150 4850 1100
+$Comp
+L power:GNDREF #PWR?
+U 1 1 5BA3ECA2
+P 4850 1300
+F 0 "#PWR?" H 4850 1050 50  0001 C CNN
+F 1 "GNDREF" H 4855 1127 50  0000 C CNN
+F 2 "" H 4850 1300 50  0001 C CNN
+F 3 "" H 4850 1300 50  0001 C CNN
+	1    4850 1300
+	1    0    0    -1
+$EndComp
+Wire Wire Line
+	5050 1250 4850 1250
+Wire Wire Line
+	4850 1250 4850 1300
+Wire Wire Line
+	4850 1150 5050 1150
+$Comp
+L power:+5V #PWR?
+U 1 1 5BA44B93
+P 2400 2000
+F 0 "#PWR?" H 2400 1850 50  0001 C CNN
+F 1 "+5V" H 2415 2173 50  0000 C CNN
+F 2 "" H 2400 2000 50  0001 C CNN
+F 3 "" H 2400 2000 50  0001 C CNN
+	1    2400 2000
+	1    0    0    -1
+$EndComp
+Wire Wire Line
+	2400 2000 2400 2250
+NoConn ~ 5050 1350
+NoConn ~ 5050 1450
+NoConn ~ 5050 1550
+Wire Wire Line
+	4250 2550 4800 2550
+Wire Wire Line
+	4350 1750 4350 2250
+Wire Wire Line
+	4800 1850 5050 1850
+Wire Wire Line
+	4650 1750 5050 1750
+Wire Wire Line
+	4650 1650 5050 1650
+Wire Wire Line
+	4250 3250 5950 3250
 $EndSCHEMATC

Commit message: 0.0.2 Picked Part
Parts:
- C1: footprint (none) -> Capacitor_SMD:C_0603_1608Metric
- F1: footprint (none) -> Fuse:Fuse_0402_1005Metric
- J1: renamed from J?; footprint (none) -> Connector_USB:USB_Micro-B_Amphenol_10103594-0001LF_Horizontal
- J2: renamed from J?; value 8_Pin -> Jumper_For_RJ45; footprint (none) -> Connector_PinHeader_1.27mm:PinHeader_1x08_P1.27mm_Vertical
- R1, R2: footprint (none) -> Resistor_SMD:R_0402_1005Metric
- R3: renamed from R100; value R3 -> 100; footprint (none) -> Resistor_SMD:R_0402_1005Metric
- R4: renamed from R100; value R4 -> 100; footprint (none) -> Resistor_SMD:R_0402_1005Metric
- RX1: renamed from RX; footprint (none) -> LED_SMD:LED_0603_1608Metric
- TX1: renamed from TX; footprint (none) -> LED_SMD:LED_0603_1608Metric
Other:
- note removed: "RESET"
Changed lines of the file:
@@
 EELAYER 26 0
 EELAYER END
-$Descr A4 11693 8268
+$Descr B 17000 11000
 encoding utf-8
 Sheet 1 1
-Title ""
-Date ""
-Rev ""
-Comp ""
-Comment1 ""
-Comment2 ""
-Comment3 ""
-Comment4 ""
+Title "Programmer Board"
+Date "2018-09-19"
+Rev "0.0.2"
+Comp "Missouri University of Science and Techology - Underwater Robotics"
+Comment1 "This board is the programmer for Titan Modules"
+Comment2 "https://github.com/MST-Robotics/TITAN-Electrical.git"
+Comment3 "programmer"
+Comment4 "NOTICE: The Missouri S&T Underwater Robotics Team makes no claim to the accuracy or usability of this document. Email mstrobotics@mst.edu for more information. Printed copies are not maintained."
 $EndDescr
 $Comp
@@
 $EndComp
 $Comp
-L Connector:USB_B_Micro J?
+L Connector:USB_B_Micro J1
 U 1 1 5B7F2F5E
 P 1750 2450
-F 0 "J?" H 1805 2917 50  0000 C CNN
+F 0 "J1" H 1805 2917 50  0000 C CNN
 F 1 "USB_B_Micro" H 1805 2826 50  0000 C CNN
-F 2 "" H 1900 2400 50  0001 C CNN
+F 2 "Connector_USB:USB_Micro-B_Amphenol_10103594-0001LF_Horizontal" H 1900 2400 50  0001 C CNN
 F 3 "~" H 1900 2400 50  0001 C CNN
 	1    1750 2450
@@
 F 0 "F1" V 2053 2250 50  0000 C CNN
 F 1 "500mA" V 2144 2250 50  0000 C CNN
-F 2 "" V 2180 2250 50  0001 C CNN
+F 2 "Fuse:Fuse_0402_1005Metric" V 2180 2250 50  0001 C CNN
 F 3 "~" H 2250 2250 50  0001 C CNN
 	1    2250 2250
@@
 	2050 2250 2100 2250
 $Comp
-L power:Earth #PWR?
+L power:Earth #PWR0101
 U 1 1 5B7F3E74
 P 1900 2900
-F 0 "#PWR?" H 1900 2650 50  0001 C CNN
+F 0 "#PWR0101" H 1900 2650 50  0001 C CNN
 F 1 "Earth" H 1900 2750 50  0001 C CNN
 F 2 "" H 1900 2900 50  0001 C CNN
@@
 	1750 2900 1900 2900
 $Comp
-L power:Earth #PWR?
+L power:Earth #PWR0102
 U 1 1 5B7F436B
 P 3950 4050
-F 0 "#PWR?" H 3950 3800 50  0001 C CNN
+F 0 "#PWR0102" H 3950 3800 50  0001 C CNN
 F 1 "Earth" H 3950 3900 50  0001 C CNN
 F 2 "" H 3950 4050 50  0001 C CNN
@@
 Connection ~ 3650 3900
 $Comp
-L power:Earth #PWR?
+L power:Earth #PWR0103
 U 1 1 5B7F45BE
 P 2350 3750
-F 0 "#PWR?" H 2350 3500 50  0001 C CNN
+F 0 "#PWR0103" H 2350 3500 50  0001 C CNN
 F 1 "Earth" H 2350 3600 50  0001 C CNN
 F 2 "" H 2350 3750 50  0001 C CNN
@@
 	2650 3550 2350 3550
 $Comp
-L power:+5V #PWR?
+L power:+5V #PWR0104
 U 1 1 5B7F5369
 P 3350 1700
-F 0 "#PWR?" H 3350 1550 50  0001 C CNN
+F 0 "#PWR0104" H 3350 1550 50  0001 C CNN
 F 1 "+5V" H 3365 1873 50  0000 C CNN
 F 2 "" H 3350 1700 50  0001 C CNN
@@
 F 0 "C1" V 4548 2350 50  0000 C CNN
 F 1 "100nF" V 4639 2350 50  0000 C CNN
-F 2 "" H 4838 2200 50  0001 C CNN
+F 2 "Capacitor_SMD:C_0603_1608Metric" H 4838 2200 50  0001 C CNN
 F 3 "~" H 4800 2350 50  0001 C CNN
 	1    4800 2350
 	1    0    0    -1
 $EndComp
-Text Notes 4800 2300 1    50   ~ 0
-RESET
 $Comp
 L Device:R R1
@@
 F 0 "R1" H 5670 2946 50  0000 L CNN
 F 1 "1K" H 5670 2855 50  0000 L CNN
-F 2 "" V 5530 2900 50  0001 C CNN
+F 2 "Resistor_SMD:R_0402_1005Metric" V 5530 2900 50  0001 C CNN
 F 3 "~" H 5600 2900 50  0001 C CNN
 	1    5600 2900
@@
 F 0 "R2" H 6020 2946 50  0000 L CNN
 F 1 "1K" H 6020 2855 50  0000 L CNN
-F 2 "" V 5880 2900 50  0001 C CNN
+F 2 "Resistor_SMD:R_0402_1005Metric" V 5880 2900 50  0001 C CNN
 F 3 "~" H 5950 2900 50  0001 C CNN
 	1    5950 2900
@@
 	5950 2750 5950 2500
 $Comp
-L power:+5V #PWR?
+L power:+5V #PWR0105
 U 1 1 5B7F6C85
 P 5600 1850
-F 0 "#PWR?" H 5600 1700 50  0001 C CNN
+F 0 "#PWR0105" H 5600 1700 50  0001 C CNN
 F 1 "+5V" H 5615 2023 50  0000 C CNN
 F 2 "" H 5600 1850 50  0001 C CNN
@@
 $EndComp
 $Comp
-L power:+5V #PWR?
+L power:+5V #PWR0106
 U 1 1 5B7F6CC2
 P 5950 1850
-F 0 "#PWR?" H 5950 1700 50  0001 C CNN
+F 0 "#PWR0106" H 5950 1700 50  0001 C CNN
 F 1 "+5V" H 5965 2023 50  0000 C CNN
 F 2 "" H 5950 1850 50  0001 C CNN
@@
 	5950 2200 5950 1850
 $Comp
-L Connector:Conn_01x08_Male J?
+L Connector:Conn_01x08_Male J2
 U 1 1 5B875270
 P 5250 1550
-F 0 "J?" H 5400 2050 50  0000 C CNN
-F 1 "8_Pin" H 5350 1950 50  0000 C CNN
-F 2 "" H 5250 1550 50  0001 C CNN
+F 0 "J2" H 5400 2050 50  0000 C CNN
+F 1 "Jumper_For_RJ45" H 5350 1950 50  0000 C CNN
+F 2 "Connector_PinHeader_1.27mm:PinHeader_1x08_P1.27mm_Vertical" H 5250 1550 50  0001 C CNN
 F 3 "~" H 5250 1550 50  0001 C CNN
 	1    5250 1550
@@
 	4350 2250 4250 2250
 $Comp
-L Device:R R100
+L Device:R R3
 U 1 1 5B87B2E1
 P 4500 1750
-F 0 "R100" V 4600 1750 50  0000 C CNN
-F 1 "R3" V 4700 1750 50  0000 C CNN
-F 2 "" V 4430 1750 50  0001 C CNN
+F 0 "R3" V 4600 1750 50  0000 C CNN
+F 1 "100" V 4700 1750 50  0000 C CNN
+F 2 "Resistor_SMD:R_0402_1005Metric" V 4430 1750 50  0001 C CNN
 F 3 "~" H 4500 1750 50  0001 C CNN
 	1    4500 1750
@@
 $EndComp
 $Comp
-L Device:R R100
+L Device:R R4
 U 1 1 5B87B57E
 P 4500 1650
-F 0 "R100" V 4293 1650 50  0000 C CNN
-F 1 "R4" V 4384 1650 50  0000 C CNN
-F 2 "" V 4430 1650 50  0001 C CNN
+F 0 "R4" V 4293 1650 50  0000 C CNN
+F 1 "100" V 4384 1650 50  0000 C CNN
+F 2 "Resistor_SMD:R_0402_1005Metric" V 4430 1650 50  0001 C CNN
 F 3 "~" H 4500 1650 50  0001 C CNN
 	1    4500 1650
@@
 	2350 3750 2350 3550
 $Comp
-L Device:LED TX
+L Device:LED TX1
 U 1 1 5B9A0C7A
 P 5950 2350
-F 0 "TX" V 5988 2233 50  0000 R CNN
+F 0 "TX1" V 5988 2233 50  0000 R CNN
 F 1 "Green" V 5897 2233 50  0000 R CNN
-F 2 "" H 5950 2350 50  0001 C CNN
+F 2 "LED_SMD:LED_0603_1608Metric" H 5950 2350 50  0001 C CNN
 F 3 "~" H 5950 2350 50  0001 C CNN
 	1    5950 2350
@@
 $EndComp
 $Comp
-L Device:LED RX
+L Device:LED RX1
 U 1 1 5B9A36D9
 P 5600 2350
-F 0 "RX" V 5650 2250 50  0000 R CNN
+F 0 "RX1" V 5650 2250 50  0000 R CNN
 F 1 "Blue" V 5550 2250 50  0000 R CNN
-F 2 "" H 5600 2350 50  0001 C CNN
+F 2 "LED_SMD:LED_0603_1608Metric" H 5600 2350 50  0001 C CNN
 F 3 "~" H 5600 2350 50  0001 C CNN
 	1    5600 2350
@@
 	3350 1850 3350 1800
 $Comp
-L power:+5V #PWR?
+L power:+5V #PWR0107
 U 1 1 5BA3C5A4
 P 4850 1100
-F 0 "#PWR?" H 4850 950 50  0001 C CNN
+F 0 "#PWR0107" H 4850 950 50  0001 C CNN
 F 1 "+5V" H 4865 1273 50  0000 C CNN
 F 2 "" H 4850 1100 50  0001 C CNN
@@
 	4850 1150 4850 1100
 $Comp
-L power:GNDREF #PWR?
+L power:GNDREF #PWR0108
 U 1 1 5BA3ECA2
 P 4850 1300
-F 0 "#PWR?" H 4850 1050 50  0001 C CNN
+F 0 "#PWR0108" H 4850 1050 50  0001 C CNN
 F 1 "GNDREF" H 4855 1127 50  0000 C CNN
 F 2 "" H 4850 1300 50  0001 C CNN
@@
 	4850 1150 5050 1150
 $Comp
-L power:+5V #PWR?
+L power:+5V #PWR0109
 U 1 1 5BA44B93
 P 2400 2000
-F 0 "#PWR?" H 2400 1850 50  0001 C CNN
+F 0 "#PWR0109" H 2400 1850 50  0001 C CNN
 F 1 "+5V" H 2415 2173 50  0000 C CNN
 F 2 "" H 2400 2000 50  0001 C CNN

Commit message: Finished Rev 0.0.2
Parts:
- F1: value 500mA -> 2A
Connections:
- net labels removed: Earth
Other:
- note added: "PROGRAMMER BOARD"
- moved on the sheet: C1, F1, IC1, J1, J2, R1, R2, R3, R4, RX1, TX1

Commit message: Updated resistor sizes
Parts:
- F1: footprint Fuse:Fuse_0402_1005Metric -> Fuse:Fuse_1210_3225Metric
- R1, R2, R3, R4: footprint Resistor_SMD:R_0402_1005Metric -> Resistor_SMD:R_0603_1608Metric
Changed lines of the file:
@@
 Title "Programmer Board"
 Date "2018-10-10"
-Rev "0.0.2"
+Rev "1.0.0"
 Comp "Missouri University of Science and Techology - Underwater Robotics"
 Comment1 "This board is the programmer for Titan Modules"
@@
 F 0 "F1" V 4503 2900 50  0000 C CNN
 F 1 "2A" V 4594 2900 50  0000 C CNN
-F 2 "Fuse:Fuse_0402_1005Metric" V 4630 2900 50  0001 C CNN
+F 2 "Fuse:Fuse_1210_3225Metric" V 4630 2900 50  0001 C CNN
 F 3 "~" H 4700 2900 50  0001 C CNN
 	1    4700 2900
@@
 F 0 "R1" H 8120 3596 50  0000 L CNN
 F 1 "1K" V 8050 3500 50  0000 L CNN
-F 2 "Resistor_SMD:R_0402_1005Metric" V 7980 3550 50  0001 C CNN
+F 2 "Resistor_SMD:R_0603_1608Metric" V 7980 3550 50  0001 C CNN
 F 3 "~" H 8050 3550 50  0001 C CNN
 	1    8050 3550
@@
 F 0 "R2" H 8470 3596 50  0000 L CNN
 F 1 "1K" V 8400 3500 50  0000 L CNN
-F 2 "Resistor_SMD:R_0402_1005Metric" V 8330 3550 50  0001 C CNN
+F 2 "Resistor_SMD:R_0603_1608Metric" V 8330 3550 50  0001 C CNN
 F 3 "~" H 8400 3550 50  0001 C CNN
 	1    8400 3550
@@
 F 0 "R3" V 7050 2400 50  0000 C CNN
 F 1 "100" V 6950 2400 50  0000 C CNN
-F 2 "Resistor_SMD:R_0402_1005Metric" V 6880 2400 50  0001 C CNN
+F 2 "Resistor_SMD:R_0603_1608Metric" V 6880 2400 50  0001 C CNN
 F 3 "~" H 6950 2400 50  0001 C CNN
 	1    6950 2400
@@
 F 0 "R4" V 6850 2300 50  0000 C CNN
 F 1 "100" V 6950 2300 50  0000 C CNN
-F 2 "Resistor_SMD:R_0402_1005Metric" V 6880 2300 50  0001 C CNN
+F 2 "Resistor_SMD:R_0603_1608Metric" V 6880 2300 50  0001 C CNN
 F 3 "~" H 6950 2300 50  0001 C CNN
 	1    6950 2300
@@
 PROGRAMMER BOARD
 $Comp
-L power:GNDREF #PWR?
+L power:GNDREF #PWR0101
 U 1 1 5BC8224C
 P 6400 4700
-F 0 "#PWR?" H 6400 4450 50  0001 C CNN
+F 0 "#PWR0101" H 6400 4450 50  0001 C CNN
 F 1 "GNDREF" H 6405 4527 50  0000 C CNN
 F 2 "" H 6400 4700 50  0001 C CNN
@@
 $EndComp
 $Comp
-L power:GNDREF #PWR?
+L power:GNDREF #PWR0102
 U 1 1 5BC832AD
 P 4800 4400
-F 0 "#PWR?" H 4800 4150 50  0001 C CNN
+F 0 "#PWR0102" H 4800 4150 50  0001 C CNN
 F 1 "GNDREF" H 4805 4227 50  0000 C CNN
 F 2 "" H 4800 4400 50  0001 C CNN
@@
 $EndComp
 $Comp
-L power:GNDREF #PWR?
+L power:GNDREF #PWR0103
 U 1 1 5BC83AD8
 P 4200 3650
-F 0 "#PWR?" H 4200 3400 50  0001 C CNN
+F 0 "#PWR0103" H 4200 3400 50  0001 C CNN
 F 1 "GNDREF" H 4205 3477 50  0000 C CNN
 F 2 "" H 4200 3650 50  0001 C CNN

Commit message: S1.0.1 B1.0.1
Schematic:
* Add filter cap for 5v
* slight layout changes
* change gndref symbols to gnd

Board:
* slight via rework
* reworked ground planes
* increased 5v trace size
* moved fuse
* moved title to top
* add header label
Parts:
- added C2: 100nF, Capacitor_SMD:C_0603_1608Metric, symbol Device:C
Connections:
- net labels added: GND
- net labels removed: GNDREF
- wire segments 45 -> 44
Other:
- note added: "RJ45 CONN"
- note added: "STAT LED"
- note added: "USB CONN"
- moved on the sheet: C1, F1, IC1, J1, J2, R1, R2, R3, R4, RX1, TX1
