File: power_board/power_board.sch (KiCad schematic (older format))
At the start: 62 parts, among them J1 Conn_01x02_Female, J10 Conn_01x01_Male, J11 Conn_01x01_Male, J12 Conn_01x01_Male, J13 Conn_01x04_Female, J2 Conn_01x02_Female, J3 Conn_01x02_Female, J4 Conn_01x02_Female, J5 Conn_01x02_Female, J6 Conn_01x01_Male, J7 Conn_01x01_Male, J8 Screw_Terminal_01x02, J9 Conn_01x01_Male, Q1 2N3904, Q2 2N3906, Q3 2N3904, SW1 SW_Push, U1 ACS758xCB-050B-PFF, U2 ACS758xCB-050B-PFF, U3 MCP2515-EST, U4 MAX31855KASA, U5 MCP2551-I-SN, U6 LM5166X, U7 ATmega328P-AU, Y1 16Mhz, Y2 16Mhz

Commit message: Redline updates
Parts:
- removed C11, C12: 560pF, Capacitor_SMD:C_0603_1608Metric, symbol Device:C
- removed Q1, Q3: 2N3904, Package_TO_SOT_SMD:SOT-23, symbol Transistor_BJT:2N3904
- removed R10, R11: 100, Resistor_SMD:R_0603_1608Metric, symbol Device:R_US
- removed R4, R6: 4.7k, Resistor_SMD:R_0603_1608Metric, symbol Device:R_US
- R12: value R_US -> 0
Connections:
- net labels removed: SYSTEM_STUTOFF
- wire segments 202 -> 186
Other:
- note added: "4 motors powered by +12v\n3 motors+rest of bot on +12va"
- note added: "Add reset pin\n"
- note added: "Add the 48v input isolation"
- note added: "Add the other digital pin connections"
- note added: "Find out how many leak sensors we want to suppot\nWhole robot or just power enclosure???\n"
- note added: "Find out if we want ESC interface here"
- note added: "Find out why the inductors are in ohms and not H"
- note added: "Power Regulation"
- note removed: "Outputs not in parallel!\n4 motors powered by +12v\n3 motors+rest of bot on +12va"
Changed lines of the file:
@@
 	3900 2850 4000 2850
-$Comp
-L Transistor_BJT:2N3904 Q3
-U 1 1 5BA45DF5
-P 4350 3500
-F 0 "Q3" H 4540 3546 50  0000 L CNN
-F 1 "2N3904" H 4540 3455 50  0000 L CNN
-F 2 "Package_TO_SOT_SMD:SOT-23" H 4550 3425 50  0001 L CIN
-F 3 "https://www.fairchildsemi.com/datasheets/2N/2N3904.pdf" H 4350 3500 50  0001 L CNN
-	1    4350 3500
-	-1   0    0    -1
-$EndComp
-$Comp
-L power:GNDREF #PWR0101
-U 1 1 5BA45E84
-P 4250 3900
-F 0 "#PWR0101" H 4250 3650 50  0001 C CNN
-F 1 "GNDREF" H 4255 3727 50  0000 C CNN
-F 2 "" H 4250 3900 50  0001 C CNN
-F 3 "" H 4250 3900 50  0001 C CNN
-	1    4250 3900
-	1    0    0    -1
-$EndComp
 $Comp
 L power:GNDREF #PWR0102
@@
 $EndComp
 Connection ~ 3500 2000
-Connection ~ 3900 2850
 $Comp
 L power:+48V #PWR0104
@@
 	1850 2900 1850 3000
 $Comp
-L Device:R_US R4
-U 1 1 5BA46B94
-P 3850 3750
-F 0 "R4" V 3645 3750 50  0000 C CNN
-F 1 "4.7k" V 3736 3750 50  0000 C CNN
-F 2 "Resistor_SMD:R_0603_1608Metric" V 3890 3740 50  0001 C CNN
-F 3 "~" H 3850 3750 50  0001 C CNN
-	1    3850 3750
-	-1   0    0    1
-$EndComp
-$Comp
 L power:+12V #PWR0108
 U 1 1 5BA47210
@@
 U 1 1 5BA477AD
 P 13900 6200
-F 0 "U7" H 13900 4614 50  0000 C CNN
-F 1 "ATmega328P-AU" H 13900 4523 50  0000 C CNN
+F 0 "U7" H 14050 4750 50  0000 C CNN
+F 1 "ATmega328P-AU" H 14300 4650 50  0000 C CNN
 F 2 "Package_QFP:TQFP-32_7x7mm_P0.8mm" H 13900 6200 50  0001 C CIN
 F 3 "http://ww1.microchip.com/downloads/en/DeviceDoc/ATmega328_P%20AVR%20MCU%20with%20picoPower%20Technology%20Data%20Sheet%2040001984A.pdf" H 13900 6200 50  0001 C CNN
@@
 P 13350 2500
 F 0 "R12" H 13418 2546 50  0000 L CNN
-F 1 "R_US" H 13418 2455 50  0000 L CNN
+F 1 "0" H 13418 2455 50  0000 L CNN
 F 2 "Resistor_SMD:R_0201_0603Metric" V 13390 2490 50  0001 C CNN
 F 3 "~" H 13350 2500 50  0001 C CNN
@@
 $EndComp
 Connection ~ 13000 1700
-Text Notes 3350 1350 0    100  ~ 0
-Outputs not in parallel!\n4 motors powered by +12v\n3 motors+rest of bot on +12va
+Text Notes 3500 1300 0    75   ~ 0
+4 motors powered by +12v\n3 motors+rest of bot on +12va
 $Comp
 L Transistor_BJT:2N3906 Q2
@@
 U 1 1 5BA74C01
 P 15050 5650
-F 0 "Y2" V 15096 5761 50  0000 L CNN
-F 1 "16Mhz" V 15005 5761 50  0000 L CNN
+F 0 "Y2" V 15350 5500 50  0000 L CNN
+F 1 "16Mhz" V 15250 5350 50  0000 L CNN
 F 2 "Crystal:Resonator_SMD-3Pin_7.2x3.0mm" H 15025 5650 50  0001 C CNN
 F 3 "~" H 15025 5650 50  0001 C CNN
@@
 	1    0    0    -1
 $EndComp
-Text GLabel 3850 4200 2    50   Input ~ 0
-LEAK_DETECTED
-Text GLabel 4700 3900 2    50   Input ~ 0
-SYSTEM_STUTOFF
-$Comp
-L Transistor_BJT:2N3904 Q1
-U 1 1 5BA8707F
-P 3650 3500
-F 0 "Q1" H 3840 3546 50  0000 L CNN
-F 1 "2N3904" H 3840 3455 50  0000 L CNN
-F 2 "Package_TO_SOT_SMD:SOT-23" H 3850 3425 50  0001 L CIN
-F 3 "https://www.fairchildsemi.com/datasheets/2N/2N3904.pdf" H 3650 3500 50  0001 L CNN
-	1    3650 3500
-	-1   0    0    -1
-$EndComp
-Wire Wire Line
-	3550 3300 3900 3300
-Wire Wire Line
-	3900 2850 3900 3300
-Connection ~ 3900 3300
-Wire Wire Line
-	3900 3300 4250 3300
-$Comp
-L Device:R_US R6
-U 1 1 5BA8C7E2
-P 4550 3750
-F 0 "R6" V 4345 3750 50  0000 C CNN
-F 1 "4.7k" V 4436 3750 50  0000 C CNN
-F 2 "Resistor_SMD:R_0603_1608Metric" V 4590 3740 50  0001 C CNN
-F 3 "~" H 4550 3750 50  0001 C CNN
-	1    4550 3750
-	-1   0    0    1
-$EndComp
-$Comp
-L power:GNDREF #PWR0126
-U 1 1 5BA8C8FE
-P 3550 3900
-F 0 "#PWR0126" H 3550 3650 50  0001 C CNN
-F 1 "GNDREF" H 3555 3727 50  0000 C CNN
-F 2 "" H 3550 3900 50  0001 C CNN
-F 3 "" H 3550 3900 50  0001 C CNN
-	1    3550 3900
-	1    0    0    -1
-$EndComp
-Wire Wire Line
-	4550 3600 4550 3500
-Wire Wire Line
-	4250 3700 4250 3900
-Wire Wire Line
-	3550 3700 3550 3900
-Wire Wire Line
-	3850 3500 3850 3600
-Wire Wire Line
-	4550 3900 4700 3900
-Wire Wire Line
-	3850 3900 3850 4200
 Text GLabel 14600 7400 2    50   Input ~ 0
 SYSTEM_SHUTOFF
@@
 U 1 1 5BA9F476
 P 10900 1750
-F 0 "J9" H 11006 1928 50  0000 C CNN
-F 1 "Conn_01x01_Male" H 11006 1837 50  0000 C CNN
+F 0 "J9" H 10900 1700 50  0000 C CNN
+F 1 "Conn_01x01_Male" H 11006 1837 50  0001 C CNN
 F 2 "Connector:Banana_Jack_1Pin" H 10900 1750 50  0001 C CNN
 F 3 "~" H 10900 1750 50  0001 C CNN
@@
 U 1 1 5BA9F662
 P 10900 2000
-F 0 "J10" H 11006 2178 50  0000 C CNN
-F 1 "Conn_01x01_Male" H 11006 2087 50  0000 C CNN
+F 0 "J10" H 10900 1950 50  0000 C CNN
+F 1 "Conn_01x01_Male" H 11006 2087 50  0001 C CNN
 F 2 "Connector:Banana_Jack_1Pin" H 10900 2000 50  0001 C CNN
 F 3 "~" H 10900 2000 50  0001 C CNN
@@
 U 1 1 5BA9F800
 P 10900 2950
-F 0 "J12" H 11006 3128 50  0000 C CNN
-F 1 "Conn_01x01_Male" H 11006 3037 50  0000 C CNN
+F 0 "J12" H 10900 2900 50  0000 C CNN
+F 1 "Conn_01x01_Male" H 11006 3037 50  0001 C CNN
 F 2 "Connector:Banana_Jack_1Pin" H 10900 2950 50  0001 C CNN
 F 3 "~" H 10900 2950 50  0001 C CNN
@@
 U 1 1 5BA75738
 P 7500 1700
-F 0 "U1" V 7454 1359 50  0000 R CNN
-F 1 "ACS758xCB-050B-PFF" V 7545 1359 50  0000 R CNN
+F 0 "U1" V 7450 1300 50  0000 R CNN
+F 1 "ACS758xCB-050B-PFF" V 7550 1300 50  0000 R CNN
 F 2 "Sensor_Current:Allegro_CB_PFF" H 7500 1700 50  0001 C CNN
 F 3 "http://www.allegromicro.com/~/media/Files/Datasheets/ACS758-Datasheet.ashx?la=en" H 7500 1700 50  0001 C CNN
@@
 U 1 1 5BA9F796
 P 10900 2750
-F 0 "J11" H 11006 2928 50  0000 C CNN
-F 1 "Conn_01x01_Male" H 11006 2837 50  0000 C CNN
+F 0 "J11" H 10900 2700 50  0000 C CNN
+F 1 "Conn_01x01_Male" H 11006 2837 50  0001 C CNN
 F 2 "Connector:Banana_Jack_1Pin" H 10900 2750 50  0001 C CNN
 F 3 "~" H 10900 2750 50  0001 C CNN
@@
 U 1 1 5BA93437
 P 7500 3050
-F 0 "U2" V 7454 2709 50  0000 R CNN
-F 1 "ACS758xCB-050B-PFF" V 7545 2709 50  0000 R CNN
+F 0 "U2" V 7450 2650 50  0000 R CNN
+F 1 "ACS758xCB-050B-PFF" V 7550 2650 50  0000 R CNN
 F 2 "Sensor_Current:Allegro_CB_PFF" H 7500 3050 50  0001 C CNN
 F 3 "http://www.allegromicro.com/~/media/Files/Datasheets/ACS758-Datasheet.ashx?la=en" H 7500 3050 50  0001 C CNN
@@
 U 1 1 5BA69BC1
 P 7600 8400
-F 0 "U3" H 7600 9378 50  0000 C CNN
-F 1 "MCP2515-EST" H 7600 9287 50  0000 C CNN
+F 0 "U3" H 7750 9350 50  0000 C CNN
+F 1 "MCP2515-EST" H 7950 9250 50  0000 C CNN
 F 2 "Package_SO:TSSOP-20_4.4x6.5mm_P0.65mm" H 7600 7500 50  0001 C CIN
 F 3 "http://ww1.microchip.com/downloads/en/DeviceDoc/21801e.pdf" H 7700 7600 50  0001 C CNN
@@
 U 1 1 5BA69EE0
 P 9850 8050
-F 0 "U5" H 9850 8628 50  0000 C CNN
-F 1 "MCP2551-I-SN" H 9850 8537 50  0000 C CNN
+F 0 "U5" H 9950 8650 50  0000 C CNN
+F 1 "MCP2551-I-SN" H 10200 8550 50  0000 C CNN
 F 2 "Package_SO:SOIC-8_3.9x4.9mm_P1.27mm" H 9850 7550 50  0001 C CIN
 F 3 "http://ww1.microchip.com/downloads/en/devicedoc/21667d.pdf" H 9850 8050 50  0001 C CNN
@@
 U 1 1 5BB39D19
 P 6600 8650
-F 0 "Y1" V 6554 8781 50  0000 L CNN
-F 1 "16Mhz" V 6645 8781 50  0000 L CNN
+F 0 "Y1" V 6300 8700 50  0000 L CNN
+F 1 "16Mhz" V 6400 8700 50  0000 L CNN
 F 2 "Crystal:Resonator_SMD-3Pin_7.2x3.0mm" H 6600 8650 50  0001 C CNN
 F 3 "~" H 6600 8650 50  0001 C CNN
@@
 U 1 1 5BB3A110
 P 6350 8800
-F 0 "C4" H 6465 8846 50  0000 L CNN
-F 1 "22pF" H 6465 8755 50  0000 L CNN
+F 0 "C4" H 6500 8750 50  0000 L CNN
+F 1 "22pF" H 6450 8850 50  0000 L CNN
 F 2 "Capacitor_SMD:C_0603_1608Metric" H 6388 8650 50  0001 C CNN
 F 3 "~" H 6350 8800 50  0001 C CNN
@@
 	9850 8450 9850 8600
 Connection ~ 9850 8600
-$Comp
-L Device:R_US R10
-U 1 1 5BB9B5D3
-P 10550 8300
-F 0 "R10" V 10755 8300 50  0000 C CNN
-F 1 "100" V 10664 8300 50  0000 C CNN
-F 2 "Resistor_SMD:R_0603_1608Metric" V 10590 8290 50  0001 C CNN
-F 3 "~" H 10550 8300 50  0001 C CNN
-	1    10550 8300
-	-1   0    0    1
-$EndComp
-$Comp
-L Device:R_US R11
-U 1 1 5BB9B67D
-P 10900 8300
-F 0 "R11" V 11105 8300 50  0000 C CNN
-F 1 "100" V 11014 8300 50  0000 C CNN
-F 2 "Resistor_SMD:R_0603_1608Metric" V 10940 8290 50  0001 C CNN
-F 3 "~" H 10900 8300 50  0001 C CNN
-	1    10900 8300
-	-1   0    0    1
-$EndComp
-$Comp
-L Device:C C11
-U 1 1 5BB9B889
-P 10550 8650
-F 0 "C11" H 10665 8696 50  0000 L CNN
-F 1 "560pF" H 10665 8605 50  0000 L CNN
-F 2 "Capacitor_SMD:C_0603_1608Metric" H 10588 8500 50  0001 C CNN
-F 3 "~" H 10550 8650 50  0001 C CNN
-	1    10550 8650
-	-1   0    0    1
-$EndComp
-$Comp
-L Device:C C12
-U 1 1 5BB9B993
-P 10900 8650
-F 0 "C12" H 11015 8696 50  0000 L CNN
-F 1 "560pF" H 11015 8605 50  0000 L CNN
-F 2 "Capacitor_SMD:C_0603_1608Metric" H 10938 8500 50  0001 C CNN
-F 3 "~" H 10900 8650 50  0001 C CNN
-	1    10900 8650
-	1    0    0    -1
-$EndComp
-Wire Wire Line
-	10350 8150 10550 8150
-Wire Wire Line
-	10550 8500 10550 8450
-Wire Wire Line
-	10550 8800 10750 8800
-Wire Wire Line
-	10900 8500 10900 8450
-Wire Wire Line
-	10900 8150 10900 7950
-Wire Wire Line
-	10900 7950 10350 7950
-$Comp
-L power:GNDREF #PWR0151
-U 1 1 5BBCB133
-P 10750 8800
-F 0 "#PWR0151" H 10750 8550 50  0001 C CNN
-F 1 "GNDREF" H 10755 8627 50  0000 C CNN
-F 2 "" H 10750 8800 50  0001 C CNN
-F 3 "" H 10750 8800 50  0001 C CNN
-	1    10750 8800
-	1    0    0    -1
-$EndComp
-Connection ~ 10750 8800
-Wire Wire Line
-	10750 8800 10900 8800
-Text GLabel 10950 7950 2    50   Input ~ 0
+Text GLabel 10600 7950 2    50   Input ~ 0
 CANH
-Wire Wire Line
-	10950 7950 10900 7950
-Connection ~ 10900 7950
 Text GLabel 10600 8150 2    50   Input ~ 0
 CANL
-Wire Wire Line
-	10550 8150 10600 8150
-Connection ~ 10550 8150
 Text GLabel 8250 8400 2    50   Input ~ 0
 CAN_INT
@@
 Text Notes 2550 9600 0    100  ~ 0
 REF: BlueRobotics\nLeak Sensor\n
+Text Notes 3850 950  0    100  ~ 0
+Power Regulation
+Text Notes 9700 1000 0    100  ~ 20
+Find out if we want ESC interface here
+Wire Wire Line
+	10350 8150 10600 8150
+Wire Wire Line
+	10350 7950 10600 7950
+Text Notes 6850 4450 0    100  ~ 20
+Find out why the inductors are in ohms and not H
+Text Notes 1500 7050 0    100  ~ 20
+Find out how many leak sensors we want to suppot\nWhole robot or just power enclosure???\n
+Text Notes 7400 9850 0    100  ~ 20
+Add the other digital pin connections
+Text Notes 3100 3750 0    100  ~ 20
+Add the 48v input isolation
+Text Notes 10350 6300 0    100  ~ 20
+Add reset pin\n
 $EndSCHEMATC

Commit message: Updates
Parts:
- removed J1, J2, J3: Conn_01x02_Female, Connector_JST:JST_GH_BM02B-GHS-TBT_1x02-1MP_P1.25mm_Vertical, symbol Connector:Conn_01x02_Female
- removed J10, J11, J12, J9: Conn_01x01_Male, Connector:Banana_Jack_1Pin, symbol Connector:Conn_01x01_Male
- removed J13: Conn_01x04_Female, Connector_PinHeader_2.54mm:PinHeader_1x04_P2.54mm_Horizontal, symbol Connector:Conn_01x04_Female
- added J?: M1, symbol Connector:Screw_Terminal_01x02
- added J?: M2, symbol Connector:Screw_Terminal_01x02
- added J?: M3, symbol Connector:Screw_Terminal_01x02
- added J?: M4, symbol Connector:Screw_Terminal_01x02
- added J?: M5, symbol Connector:Screw_Terminal_01x02
- added J?: M6, symbol Connector:Screw_Terminal_01x02
- added J?: M7, symbol Connector:Screw_Terminal_01x02
- added J?: FAN, symbol Connector:Screw_Terminal_01x02
- added J?: MainBoard, symbol Connector:Screw_Terminal_01x02
- added J?: PROG, symbol Connector:Conn_01x05_Female
- added Q? (x2): Q_NMOS_DGS, symbol Device:Q_NMOS_DGS
- added Q?: Q_NPN_BEC, symbol Device:Q_NPN_BEC
- added R? (x2): 10k, Resistor_SMD:R_0603_1608Metric, symbol Device:R_US
- added R? (x4): 1k, Resistor_SMD:R_0603_1608Metric, symbol Device:R_US
Connections:
- net labels added: +5VA, RX1BF, RX_INT, TX0RTS, TX1RTS, TX2RTS
- net labels removed: SYSTEM_SHUTOFF
- wire segments 186 -> 228
Other:
- note added: "A2"
- note added: "A3"
- note added: "A4"
- note added: "A5"
- note added: "D3"
- note added: "D5"
- note added: "D6"
- note added: "LEAK States\nDry - 5V\nWet - 0V\n"
- note added: "Leak Sensor Support"
- note added: "VERIFY PIN ORDER!!!\n\n"
- note added: "WARNING: +5VA will always be present \nwith voltage on tether. This reference is needed\nto be able to control shutoff mosfets.\n\n"
- note removed: "Add reset pin\n"
- note removed: "Add the 48v input isolation"
- note removed: "Add the other digital pin connections"
- note removed: "D7"
- note removed: "Find out how many leak sensors we want to suppot\nWhole robot or just power enclosure???\n"
- note removed: "Find out if we want ESC interface here"
- note removed: "Leak Sensor Inputs"
- note removed: "Leak Sensor Support\nCutoff States:\n *0 - DRY\n *1 - WET"
- note removed: "REF: BlueRobotics\nLeak Sensor\n"
- moved on the sheet: U1, U2, U6

Commit message: finishing touches
Parts:
- removed C6: 10nF, Capacitor_SMD:C_0603_1608Metric, symbol Device:C
- removed L1, L2: 470ohm, Inductor_SMD:L_0603_1608Metric, symbol pspice:INDUCTOR
- removed Q2: 2N3906, Package_TO_SOT_SMD:SOT-23, symbol Transistor_BJT:2N3906
- removed Q?: Q_NPN_BEC, symbol Device:Q_NPN_BEC
- removed R2, R5, R? (x2): 1k, Resistor_SMD:R_0603_1608Metric, symbol Device:R_US
- removed R3: 27k, Resistor_SMD:R_0603_1608Metric, symbol Device:R_US
- added Q3, Q4: Q_NMOS_DGS, Package_TO_SOT_SMD:TO-263-2, symbol Device:Q_NMOS_DGS
- J1: renamed from J?; footprint (none) -> Connector_PinHeader_2.54mm:PinHeader_1x05_P2.54mm_Vertical
- J10, J11, J12, J13, J14, J15, J2, J3, J9: renamed from J?; footprint (none) -> TerminalBlock:TerminalBlock_bornier-2_P5.08mm
- Q1, Q2: renamed from Q?; footprint (none) -> Package_TO_SOT_SMD:TO-263-2
- R4: renamed from R?; value 1k -> 10k
- R5: renamed from R?; value 1k -> 1.1k
- gave numbers to parts that had none: 2
Connections:
- net labels removed: PROBE
- wire segments 228 -> 223
Other:
- note added: "Leak Sensor Input"
- note added: "Power Shutoff Bias"
- note added: "Power is cut when LEAK_DETECTED is pulled low \nincating a leak."
- note added: "SWAP CAN TRANSCIEVER\n\n"
- note added: "WARNING: +5VA will always \nbe present."
- note removed: "Find out why the inductors are in ohms and not H"
- note removed: "LEAK States\nDry - 5V\nWet - 0V\n"
- note removed: "Leak Sensor Support"
- note removed: "WARNING: +5VA will always be present \nwith voltage on tether. This reference is needed\nto be able to control shutoff mosfets.\n\n"

Commit message: Finished adding power regulator isolation
Parts:
- removed Q1, Q2, Q3, Q4: Q_NMOS_DGS, Package_TO_SOT_SMD:TO-263-2, symbol Device:Q_NMOS_DGS
- removed R12: 0, Resistor_SMD:R_0201_0603Metric, symbol Device:R_US
- removed R13: 0.5, Resistor_SMD:R_0201_0603Metric, symbol Device:R_US
- removed U6: LM5166X, Package_SON:Texas_S-PVSON-N10_ThermalVias, symbol Regulator_Switching:LM5166X
- added D3: --, Diode_SMD:D_0603_1608Metric, symbol Device:D_Schottky
- added J16: Screw_Terminal_01x02, TerminalBlock:TerminalBlock_bornier-2_P5.08mm, symbol Connector:Screw_Terminal_01x02
- added Q1: 2N3906, Package_TO_SOT_SMD:SOT-23, symbol Device:Q_PNP_BCE
- added R6: 10k, Resistor_SMD:R_0603_1608Metric, symbol Device:R_US
- added U6, U8: BTS6163D, Package_TO_SOT_SMD:TO-252-4, symbol Power_Management:BTS6163D
- added U9: LM2596S-5, Package_TO_SOT_SMD:TO-263-5_TabPin3, symbol Regulator_Switching:LM2596S-5
- C1, C2: value CP -> 300uF
- C14: value 2.2uF -> 680uF; footprint Capacitor_SMD:C_0603_1608Metric -> Capacitor_THT:CP_Radial_D7.5mm_P2.50mm
- C15: value 47uF -> 220uF; footprint Capacitor_SMD:C_0805_2012Metric -> Capacitor_THT:CP_Radial_D5.0mm_P2.50mm
- D2: value D_Schottky -> 1N5824
- L3: value 150uH -> 33uH; footprint Inductor_SMD:L_0805_2012Metric -> Inductor_SMD:L_Bourns_SRP1245A
- R14: footprint Resistor_SMD:R_0201_0603Metric -> Resistor_SMD:R_0603_1608Metric
- R2: value 10k -> 1k
Connections:
- net labels added: SHUTOFF
- net labels removed: LEAK_DETECTED
- wire segments 223 -> 224
- no-connect marks 0 -> 14
Other:
- note added: "5V, 3A Max"
- note added: "BTS6163D is a high side load driver. 60V, 21.5A Max\nShould disspiate < 20W of power each. (Ids^2*Ron)\n"
- note added: "Leak Sensor Support"
- note added: "Power is cut when a short is present \non J4 or J5 incating a leak."
- note added: "WARNING: +5VA will always be present."
- note removed: "5V, 500mA Max"
- note removed: "Leak Sensor Input"
- note removed: "Power is cut when LEAK_DETECTED is pulled low \nincating a leak."
- note removed: "WARNING: +5VA will always \nbe present."

Commit message: PCB Layout work
Parts:
- added J17: MB_interface, Connector_PinHeader_2.54mm:PinHeader_1x04_P2.54mm_Vertical, symbol Connector:Conn_01x04_Female
- added J19: 12V_1, TerminalBlock:TerminalBlock_bornier-2_P5.08mm, symbol Connector:Screw_Terminal_01x02
- added J20: 12V_2, TerminalBlock:TerminalBlock_bornier-2_P5.08mm, symbol Connector:Screw_Terminal_01x02
- added J21: 12V_3, TerminalBlock:TerminalBlock_bornier-2_P5.08mm, symbol Connector:Screw_Terminal_01x02
- added J22: 12V_4, TerminalBlock:TerminalBlock_bornier-2_P5.08mm, symbol Connector:Screw_Terminal_01x02
- added J23: 48V_1, TerminalBlock:TerminalBlock_bornier-2_P5.08mm, symbol Connector:Screw_Terminal_01x02
- added J24: 48V_2, TerminalBlock:TerminalBlock_bornier-2_P5.08mm, symbol Connector:Screw_Terminal_01x02
- added J25: 48V_3, TerminalBlock:TerminalBlock_bornier-2_P5.08mm, symbol Connector:Screw_Terminal_01x02
- added J26: 48V_4, TerminalBlock:TerminalBlock_bornier-2_P5.08mm, symbol Connector:Screw_Terminal_01x02
- J11: value MainBoard -> 5V_1
- Y1: value 16Mhz -> 20Mhz
Connections:
- net labels added: 48V
- wire segments 224 -> 263
Other:
- note added: "Main Board \nInterface\n\n"

Commit message: HIgh power routing work
Parts:
- removed U6, U8: BTS6163D, Package_TO_SOT_SMD:TO-252-4, symbol Power_Management:BTS6163D
- added U6, U8: BTS50085-1TMA, Package_TO_SOT_SMD:Infineon_PG-TO-220-7Lead_TabPin8, symbol Power_Management:BTS50085-1TMA
Connections:
- wire segments 263 -> 279
Other:
- note added: "BTS50085 is a high side load driver. 60V, 21.5A Max\nShould disspiate < 20W of power each. (Ids^2*Ron)\n"
- note removed: "BTS6163D is a high side load driver. 60V, 21.5A Max\nShould disspiate < 20W of power each. (Ids^2*Ron)\n"
Changed lines of the file:
@@
 L power:+48V #PWR0121
 U 1 1 5BAEA3D2
-P 2000 5350
-F 0 "#PWR0121" H 2000 5200 50  0001 C CNN
-F 1 "+48V" H 2015 5523 50  0000 C CNN
-F 2 "" H 2000 5350 50  0001 C CNN
-F 3 "" H 2000 5350 50  0001 C CNN
-	1    2000 5350
+P 2000 5300
+F 0 "#PWR0121" H 2000 5150 50  0001 C CNN
+F 1 "+48V" H 2015 5473 50  0000 C CNN
+F 2 "" H 2000 5300 50  0001 C CNN
+F 3 "" H 2000 5300 50  0001 C CNN
+	1    2000 5300
 	1    0    0    -1
 $EndComp
@@
 L power:+48V #PWR0126
 U 1 1 5BAEA445
-P 2000 4100
-F 0 "#PWR0126" H 2000 3950 50  0001 C CNN
-F 1 "+48V" H 2015 4273 50  0000 C CNN
-F 2 "" H 2000 4100 50  0001 C CNN
-F 3 "" H 2000 4100 50  0001 C CNN
-	1    2000 4100
+P 2000 4050
+F 0 "#PWR0126" H 2000 3900 50  0001 C CNN
+F 1 "+48V" H 2015 4223 50  0000 C CNN
+F 2 "" H 2000 4050 50  0001 C CNN
+F 3 "" H 2000 4050 50  0001 C CNN
+	1    2000 4050
 	1    0    0    -1
 $EndComp
@@
 Text GLabel 1500 4550 0    50   Input ~ 0
 SHUTOFF
-$Comp
-L Power_Management:BTS6163D U6
-U 1 1 5BB216EF
-P 2000 4550
-F 0 "U6" H 2000 4176 50  0000 C CNN
-F 1 "BTS6163D" H 2000 4085 50  0000 C CNN
-F 2 "Package_TO_SOT_SMD:TO-252-4" H 2000 4150 50  0001 C CNN
-F 3 "http://www.infineon.com/dgdl/Infineon-BTS6163D-DS-v01_00-EN.pdf?fileId=5546d4625a888733015aa3da01a1101e" H 2000 4150 50  0001 C CNN
-	1    2000 4550
-	1    0    0    -1
-$EndComp
-$Comp
-L Power_Management:BTS6163D U8
-U 1 1 5BB3D1D7
-P 2000 5800
-F 0 "U8" H 2000 5426 50  0000 C CNN
-F 1 "BTS6163D" H 2000 5335 50  0000 C CNN
-F 2 "Package_TO_SOT_SMD:TO-252-4" H 2000 5400 50  0001 C CNN
-F 3 "http://www.infineon.com/dgdl/Infineon-BTS6163D-DS-v01_00-EN.pdf?fileId=5546d4625a888733015aa3da01a1101e" H 2000 5400 50  0001 C CNN
-	1    2000 5800
-	1    0    0    -1
-$EndComp
 Wire Wire Line
 	2400 4450 2400 4500
@@
 Connection ~ 2600 4500
 Wire Wire Line
-	2600 4500 2400 4500
+	2600 4500 2450 4500
 Wire Wire Line
 	2600 4500 2900 4500
@@
 Connection ~ 2600 5750
 Wire Wire Line
-	2600 5750 2400 5750
+	2600 5750 2450 5750
 Wire Wire Line
 	2850 6050 2600 6050
@@
 Wire Wire Line
 	1500 5800 1600 5800
-Wire Wire Line
-	2000 5400 2000 5350
-Wire Wire Line
-	2000 4150 2000 4100
 Wire Notes Line width 10 style solid
 	1050 3300 4550 3300
@@
 	1550 8550 1800 8550
 Text Notes 1100 6750 0    75   ~ 0
-BTS6163D is a high side load driver. 60V, 21.5A Max\nShould disspiate < 20W of power each. (Ids^2*Ron)\n
+BTS50085 is a high side load driver. 60V, 21.5A Max\nShould disspiate < 20W of power each. (Ids^2*Ron)\n
 Wire Notes Line width 10 style solid
 	4550 6800 4550 3300
@@
 Wire Notes Line width 10 style solid
 	12150 4750 12150 6150
+$Comp
+L Power_Management:BTS50085-1TMA U8
+U 1 1 5BC0879A
+P 2000 5800
+F 0 "U8" H 2000 5426 50  0000 C CNN
+F 1 "BTS50085-1TMA" H 2000 5335 50  0000 C CNN
+F 2 "Package_TO_SOT_SMD:Infineon_PG-TO-220-7Lead_TabPin8" H 2000 5400 50  0001 C CNN
+F 3 "http://www.infineon.com/dgdl/Infineon-BTS50085-1TMA-DS-v01_00-EN.pdf?fileId=5546d4625a888733015aa435bccd114b" H 2000 5400 50  0001 C CNN
+	1    2000 5800
+	1    0    0    -1
+$EndComp
+Wire Wire Line
+	2400 5600 2450 5600
+Wire Wire Line
+	2450 5600 2450 5750
+Connection ~ 2450 5750
+Wire Wire Line
+	2450 5750 2400 5750
+Wire Wire Line
+	2400 5900 2450 5900
+Wire Wire Line
+	2450 5900 2450 5750
+Wire Wire Line
+	2000 5300 2000 5350
+Wire Wire Line
+	1900 5400 1900 5350
+Wire Wire Line
+	1900 5350 2000 5350
+Connection ~ 2000 5350
+Wire Wire Line
+	2000 5350 2000 5400
+$Comp
+L Power_Management:BTS50085-1TMA U6
+U 1 1 5BC5BD8A
+P 2000 4550
+F 0 "U6" H 2000 4176 50  0000 C CNN
+F 1 "BTS50085-1TMA" H 2000 4085 50  0000 C CNN
+F 2 "Package_TO_SOT_SMD:Infineon_PG-TO-220-7Lead_TabPin8" H 2000 4150 50  0001 C CNN
+F 3 "http://www.infineon.com/dgdl/Infineon-BTS50085-1TMA-DS-v01_00-EN.pdf?fileId=5546d4625a888733015aa435bccd114b" H 2000 4150 50  0001 C CNN
+	1    2000 4550
+	1    0    0    -1
+$EndComp
+Wire Wire Line
+	2400 4350 2450 4350
+Wire Wire Line
+	2450 4350 2450 4500
+Connection ~ 2450 4500
+Wire Wire Line
+	2450 4500 2400 4500
+Wire Wire Line
+	2400 4650 2450 4650
+Wire Wire Line
+	2450 4650 2450 4500
+Wire Wire Line
+	2000 4050 2000 4100
+Wire Wire Line
+	1900 4150 1900 4100
+Wire Wire Line
+	1900 4100 2000 4100
+Connection ~ 2000 4100
+Wire Wire Line
+	2000 4100 2000 4150
 $EndSCHEMATC
