File: power_board/power_board.sch (KiCad schematic (older format))
At the start: 66 parts, among them J1 PROG, J10 M4, J11 5V_1, J12 M5, J13 M6, J14 M7, J15 FAN, J16 Screw_Terminal_01x02, J17 MB_interface, J19 12V_1, J2 M1, J20 12V_2, J21 12V_3, J22 12V_4, J23 48V_1, J24 48V_2, J25 48V_3, J26 48V_4, J3 M2, J4 Conn_01x02_Female, J5 Conn_01x02_Female, J6 Conn_01x01_Male, J7 Conn_01x01_Male, J8 Screw_Terminal_01x02, J9 M3, Q1 2N3906, SW1 SW_Push, U1 ACS758xCB-050B-PFF, U2 ACS758xCB-050B-PFF, U3 MCP2515-EST, U4 MAX31855KASA, U5 MCP2551-I-SN, U6 BTS50085-1TMA, U7 ATmega328P-AU, U8 BTS50085-1TMA, U9 LM2596S-5, Y1 20Mhz, Y2 16Mhz

Commit message: Finished high power routing
Parts:
- added J18: Conn_01x02_Female, Connector_JST:JST_GH_BM02B-GHS-TBT_1x02-1MP_P1.25mm_Vertical, symbol Connector:Conn_01x02_Female
Connections:
- wire segments 279 -> 284
Changed lines of the file:
@@
 L Connector:Conn_01x02_Female J4
 U 1 1 5BA58C27
-P 1150 8250
-F 0 "J4" H 1050 8050 50  0000 C CNN
-F 1 "Conn_01x02_Female" H 1044 8016 50  0001 C CNN
-F 2 "Connector_JST:JST_GH_BM02B-GHS-TBT_1x02-1MP_P1.25mm_Vertical" H 1150 8250 50  0001 C CNN
-F 3 "~" H 1150 8250 50  0001 C CNN
-	1    1150 8250
+P 1150 8400
+F 0 "J4" H 1050 8200 50  0000 C CNN
+F 1 "Conn_01x02_Female" H 1044 8166 50  0001 C CNN
+F 2 "Connector_JST:JST_GH_BM02B-GHS-TBT_1x02-1MP_P1.25mm_Vertical" H 1150 8400 50  0001 C CNN
+F 3 "~" H 1150 8400 50  0001 C CNN
+	1    1150 8400
 	-1   0    0    1
 $EndComp
@@
 $EndComp
 Wire Wire Line
-	1350 8650 1450 8650
+	1350 8650 1400 8650
 Wire Wire Line
 	1450 8650 1450 8700
-Wire Wire Line
-	1350 8250 1450 8250
-Wire Wire Line
-	1450 8250 1450 8650
-Connection ~ 1450 8650
 Text Notes 1400 7800 0    100  ~ 0
 Leak Sensor Support
@@
 	1    0    0    -1
 $EndComp
-Wire Wire Line
-	1350 8150 1550 8150
-Wire Wire Line
-	1550 8150 1550 8550
-Wire Wire Line
-	1350 8550 1550 8550
-Connection ~ 1550 8550
 $Comp
 L power:+5VA #PWR0157
@@
 Wire Notes Line width 10 style solid
 	1050 6800 4550 6800
-Wire Wire Line
-	1550 8550 1800 8550
 Text Notes 1100 6750 0    75   ~ 0
 BTS50085 is a high side load driver. 60V, 21.5A Max\nShould disspiate < 20W of power each. (Ids^2*Ron)\n
@@
 Wire Wire Line
 	2000 4100 2000 4150
+Wire Wire Line
+	1350 8550 1500 8550
+$Comp
+L Connector:Conn_01x02_Female J18
+U 1 1 5BC10D2D
+P 1150 8150
+F 0 "J18" H 1050 7950 50  0000 C CNN
+F 1 "Conn_01x02_Female" H 1044 7916 50  0001 C CNN
+F 2 "Connector_JST:JST_GH_BM02B-GHS-TBT_1x02-1MP_P1.25mm_Vertical" H 1150 8150 50  0001 C CNN
+F 3 "~" H 1150 8150 50  0001 C CNN
+	1    1150 8150
+	-1   0    0    1
+$EndComp
+Wire Wire Line
+	1350 8300 1500 8300
+Wire Wire Line
+	1500 8300 1500 8550
+Connection ~ 1500 8550
+Wire Wire Line
+	1500 8550 1800 8550
+Wire Wire Line
+	1350 8050 1500 8050
+Wire Wire Line
+	1500 8050 1500 8300
+Connection ~ 1500 8300
+Wire Wire Line
+	1350 8150 1400 8150
+Wire Wire Line
+	1400 8150 1400 8400
+Connection ~ 1400 8650
+Wire Wire Line
+	1400 8650 1450 8650
+Wire Wire Line
+	1350 8400 1400 8400
+Connection ~ 1400 8400
+Wire Wire Line
+	1400 8400 1400 8650
 $EndSCHEMATC

Commit message: Current sensor routing/finishing touches
Changed lines of the file:
@@
 	1    0    0    -1
 $EndComp
+Text GLabel 10500 8950 0    50   Input ~ 0
+CANH
 Text GLabel 10500 8850 0    50   Input ~ 0
-CANH
-Text GLabel 10500 8950 0    50   Input ~ 0
 CANL
 $Comp
