File: main-board/_saved_main-board.sch (KiCad schematic (older format))
At the start: 26 parts

Commit message: add video, sans new balun
Parts:
- removed J?: Conn_01x04_Female, symbol Connector:Conn_01x04_Female
Changed lines of the file:
@@
-$EndComp
-$Comp
-L Connector:Conn_01x04_Female J?
-U 1 1 5BBE9559
-P 15550 8350
-F 0 "J?" H 15577 8326 50  0000 L CNN
-F 1 "Conn_01x04_Female" H 15577 8235 50  0000 L CNN
-F 2 "" H 15550 8350 50  0001 C CNN
-F 3 "~" H 15550 8350 50  0001 C CNN
-	1    15550 8350
-	1    0    0    -1
 $EndComp
 $Comp
@@
 Wire Wire Line
 	8500 6800 8700 6800
+Text GLabel 6300 1650 2    50   Input ~ 0
+VID00
+Text GLabel 6300 1750 2    50   Input ~ 0
+VID01
+Text GLabel 6300 1850 2    50   Input ~ 0
+VID02
+Text GLabel 6300 1950 2    50   Input ~ 0
+VID10
+Text GLabel 6300 2050 2    50   Input ~ 0
+VID11
+Text GLabel 6300 2150 2    50   Input ~ 0
+VID12
 $EndSCHEMATC
