File: main-board/main-board.sch (KiCad schematic (older format))
At the start: 26 parts

Commit message: add programming header
Parts:
- removed J?: Conn_01x04_Female, symbol Connector:Conn_01x04_Female
- added J?: PROGRAMMER, symbol Connector:Conn_01x05_Male
Connections:
- net labels added: +3V3, PROG-RX, PROG-TX, T0
- wire segments 26 -> 27
Changed lines of the file:
@@
-$EndComp
-$Comp
-L Connector:Conn_01x04_Female J?
-U 1 1 5BBE9559
-P 15550 8350
-F 0 "J?" H 15577 8326 50  0000 L CNN
-F 1 "Conn_01x04_Female" H 15577 8235 50  0000 L CNN
-F 2 "" H 15550 8350 50  0001 C CNN
-F 3 "~" H 15550 8350 50  0001 C CNN
-	1    15550 8350
-	1    0    0    -1
 $EndComp
 $Comp
@@
 Wire Wire Line
 	8500 6800 8700 6800
+Text GLabel 6300 1650 2    50   Input ~ 0
+VID00
+Text GLabel 6300 1750 2    50   Input ~ 0
+VID01
+Text GLabel 6300 1850 2    50   Input ~ 0
+VID02
+Text GLabel 6300 1950 2    50   Input ~ 0
+VID10
+Text GLabel 6300 2050 2    50   Input ~ 0
+VID11
+Text GLabel 6300 2150 2    50   Input ~ 0
+VID12
+Text GLabel 3500 1650 2    50   Input ~ 0
+M0
+Text GLabel 3500 1750 2    50   Input ~ 0
+M1
+Text GLabel 3500 1850 2    50   Input ~ 0
+M2
+Text GLabel 3500 1950 2    50   Input ~ 0
+M3
+Text GLabel 3500 2050 2    50   Input ~ 0
+M4
+Text GLabel 3500 2150 2    50   Input ~ 0
+M5
+Text GLabel 3500 2250 2    50   Input ~ 0
+M6
+Text GLabel 3500 2350 2    50   Input ~ 0
+M7
+Text GLabel 6300 3450 2    50   Input ~ 0
+T0
+Text GLabel 6300 3550 2    50   Input ~ 0
+T1
+Text GLabel 6300 3650 2    50   Input ~ 0
+T2
+Text GLabel 6300 3750 2    50   Input ~ 0
+T3
+Text GLabel 6300 3850 2    50   Input ~ 0
+T4
+Text GLabel 6300 3950 2    50   Input ~ 0
+T5
+Text GLabel 6300 4050 2    50   Input ~ 0
+T6
+Text GLabel 6300 4150 2    50   Input ~ 0
+T7
+$Comp
+L Connector:Conn_01x05_Male J?
+U 1 1 5BCA3C8B
+P 10750 8150
+F 0 "J?" H 10500 8250 50  0000 C CNN
+F 1 "PROGRAMMER" H 10450 8350 50  0000 C CNN
+F 2 "" H 10750 8150 50  0001 C CNN
+F 3 "~" H 10750 8150 50  0001 C CNN
+	1    10750 8150
+	1    0    0    -1
+$EndComp
+$Comp
+L power:GND #PWR?
+U 1 1 5BCA42E8
+P 10950 8350
+F 0 "#PWR?" H 10950 8100 50  0001 C CNN
+F 1 "GND" H 10955 8177 50  0000 C CNN
+F 2 "" H 10950 8350 50  0001 C CNN
+F 3 "" H 10950 8350 50  0001 C CNN
+	1    10950 8350
+	1    0    0    -1
+$EndComp
+$Comp
+L power:+5V #PWR?
+U 1 1 5BCA444A
+P 10950 7950
+F 0 "#PWR?" H 10950 7800 50  0001 C CNN
+F 1 "+5V" H 10965 8123 50  0000 C CNN
+F 2 "" H 10950 7950 50  0001 C CNN
+F 3 "" H 10950 7950 50  0001 C CNN
+	1    10950 7950
+	1    0    0    -1
+$EndComp
+$Comp
+L power:+3V3 #PWR?
+U 1 1 5BCA44F9
+P 11100 8050
+F 0 "#PWR?" H 11100 7900 50  0001 C CNN
+F 1 "+3V3" H 11115 8223 50  0000 C CNN
+F 2 "" H 11100 8050 50  0001 C CNN
+F 3 "" H 11100 8050 50  0001 C CNN
+	1    11100 8050
+	1    0    0    -1
+$EndComp
+Wire Wire Line
+	10950 8050 11100 8050
+Text GLabel 10950 8150 2    50   Input ~ 0
+PROG-TX
+Text GLabel 10950 8250 2    50   Input ~ 0
+PROG-RX
 $EndSCHEMATC

Commit message: add CAN
Parts:
- added C? (x2): 15p, symbol Device:C_Small
- added J?: PROGRAMMER, symbol Connector:Conn_01x05_Male
- added R? (x3): 10k, symbol Device:R_Small
- added U?: MCP2515-EST, Package_SO:TSSOP-20_4.4x6.5mm_P0.65mm, symbol Interface_CAN_LIN:MCP2515-EST
- added U?: ATA6560, symbol ATA6560:ATA6560
- added Y?: 20MHz, symbol Device:Crystal_Small
Connections:
- net labels added: CANH, CANL, INT, INTERCON0, INTERCON1, PROG0-RX, PROG0-TX, PROG1-RX, PROG1-TX, RX0, RX1, SCK, SI, SO, SS, TX0, TX1, TX2
- net labels removed: PROG-RX, PROG-TX, T8
- wire segments 27 -> 55
- no-connect marks 0 -> 1
Other:
- moved on the sheet: J?

Commit message: done sans power
Parts:
- removed J?: MOTOR0, symbol Connector:Conn_01x03_Male
- removed J?: MOTOR1, symbol Connector:Conn_01x03_Male
- removed J?: MOTOR2, symbol Connector:Conn_01x03_Male
- removed J?: MOTOR3, symbol Connector:Conn_01x03_Male
- removed J?: MOTOR5, symbol Connector:Conn_01x03_Male
- removed J?: MOTOR6, symbol Connector:Conn_01x03_Male
- removed J?: MOTOR7, symbol Connector:Conn_01x03_Male
- removed U? (x2): 2450BM08B0003T, symbol 2450BM08B0003T:2450BM08B0003T
- added J?: MOTOR5, symbol Connector:Conn_01x03_Male
- added J?: MOTOR6, symbol Connector:Conn_01x03_Male
- added J?: MOTOR7, symbol Connector:Conn_01x03_Male
- added J?: MOTOR0, symbol Connector:Conn_01x03_Male
- added J?: MOTOR1, symbol Connector:Conn_01x03_Male
- added J?: MOTOR2, symbol Connector:Conn_01x03_Male
- added J?: MOTOR3, symbol Connector:Conn_01x03_Male
- added T? (x2): ATB2012E-50011M-T01, XFMR_ATB2012E-50011M-T01, symbol ATB2012E-50011M-T01:ATB2012E-50011M-T01
- added U? (x2): OPAMP, symbol pspice:OPAMP
Connections:
- net labels added: CAN+, CAN-, RJ45+, RJ45-
- net labels removed: CANH, CANL
- wire segments 55 -> 56

Commit message: ready for review
Parts:
- removed J?: CAM4, symbol Connector:Conn_01x02_Male
- removed J?: CAM5, symbol Connector:Conn_01x02_Male
- removed J?: CAM6, symbol Connector:Conn_01x02_Male
- removed J?: CAM7, symbol Connector:Conn_01x02_Male
- removed J?: CAM0, symbol Connector:Conn_01x02_Male
- removed J?: CAM1, symbol Connector:Conn_01x02_Male
- removed J?: CAM2, symbol Connector:Conn_01x02_Male
- removed J?: CAM3, symbol Connector:Conn_01x02_Male
- added C? (x2): 1uF, symbol Device:C_Small
- added C? (x2): 10uF, symbol Device:C_Small
- added D?: D_Small, symbol Device:D_Small
- added J?: CAM0, symbol Connector_Generic:Conn_02x03_Counter_Clockwise
- added J?: CAM1, symbol Connector_Generic:Conn_02x03_Counter_Clockwise
- added J?: CAM2, symbol Connector_Generic:Conn_02x03_Counter_Clockwise
- added J?: CAM3, symbol Connector_Generic:Conn_02x03_Counter_Clockwise
- added J?: CAM4, symbol Connector_Generic:Conn_02x03_Counter_Clockwise
- added J?: CAM5, symbol Connector_Generic:Conn_02x03_Counter_Clockwise
- added J?: CAM6, symbol Connector_Generic:Conn_02x03_Counter_Clockwise
- added J?: CAM7, symbol Connector_Generic:Conn_02x03_Counter_Clockwise
- added R? (x4): 100k, symbol Device:R_Small
- added SW? (x2): SW_SPST, symbol Switch:SW_SPST
- added U?: LTC1983ES6-5-TRPBF, SOT-23_S6, symbol LTC1983ES6-5:LTC1983ES6-5-TRPBF
- added U?: SN75HVD3082EDR, D8, symbol SN75HVD3082EDR_:SN75HVD3082EDR
Connections:
- net labels added: RESET-MAIN, RESET-MOTOR, RS485+, RS485-, RS485-D, RS485-R
- net labels removed: +3V3, RESET, RX1
- wire segments 56 -> 108
- no-connect marks 1 -> 141

Commit message: address review comments
Parts:
- removed J? (x2): Conn_01x02_Male, symbol Connector:Conn_01x02_Male
- removed J?: PROGRAMMER, symbol Connector:Conn_01x05_Male
- removed R?: 100k, symbol Device:R_Small
- removed SW?: SW_SPST, symbol Switch:SW_SPST
- removed U?: ATmega2560-16AU | Motor Cont., Package_QFP:TQFP-100_14x14mm_P0.5mm, symbol MCU_Microchip_ATmega:ATmega2560-16AU
- added C? (x2): 22pF, symbol Device:C_Small
- added C?: 100nF, symbol Device:C_Small
- added D?: CDSOT23-SM712, SOT-23-3, symbol CDSOT23-SM712:CDSOT23-SM712
- added R? (x2): 10, symbol Device:R_Small
- added R? (x2): 10k, symbol Device:R_Small
- added R?: 100k, symbol Device:R_Small
- added Y?: 20MHz, symbol Device:Crystal_Small
- T? (x2): symbol ATB2012E-50011M-T01:ATB2012E-50011M-T01 -> main-board-rescue:ATB2012E-50011M-T01-ATB2012E-50011M-T01
- U?: symbol MCU_Microchip_ATmega:ATmega2560-16AU -> main-board-rescue:ATmega2560-16AU-MCU_Microchip_ATmega
- U? (x2): symbol mc14051B:MC14051B -> main-board-rescue:MC14051B-mc14051B
- U?: symbol ATA6560:ATA6560 -> main-board-rescue:ATA6560-ATA6560
- U?: symbol LTC1983ES6-5:LTC1983ES6-5-TRPBF -> main-board-rescue:LTC1983ES6-5-TRPBF-LTC1983ES6-5
- U?: symbol SN75HVD3082EDR_:SN75HVD3082EDR -> main-board-rescue:SN75HVD3082EDR-SN75HVD3082EDR_
Connections:
- net labels added: RS485-DIR, RX0BF, RX1BF, TX0RTS, TX1RTS, TX2RTS, VID0-0, VID0-1, VID0-2, VID1-0, VID1-1, VID1-2
- net labels removed: INTERCON0, INTERCON1, PROG1-RX, PROG1-TX, RESET-MOTOR, RJ45+, RJ45-, RX0, T0, T1, T2, T3, T4, T5, T6, T7, XTAL1, XTAL2, XTL1, XTL2
- wire segments 108 -> 140
- no-connect marks 141 -> 67
Other:
- note added: "Near uC"
- note added: "Pulse-Proof Thick-Film Resistor\nCRCW060310RJNEAHP\n"
- moved on the sheet: C?, D?, R?
