File: main-board/main-board.sch (KiCad schematic (older format))
At the start: 69 parts, among them J1 MOTOR0, J10 PROGRAMMER, J11 CAM0, J12 CAM1, J13 CAM2, J14 CAM3, J15 CAM4, J16 CAM5, J17 CAM6, J18 CAM7, J19 PowerBoard Interface, J2 MOTOR1, J20 IMU Breakout, J21 ICSP (DO NOT POPULATE), J3 MOTOR2, J4 MOTOR3, J5 Tether Interface, J6 MOTOR4, J7 MOTOR5, J8 MOTOR6, J9 MOTOR7, SW1 SW_SPST, U1 MCP2515-EST, U10 MAX4449ESE+, U2 ATA6560, U3 ATmega2560-16AU | Main Proc, U4 MC14051B, U5 MC14051B, U6 MAX490E, U7 LTC1983ES6-5-TRPBF, U8 MAX4449ESE+, Y1 20MHz, Y2 20MHz

Commit message: S1.0.3 B1.0.3 See Desc
* various layout changes
* remove 0-ohm resistors on CAN
* add RS485 full-duplex
* add optional USB connection
* change crystal footprint
* I'm sure I've forgotten things sorry
Parts:
- removed J19: PowerBoard Interface, Connector_PinHeader_2.54mm:PinHeader_1x04_P2.54mm_Vertical, symbol Connector:Conn_01x04_Male
- removed J5: Tether Interface, Connector_PinHeader_2.54mm:PinHeader_2x06_P2.54mm_Vertical, symbol Connector_Generic:Conn_02x06_Counter_Clockwise
- removed R1: 10k, Resistor_SMD:R_0603_1608Metric, symbol Device:R_Small
- removed R19, R20: 0, Resistor_SMD:R_0603_1608Metric, symbol Device:R
- added J19: PowerBoard Interface, Connector_PinSocket_2.54mm:PinSocket_1x04_P2.54mm_Vertical, symbol Connector:Conn_01x04_Female
- added J22: PLAN (US)B PINS, Connector_PinHeader_2.54mm:PinHeader_1x02_P2.54mm_Vertical, symbol Connector:Conn_01x02_Male
- added J5: TETHER INTERFACE, Connector_PinHeader_2.54mm:PinHeader_2x06_P2.54mm_Vertical, symbol Connector_Generic:Conn_02x06_Odd_Even
- Y1, Y2: footprint Crystal:Crystal_HC49-U_Vertical -> Crystal:Crystal_SMD_Abracon_ABM7-2Pin_6.0x3.5mm
Connections:
- net labels removed: RESET-MAIN
- wire segments 191 -> 189
- no-connect marks 69 -> 67
Changed lines of the file:
@@
 Title "TITAN-II Main Board"
 Date "2018-11-02"
-Rev "1.0.2"
+Rev "1.0.3"
 Comp "Missouri University of Science and Technology - Underwater Robotics Team"
 Comment1 "The main logic board / motherboard of the TITAN-II 2018-2019 UROV"
@@
 $EndComp
 Text GLabel 1700 1500 1    50   Input ~ 0
-RESET-MAIN
+RESET_MAIN
 $Comp
 L power:GND #PWR013
@@
 	1    0    0    -1
 $EndComp
-Text GLabel 7650 9400 2    50   Input ~ 0
+Text GLabel 6650 9400 0    50   Input ~ 0
 CAN-
-Text GLabel 7650 9500 2    50   Input ~ 0
+Text GLabel 6650 9500 0    50   Input ~ 0
 CAN+
 $Comp
@@
 SCK
 NoConn ~ 2050 9200
-$Comp
-L Device:R_Small R1
-U 1 1 5BCB3C5C
-P 1800 9050
-F 0 "R1" V 1900 9050 50  0000 C CNN
-F 1 "10k" V 1800 9050 50  0000 C CNN
-F 2 "Resistor_SMD:R_0603_1608Metric" H 1800 9050 50  0001 C CNN
-F 3 "~" H 1800 9050 50  0001 C CNN
-	1    1800 9050
-	-1   0    0    1
-$EndComp
 Wire Wire Line
 	2050 9000 1950 9000
@@
 	2050 9100 1950 9100
 Wire Wire Line
-	1800 8950 1950 8950
-Wire Wire Line
 	1950 8950 1950 9000
 Wire Wire Line
 	1950 9100 1950 9150
-Wire Wire Line
-	1950 9150 1800 9150
 $Comp
 L Device:Crystal_Small Y1
@@
 F 0 "Y1" H 1450 8950 50  0000 L CNN
 F 1 "20MHz" V 1700 8950 50  0000 L CNN
-F 2 "Crystal:Crystal_HC49-U_Vertical" H 1500 9050 50  0001 C CNN
+F 2 "Crystal:Crystal_SMD_Abracon_ABM7-2Pin_6.0x3.5mm" H 1500 9050 50  0001 C CNN
 F 3 "~" H 1500 9050 50  0001 C CNN
 	1    1500 9050
 	0    1    1    0
 $EndComp
-Wire Wire Line
-	1800 9150 1500 9150
-Connection ~ 1800 9150
-Wire Wire Line
-	1500 8950 1800 8950
-Connection ~ 1800 8950
 $Comp
 L Device:C_Small C1
@@
 Wire Wire Line
 	4800 6750 5050 6750
+Text GLabel 6650 9100 0    50   Input ~ 0
+VID0+
+Text GLabel 6650 9000 0    50   Input ~ 0
+VID0-
+Text GLabel 6650 9200 0    50   Input ~ 0
+VID1+
 Text GLabel 6650 9300 0    50   Input ~ 0
-VID0+
-Text GLabel 6650 9200 0    50   Input ~ 0
-VID0-
-Text GLabel 6650 9100 0    50   Input ~ 0
-VID1+
-Text GLabel 6650 9000 0    50   Input ~ 0
 VID1-
 Text GLabel 3650 2500 2    50   Input ~ 0
@@
 SO
 Text GLabel 9900 8300 2    50   Input ~ 0
-RESET-MAIN
+RESET_MAIN
 $Comp
 L Switch:SW_SPST SW1
@@
 F 0 "Y2" V 1354 2088 50  0000 L CNN
 F 1 "20MHz" V 1600 1800 50  0000 L CNN
-F 2 "Crystal:Crystal_HC49-U_Vertical" H 1400 2000 50  0001 C CNN
+F 2 "Crystal:Crystal_SMD_Abracon_ABM7-2Pin_6.0x3.5mm" H 1400 2000 50  0001 C CNN
 F 3 "~" H 1400 2000 50  0001 C CNN
 	1    1400 2000
@@
 	1850 1500 1700 1500
 $Comp
-L Connector:Conn_01x04_Male J19
-U 1 1 5BD2A605
-P 9750 9300
-F 0 "J19" H 9700 9600 50  0000 C CNN
-F 1 "PowerBoard Interface" H 9850 9700 50  0000 C CNN
-F 2 "Connector_PinHeader_2.54mm:PinHeader_1x04_P2.54mm_Vertical" H 9750 9300 50  0001 C CNN
-F 3 "~" H 9750 9300 50  0001 C CNN
-	1    9750 9300
-	1    0    0    -1
-$EndComp
-$Comp
 L power:+5V #PWR0101
 U 1 1 5BD2A907
@@
 NoConn ~ 3650 4600
 $Comp
-L power:+5V #PWR0116
-U 1 1 5BE8B81C
-P 3650 950
-F 0 "#PWR0116" H 3650 800 50  0001 C CNN
-F 1 "+5V" H 3665 1123 50  0000 C CNN
-F 2 "" H 3650 950 50  0001 C CNN
-F 3 "" H 3650 950 50  0001 C CNN
-	1    3650 950
-	1    0    0    -1
-$EndComp
-$Comp
 L Device:C_Small C12
 U 1 1 5BE8B822
@@
 Wire Wire Line
 	3450 1200 2950 1200
-Connection ~ 3650 950
 Connection ~ 2950 1200
 $Comp
@@
 	13950 7375 13950 7275
 $Comp
-L Device:R R20
-U 1 1 5BDFC8D5
-P 7500 9500
-F 0 "R20" V 7600 9700 50  0000 C CNN
-F 1 "0" V 7500 9500 50  0000 C CNN
-F 2 "Resistor_SMD:R_0603_1608Metric" V 7430 9500 50  0001 C CNN
-F 3 "~" H 7500 9500 50  0001 C CNN
-	1    7500 9500
-	0    1    1    0
-$EndComp
-$Comp
-L Device:R R19
-U 1 1 5BE4CF75
-P 7500 9400
-F 0 "R19" V 7400 9600 50  0000 C CNN
-F 1 "0" V 7500 9400 50  0000 C CNN
-F 2 "Resistor_SMD:R_0603_1608Metric" V 7430 9400 50  0001 C CNN
-F 3 "~" H 7500 9400 50  0001 C CNN
-	1    7500 9400
-	0    1    1    0
-$EndComp
-$Comp
 L power:-5V #PWR0109
 U 1 1 5BDDDC28
@@
 Wire Wire Line
 	13600 1800 13950 1800
+Text GLabel 7350 9300 2    50   Input ~ 0
+TX_H
+Text GLabel 7350 9200 2    50   Input ~ 0
+TX_L
+Text GLabel 7350 9100 2    50   Input ~ 0
+RX_L
 Text GLabel 7350 9000 2    50   Input ~ 0
-TX_H
-Text GLabel 7350 9100 2    50   Input ~ 0
-TX_L
-Text GLabel 7350 9300 2    50   Input ~ 0
-RX_L
-Text GLabel 7350 9200 2    50   Input ~ 0
 RX_H
 Wire Wire Line
@@
 Wire Wire Line
 	7250 9300 7350 9300
-$Comp
-L Connector_Generic:Conn_02x06_Counter_Clockwise J5
-U 1 1 5BFD6972
+Wire Wire Line
+	6750 9400 6650 9400
+Wire Wire Line
+	6750 9500 6650 9500
+Wire Wire Line
+	6650 9000 6750 9000
+Wire Wire Line
+	6650 9100 6750 9100
+Wire Wire Line
+	6650 9200 6750 9200
+Wire Wire Line
+	6650 9300 6750 9300
+$Comp
+L Connector:Conn_01x02_Male J22
+U 1 1 5BE1A1EF
+P 7450 9400
+F 0 "J22" H 7450 9100 50  0000 C CNN
+F 1 "PLAN (US)B PINS" H 7450 9225 50  0000 C CNN
+F 2 "Connector_PinHeader_2.54mm:PinHeader_1x02_P2.54mm_Vertical" H 7450 9400 50  0001 C CNN
+F 3 "~" H 7450 9400 50  0001 C CNN
+	1    7450 9400
+	-1   0    0    -1
+$EndComp
+$Comp
+L Connector_Generic:Conn_02x06_Odd_Even J5
+U 1 1 5BE1B408
 P 6950 9200
 F 0 "J5" H 7000 9617 50  0000 C CNN
-F 1 "Tether Interface" H 7000 9526 50  0000 C CNN
+F 1 "TETHER INTERFACE" H 7000 9526 50  0000 C CNN
 F 2 "Connector_PinHeader_2.54mm:PinHeader_2x06_P2.54mm_Vertical" H 6950 9200 50  0001 C CNN
 F 3 "~" H 6950 9200 50  0001 C CNN
@@
 	1    0    0    -1
 $EndComp
-Wire Wire Line
-	7250 9400 7350 9400
-Wire Wire Line
-	7250 9500 7350 9500
-Wire Wire Line
-	6650 9000 6750 9000
-Wire Wire Line
-	6650 9100 6750 9100
-Wire Wire Line
-	6650 9200 6750 9200
-Wire Wire Line
-	6650 9300 6750 9300
-NoConn ~ 6750 9400
-NoConn ~ 6750 9500
+$Comp
+L Connector:Conn_01x04_Female J19
+U 1 1 5BE7B491
+P 9750 9400
+F 0 "J19" H 10125 9275 50  0000 C CNN
+F 1 "PowerBoard Interface" H 10150 9350 50  0000 C CNN
+F 2 "Connector_PinSocket_2.54mm:PinSocket_1x04_P2.54mm_Vertical" H 9750 9400 50  0001 C CNN
+F 3 "~" H 9750 9400 50  0001 C CNN
+	1    9750 9400
+	-1   0    0    1
+$EndComp
+Wire Wire Line
+	1500 9150 1950 9150
+Wire Wire Line
+	1500 8950 1950 8950
 $EndSCHEMATC
