File: module-tester-board/module-tester-board.sch (KiCad schematic (older format))
At the start: 26 parts, among them J1 Conn_01x08_Male, J2 Barrel_Jack, J4 Conn_01x04_Male, SW1 SW_DIP_x04, U1 LT8330, U4 MCP2515-EST, U5 ATA6560,1, Y1 20MHz

Commit message: S1.0.0 B1.0.0 (See Desc)
* Add step
* move gerbers
* remove library
* assign 3d models and generate step file
* add more ground plane vias
Parts:
- U5: symbol URT_cache:ATA6560,1 -> ATA6560_1:ATA6560,1
Changed lines of the file:
@@
 Sheet 1 1
 Title "module-tester-board"
-Date "2018-10-05"
-Rev "0.0.12"
+Date "2018-11-01"
+Rev "1.0.0"
 Comp "Missouri University of Science and Technology - Underwater Robotics Team"
 Comment1 "Board for testing ROV modules away from ROV."
@@
 $EndComp
 $Comp
-L URT_cache:ATA6560,1 U5
+L ATA6560_1:ATA6560,1 U5
 U 1 1 5B822EF5
 P 9550 3000
