File: module-tester-board/module-tester-board.sch (KiCad schematic (older format))
At the start: 29 parts, among them J1 Conn_01x08_Male, J2 Barrel_Jack, J4 Conn_01x04_Male, SW1 SW_SPST, SW2 SW_SPST, SW3 SW_SPST, SW4 SW_SPST, U1 LT8330, U4 MCP2515-EST, U5 ATA6560,1, Y1 20MHz

Commit message: B: 0.0.3 S: 0.0.10 12mil track and Gerber
Parts:
- removed SW1, SW2, SW3, SW4: SW_SPST, Button_Switch_THT:SW_DIP_SPSTx01_Slide_9.78x4.72mm_W7.62mm_P2.54mm, symbol Switch:SW_SPST
- added SW1: SW_DIP_x04, Button_Switch_THT:SW_DIP_SPSTx04_Slide_9.78x12.34mm_W7.62mm_P2.54mm, symbol Switch:SW_DIP_x04
Connections:
- wire segments 119 -> 116
Changed lines of the file:
@@
 Sheet 1 1
 Title "module-tester-board"
-Date "2018-09-30"
-Rev "0.0.9"
+Date "2018-10-05"
+Rev "0.0.12"
 Comp "Missouri University of Science and Technology - Underwater Robotics Team"
 Comment1 "Board for testing ROV modules away from ROV."
@@
 L Connector:Conn_01x04_Male J4
 U 1 1 5B823405
-P 11500 7900
-F 0 "J4" V 11350 7850 50  0000 C CNN
-F 1 "Conn_01x04_Male" V 11450 7850 50  0000 C CNN
-F 2 "Connector_PinHeader_2.54mm:PinHeader_1x04_P2.54mm_Vertical" H 11500 7900 50  0001 C CNN
-F 3 "~" H 11500 7900 50  0001 C CNN
-	1    11500 7900
-	0    -1   -1   0
+P 11600 7900
+F 0 "J4" V 11450 7850 50  0000 C CNN
+F 1 "Conn_01x04_Male" V 11550 7850 50  0000 C CNN
+F 2 "Connector_PinHeader_2.54mm:PinHeader_1x04_P2.54mm_Vertical" H 11600 7900 50  0001 C CNN
+F 3 "~" H 11600 7900 50  0001 C CNN
+	1    11600 7900
+	0    1    -1   0
 $EndComp
 $Comp
@@
 L Connector:Conn_01x08_Male J1
 U 1 1 5B833C38
-P 12650 7500
-F 0 "J1" V 12400 7450 50  0000 C CNN
-F 1 "Conn_01x08_Male" V 12550 7450 50  0000 C CNN
-F 2 "Connector_PinHeader_2.54mm:PinHeader_1x08_P2.54mm_Vertical" H 12650 7500 50  0001 C CNN
-F 3 "~" H 12650 7500 50  0001 C CNN
-	1    12650 7500
-	-1   0    0    1
+P 12650 7400
+F 0 "J1" V 12400 7350 50  0000 C CNN
+F 1 "Conn_01x08_Male" V 12550 7350 50  0000 C CNN
+F 2 "Connector_PinHeader_2.54mm:PinHeader_1x08_P2.54mm_Vertical" H 12650 7400 50  0001 C CNN
+F 3 "~" H 12650 7400 50  0001 C CNN
+	1    12650 7400
+	-1   0    0    -1
 $EndComp
 Wire Wire Line
@@
 Wire Wire Line
 	6150 7850 6150 7950
-$Comp
-L Switch:SW_SPST SW1
-U 1 1 5B890B45
-P 10650 7150
-F 0 "SW1" H 10200 7150 50  0000 C CNN
-F 1 "SW_SPST" H 9900 7150 50  0000 C CNN
-F 2 "Button_Switch_THT:SW_DIP_SPSTx01_Slide_9.78x4.72mm_W7.62mm_P2.54mm" H 10650 7150 50  0001 C CNN
-F 3 "" H 10650 7150 50  0001 C CNN
-	1    10650 7150
-	1    0    0    -1
-$EndComp
-$Comp
-L Switch:SW_SPST SW2
-U 1 1 5B8959F9
-P 10650 7300
-F 0 "SW2" H 10200 7300 50  0000 C CNN
-F 1 "SW_SPST" H 9900 7300 50  0000 C CNN
-F 2 "Button_Switch_THT:SW_DIP_SPSTx01_Slide_9.78x4.72mm_W7.62mm_P2.54mm" H 10650 7300 50  0001 C CNN
-F 3 "" H 10650 7300 50  0001 C CNN
-	1    10650 7300
-	1    0    0    -1
-$EndComp
-$Comp
-L Switch:SW_SPST SW3
-U 1 1 5B895A49
-P 10650 7450
-F 0 "SW3" H 10100 7450 50  0000 C CNN
-F 1 "SW_SPST" H 9800 7450 50  0000 C CNN
-F 2 "Button_Switch_THT:SW_DIP_SPSTx01_Slide_9.78x4.72mm_W7.62mm_P2.54mm" H 10650 7450 50  0001 C CNN
-F 3 "" H 10650 7450 50  0001 C CNN
-	1    10650 7450
-	1    0    0    -1
-$EndComp
-$Comp
-L Switch:SW_SPST SW4
-U 1 1 5B895AAF
-P 10650 7600
-F 0 "SW4" H 10100 7600 50  0000 C CNN
-F 1 "SW_SPST" H 9800 7600 50  0000 C CNN
-F 2 "Button_Switch_THT:SW_DIP_SPSTx01_Slide_9.78x4.72mm_W7.62mm_P2.54mm" H 10650 7600 50  0001 C CNN
-F 3 "" H 10650 7600 50  0001 C CNN
-	1    10650 7600
-	1    0    0    -1
-$EndComp
 Wire Wire Line
 	3500 4500 3500 4450
@@
 Text GLabel 3000 3350 0    50   Input ~ 0
 PWM0
-Text GLabel 10450 7450 0    50   Input ~ 0
+Text GLabel 10250 7500 0    50   Input ~ 0
 PWM0
 Text GLabel 3000 3450 0    50   Input ~ 0
 PWM1
-Text GLabel 10450 7600 0    50   Input ~ 0
+Text GLabel 10250 7600 0    50   Input ~ 0
 PWM1
-Text GLabel 10450 7150 0    50   Input ~ 0
+Text GLabel 10250 7300 0    50   Input ~ 0
 A0
 Text GLabel 4000 3450 2    50   Input ~ 0
 A0
-Text GLabel 10450 7300 0    50   Input ~ 0
+Text GLabel 10250 7400 0    50   Input ~ 0
 A1
 Text GLabel 4000 3550 2    50   Input ~ 0
@@
 $EndComp
 Wire Wire Line
-	10850 7450 11500 7450
-Wire Wire Line
-	11500 7450 11500 7500
-Wire Wire Line
-	11600 7300 11600 7400
-Wire Wire Line
-	10850 7300 11600 7300
-Wire Wire Line
-	11700 7150 11700 7300
-Wire Wire Line
-	10850 7150 11700 7150
+	10850 7500 11500 7500
 Wire Wire Line
 	12450 7300 11700 7300
@@
 	1    0    0    -1
 $EndComp
-Connection ~ 11700 7300
 Wire Wire Line
 	11700 7300 11700 7400
-Connection ~ 11600 7400
 Wire Wire Line
 	11600 7400 11600 7500
@@
 Wire Notes Line
 	13850 5550 15100 5550
+$Comp
+L Switch:SW_DIP_x04 SW1
+U 1 1 5BB6B3B3
+P 10550 7500
+F 0 "SW1" H 10550 7967 50  0000 C CNN
+F 1 "SW_DIP_x04" H 10550 7876 50  0000 C CNN
+F 2 "Button_Switch_THT:SW_DIP_SPSTx04_Slide_9.78x12.34mm_W7.62mm_P2.54mm" H 10550 7500 50  0001 C CNN
+F 3 "" H 10550 7500 50  0001 C CNN
+	1    10550 7500
+	1    0    0    -1
+$EndComp
+Wire Wire Line
+	11700 7300 10850 7300
+Connection ~ 11700 7300
+Wire Wire Line
+	10850 7400 11600 7400
+Connection ~ 11600 7400
 $EndSCHEMATC

Commit message: Added 5v Regulator
Moved some parts to add additonal pin
Parts:
- removed J1: Conn_01x08_Male, Connector_PinHeader_2.54mm:PinHeader_1x08_P2.54mm_Vertical, symbol Connector:Conn_01x08_Male
- added C8, C9: 100uF, Capacitor_THT:CP_Radial_D5.0mm_P2.50mm, symbol Device:CP
- added J1: Conn_01x09, Connector_PinHeader_2.54mm:PinHeader_1x09_P2.54mm_Vertical, symbol Connector_Generic:Conn_01x09
- added U2: L7805, Package_TO_SOT_SMD:SOT-223, symbol Regulator_Linear:L7805
- U5: symbol URT_cache:ATA6560,1 -> module-tester-board-rescue:ATA6560,1-URT_cache
Connections:
- net labels added: +5VD
- wire segments 116 -> 127
Other:
- note added: "Dedicated +5V Output"
Changed lines of the file:
@@
 $EndComp
 $Comp
-L URT_cache:ATA6560,1 U5
+L module-tester-board-rescue:ATA6560,1-URT_cache U5
 U 1 1 5B822EF5
 P 9550 3000
@@
 	1    3500 3450
 	1    0    0    -1
-$EndComp
-$Comp
-L Connector:Conn_01x08_Male J1
-U 1 1 5B833C38
-P 12650 7400
-F 0 "J1" V 12400 7350 50  0000 C CNN
-F 1 "Conn_01x08_Male" V 12550 7350 50  0000 C CNN
-F 2 "Connector_PinHeader_2.54mm:PinHeader_1x08_P2.54mm_Vertical" H 12650 7400 50  0001 C CNN
-F 3 "~" H 12650 7400 50  0001 C CNN
-	1    12650 7400
-	-1   0    0    -1
 $EndComp
 Wire Wire Line
@@
 L power:GND #PWR0104
 U 1 1 5B950373
-P 12450 7800
-F 0 "#PWR0104" H 12450 7550 50  0001 C CNN
-F 1 "GND" H 12455 7627 50  0000 C CNN
-F 2 "" H 12450 7800 50  0001 C CNN
-F 3 "" H 12450 7800 50  0001 C CNN
-	1    12450 7800
+P 12450 7950
+F 0 "#PWR0104" H 12450 7700 50  0001 C CNN
+F 1 "GND" H 12455 7777 50  0000 C CNN
+F 2 "" H 12450 7950 50  0001 C CNN
+F 3 "" H 12450 7950 50  0001 C CNN
+	1    12450 7950
 	1    0    0    -1
 $EndComp
@@
 Wire Wire Line
 	12450 7300 11700 7300
+Text GLabel 12450 7200 0    50   Input ~ 0
+CANH
 Text GLabel 12450 7100 0    50   Input ~ 0
-CANH
-Text GLabel 12450 7200 0    50   Input ~ 0
 CANL
 Text GLabel 10050 3100 2    50   Input ~ 0
@@
 	10850 7400 11600 7400
 Connection ~ 11600 7400
+$Comp
+L Connector_Generic:Conn_01x09 J1
+U 1 1 5BE10046
+P 12650 7500
+F 0 "J1" H 12730 7542 50  0000 L CNN
+F 1 "Conn_01x09" H 12730 7451 50  0000 L CNN
+F 2 "Connector_PinHeader_2.54mm:PinHeader_1x09_P2.54mm_Vertical" H 12650 7500 50  0001 C CNN
+F 3 "~" H 12650 7500 50  0001 C CNN
+	1    12650 7500
+	1    0    0    -1
+$EndComp
+$Comp
+L Regulator_Linear:L7805 U2
+U 1 1 5BE1018D
+P 8750 5500
+F 0 "U2" H 8750 5742 50  0000 C CNN
+F 1 "L7805" H 8750 5651 50  0000 C CNN
+F 2 "Package_TO_SOT_SMD:SOT-223" H 8775 5350 50  0001 L CIN
+F 3 "http://www.st.com/content/ccc/resource/technical/document/datasheet/41/4f/b3/b0/12/d4/47/88/CD00000444.pdf/files/CD00000444.pdf/jcr:content/translations/en.CD00000444.pdf" H 8750 5450 50  0001 C CNN
+	1    8750 5500
+	1    0    0    -1
+$EndComp
+$Comp
+L Device:CP C8
+U 1 1 5BE102EA
+P 8300 5650
+F 0 "C8" H 7950 5700 50  0000 L CNN
+F 1 "100uF" H 7950 5600 50  0000 L CNN
+F 2 "Capacitor_THT:CP_Radial_D5.0mm_P2.50mm" H 8338 5500 50  0001 C CNN
+F 3 "~" H 8300 5650 50  0001 C CNN
+	1    8300 5650
+	1    0    0    -1
+$EndComp
+$Comp
+L Device:CP C9
+U 1 1 5BE10384
+P 9200 5650
+F 0 "C9" H 9318 5696 50  0000 L CNN
+F 1 "100uF" H 9318 5605 50  0000 L CNN
+F 2 "Capacitor_THT:CP_Radial_D5.0mm_P2.50mm" H 9238 5500 50  0001 C CNN
+F 3 "~" H 9200 5650 50  0001 C CNN
+	1    9200 5650
+	1    0    0    -1
+$EndComp
+Wire Wire Line
+	9050 5500 9200 5500
+Wire Wire Line
+	8450 5500 8300 5500
+Wire Wire Line
+	8300 5800 8750 5800
+Wire Wire Line
+	8750 5800 9200 5800
+Connection ~ 8750 5800
+$Comp
+L power:GND #PWR0118
+U 1 1 5BE201DD
+P 8750 5900
+F 0 "#PWR0118" H 8750 5650 50  0001 C CNN
+F 1 "GND" H 8755 5727 50  0000 C CNN
+F 2 "" H 8750 5900 50  0001 C CNN
+F 3 "" H 8750 5900 50  0001 C CNN
+	1    8750 5900
+	1    0    0    -1
+$EndComp
+Wire Wire Line
+	8750 5900 8750 5800
+$Comp
+L power:+5VD #PWR0119
+U 1 1 5BE245C3
+P 9300 5500
+F 0 "#PWR0119" H 9300 5350 50  0001 C CNN
+F 1 "+5VD" H 9315 5673 50  0000 C CNN
+F 2 "" H 9300 5500 50  0001 C CNN
+F 3 "" H 9300 5500 50  0001 C CNN
+	1    9300 5500
+	1    0    0    -1
+$EndComp
+Wire Wire Line
+	9200 5500 9300 5500
+Connection ~ 9200 5500
+$Comp
+L power:+12V #PWR0120
+U 1 1 5BE28A11
+P 8200 5500
+F 0 "#PWR0120" H 8200 5350 50  0001 C CNN
+F 1 "+12V" H 8200 5650 50  0000 C CNN
+F 2 "" H 8200 5500 50  0001 C CNN
+F 3 "" H 8200 5500 50  0001 C CNN
+	1    8200 5500
+	1    0    0    -1
+$EndComp
+Wire Wire Line
+	8300 5500 8200 5500
+Connection ~ 8300 5500
+$Comp
+L power:+5VD #PWR0121
+U 1 1 5BE2DA0F
+P 12150 7950
+F 0 "#PWR0121" H 12150 7800 50  0001 C CNN
+F 1 "+5VD" H 12165 8123 50  0000 C CNN
+F 2 "" H 12150 7950 50  0001 C CNN
+F 3 "" H 12150 7950 50  0001 C CNN
+	1    12150 7950
+	1    0    0    -1
+$EndComp
+Wire Wire Line
+	12450 7800 12300 7800
+Wire Wire Line
+	12300 7800 12300 7950
+Wire Wire Line
+	12300 7950 12150 7950
+Wire Wire Line
+	12450 7900 12450 7950
+Text Notes 7950 6250 0    100  Italic 0
+Dedicated +5V Output
+Wire Notes Line
+	9700 5150 9700 6300
+Wire Notes Line
+	9700 6300 7900 6300
+Wire Notes Line
+	7900 6300 7900 5150
+Wire Notes Line
+	7900 5150 9700 5150
 $EndSCHEMATC
