File: Motor test module/_autosave-Motor test module.kicad_pcb (KiCad board)
At the start: 2 copper layers, 16 parts, among them U1 TPS63060, U8 ATmega2560-16AU, U9 MCP2515-EST

Commit message: Motor Test final schematic
Parts:
- added C16: 100n, Capacitor_SMD:C_0603_1608Metric, F.Cu at (172.6, 101.6)
- added C17: 100n, Capacitor_SMD:C_0603_1608Metric, F.Cu at (166.6, 100.1)
- added C18: 100n, Capacitor_SMD:C_0603_1608Metric, F.Cu at (169.6, 98.5)
- added C19: 100n, Capacitor_SMD:C_0603_1608Metric, F.Cu at (166.6, 101.6)
- added C20: 100n, Capacitor_SMD:C_0603_1608Metric, F.Cu at (169.6, 100.1)
- added C21: 100n, Capacitor_SMD:C_0603_1608Metric, F.Cu at (172.6, 98.5)
- added C22: 100n, Capacitor_SMD:C_0603_1608Metric, F.Cu at (166.6, 103.1)
- added C23: 100n, Capacitor_SMD:C_0603_1608Metric, F.Cu at (169.6, 101.6)
- added C24: 100n, Capacitor_SMD:C_0603_1608Metric, F.Cu at (172.6, 100.1)
- added C25: 100n, Capacitor_SMD:C_0603_1608Metric, F.Cu at (166.6, 104.6)
- added C26: 100n, Capacitor_SMD:C_0603_1608Metric, F.Cu at (175.6, 98.5)
- added C27: 100n, Capacitor_SMD:C_0603_1608Metric, F.Cu at (169.6, 103.1)
- added C28: 100n, Capacitor_SMD:C_0603_1608Metric, F.Cu at (175.6, 100.1)
- added C29: 100n, Capacitor_SMD:C_0603_1608Metric, F.Cu at (166.6, 98.5)
- added C30: 100n, Capacitor_SMD:C_0603_1608Metric, F.Cu at (169.6, 104.6)
- added R1: 1M, Resistor_SMD:R_0603_1608Metric, F.Cu at (178.6, 98.5)
- added R10: 10k, Resistor_SMD:R_0603_1608Metric, F.Cu at (178.6, 104.6)
- added R2: 100k, Resistor_SMD:R_0603_1608Metric, F.Cu at (172.6, 103.1)
- added R3: 1M, Resistor_SMD:R_0603_1608Metric, F.Cu at (175.6, 101.6)
- added R4: 1M, Resistor_SMD:R_0603_1608Metric, F.Cu at (178.6, 100.1)
- added R5: 100k, Resistor_SMD:R_0603_1608Metric, F.Cu at (172.6, 104.6)
- added R6: 1M, Resistor_SMD:R_0603_1608Metric, F.Cu at (175.6, 103.1)
- added R7: 10k, Resistor_SMD:R_0603_1608Metric, F.Cu at (178.6, 101.6)
- added R8: 10k, Resistor_SMD:R_0603_1608Metric, F.Cu at (175.6, 104.6)
- added R9: 27R, Resistor_SMD:R_0603_1608Metric, F.Cu at (178.6, 103.1)
