File: Motor test module/Motor test module.sch (KiCad schematic (older format))
At the start: 5 parts

Commit message: Add servos
Parts:
- added J? (x3): Conn_02x04_Counter_Clockwise, symbol Connector_Generic:Conn_02x04_Counter_Clockwise
Connections:
- net labels added: C, D, E1, E2, E3, E4, Servo1, Servo2
- net labels removed: Encoder
- wire segments 17 -> 23
- no-connect marks 1 -> 6
Other:
- moved on the sheet: U?

Commit message: First draft of motor test module
Parts:
- added J? (x2): Conn_02x04_Counter_Clockwise, symbol Connector_Generic:Conn_02x04_Counter_Clockwise
- added U? (x2): AP1017AEN, symbol h-bridge:AP1017AEN
Connections:
- net labels added: E5, E6, M+1, M+2, M-1, M-2
- wire segments 23 -> 41
- no-connect marks 6 -> 16
Other:
- moved on the sheet: U?

Commit message: Second draft of Motor Test
Connections:
- net labels added: +5V, A1+, A1-, A2+, A2-, B1+, B1-, B2+, B2-
- net labels removed: 5v
- wire segments 41 -> 54
Other:
- moved on the sheet: J?, U?

Commit message: Add power regulator
Parts:
- removed U?: L7805, symbol Regulator_Linear:L7805
- added C? (x3): C, symbol Device:C
- added L?: L, symbol Device:L
- added R? (x3): R, symbol Device:R
- added U? (x2): AP1017AEN, symbol h-bridge:AP1017AEN
- added U?: TPS63060, Package_SON:Texas_S-PWSON-N10_ThermalVias, symbol Regulator_Switching:TPS63060
Connections:
- net labels added: E, E+, E-, F, F+, F-, G, H, INA1+, INA1-, INA2+, INA2-, INB1+, INB1-, INB2+, INB2-, M1+, M1-, M2+, M2-
- net labels removed: A1+, A1-, A2+, A2-, B1+, B1-, B2+, B2-, E3, E4, E5, E6, M+1, M+2, M-1, M-2
- wire segments 54 -> 105
Other:
- moved on the sheet: J?

Commit message: Add arduino mega
Parts:
- removed A?: Arduino_Nano_v3.x, Module:Arduino_Nano, symbol MCU_Module:Arduino_Nano_v3.x
- added C1-2: 10uF, symbol Device:C
- added C4-1, C4-2, C4-3: 22uF, symbol Device:C
- added C5-1, C5-2: 20pF, symbol Device:C
- added C6, C7, C8, C9: 100nF, symbol Device:C
- added R1: 1M, symbol Device:R
- added R2: 27R, symbol Device:R
- added U?: ATmega2560-16AU, Package_QFP:TQFP-100_14x14mm_P0.5mm, symbol MCU_Microchip_ATmega:ATmega2560-16AU
- added Y1: 16MHz, symbol Device:Crystal
- C1-1: renamed from C?; value C -> 10uF
- C2: renamed from C?; value C -> 0.1uF
- C3: renamed from C?; value C -> 10pF
- L1: renamed from L?; value L -> XFL4020-102
- R1, R3: renamed from R?; value R -> 1M
- R2: renamed from R?; value R -> 111k
- gave numbers to parts that had none: 13
Connections:
- net labels added: M1A+, M1A+C, M1A-, M1A-C, M1B+, M1B+C, M1B-, M1B-C, M2A+, M2A+C, M2A-, M2A-C, M2B+, M2B+C, M2B-, M2B-C, VCC
- net labels removed: A, A+, A-, B, B+, B-, C, D, E, E+, E-, F, F+, F-, G, H, INA1+, INA1-, INA2+, INA2-, INB1+, INB1-, INB2+, INB2-
- wire segments 105 -> 157
Other:
- moved on the sheet: C1-1, C2, C3, J1, J2, J3, J4, J5, J6, L1, R1, R2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

Commit message: Module Motor Test Draft
Parts:
- added C10: 1u, symbol Device:C
- added C9-1, C9-2: 15p, symbol Device:C
- added D1: 1N4007, symbol Device:D
- added R5: 100k, symbol Device:R
- added R6: 1M, symbol Device:R
- added R7 (x2), R8: 10k, symbol Device:R
- added U9: MCP2515-EST, Package_SO:TSSOP-20_4.4x6.5mm_P0.65mm, symbol Interface_CAN_LIN:MCP2515-EST
- added U?: ATA6560,1, symbol URT_cache:ATA6560,1
- added Y?: 16MHz, symbol Device:Crystal
- C1-1, C1-2: value 10uF -> 10u
- C2: value 0.1uF -> 0.1u
- C3: value 10pF -> 10p
- C4-1, C4-2, C4-3: value 22uF -> 22u
- C5-1, C5-2: value 20pF -> 20p
- C6, C7, C8, C9: value 100nF -> 100n
- gave numbers to parts that had none: 1
- renumbered R1 to R4, R2 to R5
Connections:
- net labels added: CANH, CANL, INT, M1+C, M1-C, M2+C, M2-C, RX0, RX1, Reset, S0, SCK, SI, SS, TX0, TX1, TX2
- wire segments 157 -> 186
- no-connect marks 16 -> 73
Other:
- moved on the sheet: C1-1, C1-2, C2, C3, C4-1, C4-2, C4-3, C5-1, C5-2, C6, C7, C8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

Commit message: Motor Test final schematic
Parts:
- removed C1-1, C1-2: 10u, symbol Device:C
- removed C4-1, C4-2, C4-3: 22u, symbol Device:C
- removed C6, C7, C8: 100n, symbol Device:C
- added C1: 10u, Diode_THT:D_DO-41_SOD81_P7.62mm_Horizontal, symbol Device:CP
- added C16, C17, C18, C19, C20, C21, C22, C23, C24, C25, C26, C27, C28, C29, C30: 100n, Capacitor_SMD:C_0603_1608Metric, symbol Device:C
- added C2: 10u, symbol Device:CP
- added C5, C6, C7: 22u, Capacitor_SMD:CP_Elec_4x5.4, symbol Device:CP
- C11: renamed from C9; footprint (none) -> Capacitor_SMD:C_0603_1608Metric
- C12: renamed from C9-1; footprint (none) -> Capacitor_SMD:C_0603_1608Metric
- C13: renamed from C9-2; footprint (none) -> Capacitor_SMD:C_0603_1608Metric
- C14: renamed from C10; footprint (none) -> Capacitor_SMD:C_0603_1608Metric
- C3: renamed from C2; footprint (none) -> Capacitor_SMD:C_0603_1608Metric
- C4: renamed from C3; footprint (none) -> Capacitor_SMD:C_0603_1608Metric
- C8: renamed from C5-1; footprint (none) -> Capacitor_SMD:C_0603_1608Metric
- C9: renamed from C5-2; footprint (none) -> Capacitor_SMD:C_0603_1608Metric
- D1: footprint (none) -> Diode_THT:D_DO-41_SOD81_P2.54mm_Vertical_AnodeUp
- R1, R3, R4, R5, R6, R7, R8: footprint (none) -> Resistor_SMD:R_0603_1608Metric
- R10: renamed from R7; footprint (none) -> Resistor_SMD:R_0603_1608Metric
- R2: value 111k -> 100k; footprint (none) -> Resistor_SMD:R_0603_1608Metric
- R9: renamed from R5; footprint (none) -> Resistor_SMD:R_0603_1608Metric
- gave numbers to parts that had none: 2
Connections:
- net labels removed: VCC
- wire segments 186 -> 189
Other:
- moved on the sheet: C11, C14, D1, R5, R7, U2, U3, U4, U5, U7

Commit message: switching computers - wip
Parts:
- removed C1: 10u, Diode_THT:D_DO-41_SOD81_P7.62mm_Horizontal, symbol Device:CP
- removed C12, C13: 15p, Capacitor_SMD:C_0603_1608Metric, symbol Device:C
- removed C2: 10u, symbol Device:CP
- removed C8, C9: 20p, Capacitor_SMD:C_0603_1608Metric, symbol Device:C
- removed R4, R6: 1M, Resistor_SMD:R_0603_1608Metric, symbol Device:R
- removed R9: 27R, Resistor_SMD:R_0603_1608Metric, symbol Device:R
- removed Y1, Y2: 16MHz, symbol Device:Crystal
- added C1, C2: 10u, Capacitor_SMD:C_0603_1608Metric, symbol Device:C
- added Y1, Y2: 16MHz, Crystal:Resonator_SMD_muRata_CSTxExxV-3Pin_3.0x1.1mm, symbol Device:Resonator
- J1, J2, J3, J4, J5, J6: footprint (none) -> Connector_PinHeader_2.54mm:PinHeader_2x04_P2.54mm_Vertical
- L1: footprint (none) -> Inductor_SMD:L_0603_1608Metric
- U10: footprint (none) -> Package_SO:SO-8_5.3x6.2mm_P1.27mm; symbol URT_cache:ATA6560,1 -> Motor-test-module-rescue:ATA6560,1-URT_cache
- U2, U3, U4, U5, U6, U7: footprint (none) -> Package_SON:SON-8-1EP_3x2mm_P0.5mm_EP1.4x1.6mm
- U8: symbol MCU_Microchip_ATmega:ATmega2560-16AU -> Motor-test-module-rescue:ATmega2560-16AU-MCU_Microchip_ATmega
Connections:
- wire segments 189 -> 177
