File: Motor test module/Motor test module.sch (KiCad schematic (older format))
At the start: 51 parts, among them J1 Conn_02x04_Counter_Clockwise, J2 Conn_02x04_Counter_Clockwise, J3 Conn_02x04_Counter_Clockwise, J4 Conn_02x04_Counter_Clockwise, J5 Conn_02x04_Counter_Clockwise, J6 Conn_02x04_Counter_Clockwise, U1 TPS63060, U10 ATA6560,1, U2 AP1017AEN, U3 AP1017AEN, U4 AP1017AEN, U5 AP1017AEN, U6 AP1017AEN, U7 AP1017AEN, U8 ATmega2560-16AU, U9 MCP2515-EST, Y1 16MHz, Y2 16MHz

Commit message: beginning layout
Parts:
- U10: symbol Motor-test-module-rescue:ATA6560,1-URT_cache -> Motor-test-module-rescue:ATA6560,1-URT_cache-Motor-test-module-rescue
- U2, U3, U4, U5, U6, U7: footprint Package_SON:SON-8-1EP_3x2mm_P0.5mm_EP1.4x1.6mm -> Package_SON:WSON-8-1EP_2x2mm_P0.5mm_EP0.9x1.6mm; symbol h-bridge:AP1017AEN -> Motor-test-module-rescue:AP1017AEN-h-bridge
- U8: symbol Motor-test-module-rescue:ATmega2560-16AU-MCU_Microchip_ATmega -> Motor-test-module-rescue:ATmega2560-16AU-MCU_Microchip_ATmega-Motor-test-module-rescue
Changed lines of the file:
@@
 NoConn ~ 13400 3700
 $Comp
-L h-bridge:AP1017AEN U5
+L Motor-test-module-rescue:AP1017AEN-h-bridge U5
 U 1 1 5B95AAAE
 P 9850 8700
 F 0 "U5" H 9825 9065 50  0000 C CNN
 F 1 "AP1017AEN" H 9825 8974 50  0000 C CNN
-F 2 "Package_SON:SON-8-1EP_3x2mm_P0.5mm_EP1.4x1.6mm" H 9500 8550 50  0001 C CNN
+F 2 "Package_SON:WSON-8-1EP_2x2mm_P0.5mm_EP0.9x1.6mm" H 9500 8550 50  0001 C CNN
 F 3 "" H 9500 8550 50  0001 C CNN
 	1    9850 8700
@@
 	13300 5750 13700 5750
 $Comp
-L h-bridge:AP1017AEN U7
+L Motor-test-module-rescue:AP1017AEN-h-bridge U7
 U 1 1 5B9BFA22
 P 9850 3950
 F 0 "U7" H 9825 4315 50  0000 C CNN
 F 1 "AP1017AEN" H 9825 4224 50  0000 C CNN
-F 2 "Package_SON:SON-8-1EP_3x2mm_P0.5mm_EP1.4x1.6mm" H 9500 3800 50  0001 C CNN
+F 2 "Package_SON:WSON-8-1EP_2x2mm_P0.5mm_EP0.9x1.6mm" H 9500 3800 50  0001 C CNN
 F 3 "" H 9500 3800 50  0001 C CNN
 	1    9850 3950
@@
 	8700 3700 8700 4050
 $Comp
-L h-bridge:AP1017AEN U4
+L Motor-test-module-rescue:AP1017AEN-h-bridge U4
 U 1 1 5B9C00A7
 P 7550 8700
 F 0 "U4" H 7525 9065 50  0000 C CNN
 F 1 "AP1017AEN" H 7525 8974 50  0000 C CNN
-F 2 "Package_SON:SON-8-1EP_3x2mm_P0.5mm_EP1.4x1.6mm" H 7200 8550 50  0001 C CNN
+F 2 "Package_SON:WSON-8-1EP_2x2mm_P0.5mm_EP0.9x1.6mm" H 7200 8550 50  0001 C CNN
 F 3 "" H 7200 8550 50  0001 C CNN
 	1    7550 8700
@@
 	6300 3700 6300 4050
 $Comp
-L h-bridge:AP1017AEN U2
+L Motor-test-module-rescue:AP1017AEN-h-bridge U2
 U 1 1 5BACC3D1
 P 9850 5100
 F 0 "U2" H 9825 5465 50  0000 C CNN
 F 1 "AP1017AEN" H 9825 5374 50  0000 C CNN
-F 2 "Package_SON:SON-8-1EP_3x2mm_P0.5mm_EP1.4x1.6mm" H 9500 4950 50  0001 C CNN
+F 2 "Package_SON:WSON-8-1EP_2x2mm_P0.5mm_EP0.9x1.6mm" H 9500 4950 50  0001 C CNN
 F 3 "" H 9500 4950 50  0001 C CNN
 	1    9850 5100
@@
 $EndComp
 $Comp
-L h-bridge:AP1017AEN U3
+L Motor-test-module-rescue:AP1017AEN-h-bridge U3
 U 1 1 5BACC3FB
 P 7500 3950
 F 0 "U3" H 7475 4315 50  0000 C CNN
 F 1 "AP1017AEN" H 7475 4224 50  0000 C CNN
-F 2 "Package_SON:SON-8-1EP_3x2mm_P0.5mm_EP1.4x1.6mm" H 7150 3800 50  0001 C CNN
+F 2 "Package_SON:WSON-8-1EP_2x2mm_P0.5mm_EP0.9x1.6mm" H 7150 3800 50  0001 C CNN
 F 3 "" H 7150 3800 50  0001 C CNN
 	1    7500 3950
@@
 Reset
 $Comp
-L Motor-test-module-rescue:ATA6560,1-URT_cache U10
+L Motor-test-module-rescue:ATA6560,1-URT_cache-Motor-test-module-rescue U10
 U 1 1 5BFBD538
 P 12650 1750
@@
 NoConn ~ 3400 5900
 $Comp
-L Motor-test-module-rescue:ATmega2560-16AU-MCU_Microchip_ATmega U8
+L Motor-test-module-rescue:ATmega2560-16AU-MCU_Microchip_ATmega-Motor-test-module-rescue U8
 U 1 1 5BD5AF2A
 P 4200 6500
@@
 	6050 3400 11000 3400
 $Comp
-L h-bridge:AP1017AEN U6
+L Motor-test-module-rescue:AP1017AEN-h-bridge U6
 U 1 1 5BCC6E90
 P 7500 5100
 F 0 "U6" H 7475 5465 50  0000 C CNN
 F 1 "AP1017AEN" H 7475 5374 50  0000 C CNN
-F 2 "Package_SON:SON-8-1EP_3x2mm_P0.5mm_EP1.4x1.6mm" H 7150 4950 50  0001 C CNN
+F 2 "Package_SON:WSON-8-1EP_2x2mm_P0.5mm_EP0.9x1.6mm" H 7150 4950 50  0001 C CNN
 F 3 "" H 7150 4950 50  0001 C CNN
 	1    7500 5100

Commit message: Second draft of layout
Parts:
- removed C5, C6, C7: 22u, Capacitor_SMD:CP_Elec_4x5.4, symbol Device:CP
- added C5, C6, C7: 22u, Capacitor_SMD:C_0603_1608Metric, symbol Device:C
- added J7: Conn_01x05_MountingPin, Connector_Molex:Molex_Pico-Clasp_501331-0507_1x05-1MP_P1.00mm_Vertical, symbol Connector_Generic_MountingPin:Conn_01x05_MountingPin
- added J8: Screw_Terminal_01x02, TerminalBlock:TerminalBlock_bornier-2_P5.08mm, symbol Connector:Screw_Terminal_01x02
- added R4: 10k, Resistor_SMD:R_0603_1608Metric, symbol Device:R
- added SW1: SW_Push, Button_Switch_THT:SW_PUSH_6mm, symbol Switch:SW_Push
Connections:
- net +12V: now also J8.1 (Pin_1)
- net +5V: now also C5.1, C6.1, C7.1, R4.1
- net CANH: now also U8.95 (PF2)
- net CANL: now also U8.94 (PF3)
- net GNDREF: now also C5.2, C6.2, C7.2, J7.1 (Pin_1), J8.2 (Pin_2), SW1.1
- net at U8.30 (~RESET): now also R4.2, SW1.2
- net Vpp: now reaches U8.73 (PA5)
- net Vpp: now also J7.5 (Pin_5)
- net Rst: now reaches U8.74 (PA4)
- net Rst: now also J7.4 (Pin_4)
- net Rx: now reaches U8.75 (PA3)
- net Rx: now also J7.3 (Pin_3)
- net Tx: now reaches U8.76 (PA2)
- net Tx: now also J7.2 (Pin_2)
- no-connect marks 73 -> 68
Other:
- moved on the sheet: C16, C17, C18, C19, C22, C23, C24, C25, C26, C27, C28, C29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
