File: Motor test module/Motor test module.sch (KiCad schematic (older format))
At the start: 55 parts, among them J1 Conn_02x04_Counter_Clockwise, J2 Conn_02x04_Counter_Clockwise, J3 Conn_02x04_Counter_Clockwise, J4 Conn_02x04_Counter_Clockwise, J5 Conn_02x04_Counter_Clockwise, J6 Conn_02x04_Counter_Clockwise, J7 Conn_01x05_Male, J8 Screw_Terminal_01x02, SW1 SW_Push, U1 TPS63060, U10 ATA6560,1, U2 AP1017AEN, U3 AP1017AEN, U4 AP1017AEN, U5 AP1017AEN, U6 AP1017AEN, U7 AP1017AEN, U8 ATmega2560-16AU, U9 MCP2515-EST, Y1 16MHz, Y2 16MHz

Commit message: Fourth draft of layout
Parts:
- added D2: D_x2_KCom_AAK, Package_TO_SOT_SMD:SOT-23, symbol Device:D_x2_KCom_AAK
- added J9: Screw_Terminal_01x02, TerminalBlock:TerminalBlock_bornier-2_P5.08mm, symbol Connector:Screw_Terminal_01x02
Connections:
- net +3V3: no longer C30.1
- net +5V: now also D2.2 (A); no longer U8.10 (VCC), U8.100 (AVCC), U8.31 (VCC), U8.61 (VCC), U8.80 (VCC)
- net CANH: now also J9.1 (Pin_1); no longer U8.95 (PF2)
- net CANL: now also J9.2 (Pin_2); no longer U8.94 (PF3)
- net at J7.1 (Pin_1): now also D2.1 (A)
- new net VCC: C30.1, D2.3 (K), U8.10 (VCC), U8.100 (AVCC), U8.31 (VCC), U8.61 (VCC), U8.80 (VCC)
- no-connect marks 65 -> 67
Changed lines of the file:
@@
 	1    0    0    -1
 $EndComp
-Text GLabel 5000 8600 2    50   Input ~ 0
-CANH
-Text GLabel 5000 8700 2    50   Input ~ 0
-CANL
 $Comp
 L Connector:Screw_Terminal_01x02 J8
@@
 Wire Notes Line
 	6050 4200 6050 3350
-$Comp
-L power:+3V3 #PWR0185
-U 1 1 5C00689B
-P 1450 4100
-F 0 "#PWR0185" H 1450 3950 50  0001 C CNN
-F 1 "+3V3" H 1465 4273 50  0000 C CNN
-F 2 "" H 1450 4100 50  0001 C CNN
-F 3 "" H 1450 4100 50  0001 C CNN
-	1    1450 4100
-	1    0    0    -1
-$EndComp
 Text GLabel 5000 7600 2    50   Input ~ 0
 Tx
@@
 	0    1    1    0
 $EndComp
-Wire Notes Line
-	5900 850  7250 850
-Wire Notes Line
-	5900 2100 5900 850
-Wire Notes Line
-	7250 2100 5900 2100
-Wire Notes Line
-	7250 850  7250 2100
 $Comp
-L power:+5V #PWR?
-U 1 1 5C019AEE
-P 4300 3400
-F 0 "#PWR?" H 4300 3250 50  0001 C CNN
-F 1 "+5V" H 4315 3573 50  0000 C CNN
-F 2 "" H 4300 3400 50  0001 C CNN
-F 3 "" H 4300 3400 50  0001 C CNN
-	1    4300 3400
+L power:+5V #PWR0191
+U 1 1 5C032B9A
+P 7400 1200
+F 0 "#PWR0191" H 7400 1050 50  0001 C CNN
+F 1 "+5V" H 7415 1373 50  0000 C CNN
+F 2 "" H 7400 1200 50  0001 C CNN
+F 3 "" H 7400 1200 50  0001 C CNN
+	1    7400 1200
 	1    0    0    -1
 $EndComp
-Connection ~ 4300 3400
 $Comp
-L power:+5V #PWR?
-U 1 1 5C032B9A
+L Device:D_x2_KCom_AAK D2
+U 1 1 5C091BCF
 P 7100 1400
-F 0 "#PWR?" H 7100 1250 50  0001 C CNN
-F 1 "+5V" H 7115 1573 50  0000 C CNN
-F 2 "" H 7100 1400 50  0001 C CNN
-F 3 "" H 7100 1400 50  0001 C CNN
+F 0 "D2" H 7100 1616 50  0000 C CNN
+F 1 "D_x2_KCom_AAK" H 7100 1525 50  0000 C CNN
+F 2 "Package_TO_SOT_SMD:SOT-23" H 7100 1400 50  0001 C CNN
+F 3 "~" H 7100 1400 50  0001 C CNN
 	1    7100 1400
 	1    0    0    -1
 $EndComp
+Wire Wire Line
+	7400 1200 7400 1400
+Wire Wire Line
+	6800 1400 6750 1400
+Wire Notes Line
+	6100 1850 7600 1850
+Wire Notes Line
+	7600 1850 7600 900
+Wire Notes Line
+	7600 900  6100 900
+Wire Notes Line
+	6100 900  6100 1850
+Text GLabel 7100 1600 3    50   Input ~ 0
+VCC
+Text GLabel 4300 3400 1    50   Input ~ 0
+VCC
+Text GLabel 1450 4100 1    50   Input ~ 0
+VCC
+NoConn ~ 5000 8600
+NoConn ~ 5000 8700
+$Comp
+L Connector:Screw_Terminal_01x02 J9
+U 1 1 5C118EB3
+P 13200 850
+F 0 "J9" H 13280 842 50  0000 L CNN
+F 1 "Screw_Terminal_01x02" H 13280 751 50  0000 L CNN
+F 2 "TerminalBlock:TerminalBlock_bornier-2_P5.08mm" H 13200 850 50  0001 C CNN
+F 3 "~" H 13200 850 50  0001 C CNN
+	1    13200 850
+	1    0    0    -1
+$EndComp
+Text GLabel 13000 850  0    50   Input ~ 0
+CANH
+Text GLabel 13000 950  0    50   Input ~ 0
+CANL
 $EndSCHEMATC

Commit message: final draft
Parts:
- removed C2: 10u, Capacitor_SMD:C_0603_1608Metric, symbol Device:C
- removed R3: 1M, Resistor_SMD:R_0603_1608Metric, symbol Device:R
- added J10: ICSP, Connector_PinHeader_2.54mm:PinHeader_2x03_P2.54mm_Vertical, symbol Connector_Generic:Conn_02x03_Odd_Even
- C1: value 10u -> 22u; footprint Capacitor_SMD:C_0603_1608Metric -> Capacitor_SMD:C_0805_2012Metric
- C5, C6, C7: footprint Capacitor_SMD:CP_Elec_4x5.4 -> Capacitor_SMD:C_0805_2012Metric
- J7: value Conn_01x05_Male -> PROGRAM
Connections:
- net GNDREF: now also J10.6 (Pin_6); no longer U1.5 (PG)
- net Rst: now also J10.5 (Pin_5)
- net S0: now also J10.1 (Pin_1)
- net SCK: now also U8.20 (PB1), J10.3 (Pin_3); no longer U8.55 (PC2)
- net SI: now also J10.4 (Pin_4)
- net SS: no longer U9.18 (~CS)
- net MCP_SS: now reaches U8.76 (PA2)
- net MCP_SS: now also U9.18 (~CS)
- net VPP: now reaches D2.1 (A), J7.1 (Pin_1)
- net VPP: now also J10.2 (Pin_2)
- no-connect marks 67 -> 68
Other:
- moved on the sheet: C1, J7, J8, J9
