File: Motor test module/_saved_Motor test module.sch (KiCad schematic (older format))
At the start: 55 parts, among them J1 Conn_02x04_Counter_Clockwise, J2 Conn_02x04_Counter_Clockwise, J3 Conn_02x04_Counter_Clockwise, J4 Conn_02x04_Counter_Clockwise, J5 Conn_02x04_Counter_Clockwise, J6 Conn_02x04_Counter_Clockwise, J7 Conn_01x05_Male, J8 Screw_Terminal_01x02, SW1 SW_Push, U1 TPS63060, U10 ATA6560,1, U2 AP1017AEN, U3 AP1017AEN, U4 AP1017AEN, U5 AP1017AEN, U6 AP1017AEN, U7 AP1017AEN, U8 ATmega2560-16AU, U9 MCP2515-EST, Y1 16MHz, Y2 16MHz

Commit message: Third draft of layout
Connections:
- no-connect marks 65 -> 69
Changed lines of the file:
@@
 	7250 850  7250 2100
 $Comp
-L power:+5V #PWR?
+L power:+5V #PWR0156
 U 1 1 5C019AEE
 P 4300 3400
-F 0 "#PWR?" H 4300 3250 50  0001 C CNN
+F 0 "#PWR0156" H 4300 3250 50  0001 C CNN
 F 1 "+5V" H 4315 3573 50  0000 C CNN
 F 2 "" H 4300 3400 50  0001 C CNN
@@
 Connection ~ 4300 3400
 $Comp
-L power:+5V #PWR?
+L power:+5V #PWR0191
 U 1 1 5C032B9A
 P 7100 1400
-F 0 "#PWR?" H 7100 1250 50  0001 C CNN
+F 0 "#PWR0191" H 7100 1250 50  0001 C CNN
 F 1 "+5V" H 7115 1573 50  0000 C CNN
 F 2 "" H 7100 1400 50  0001 C CNN
@@
 	1    0    0    -1
 $EndComp
+NoConn ~ 5000 4400
+NoConn ~ 5000 4300
+NoConn ~ 5000 4200
+NoConn ~ 5000 4100
 $EndSCHEMATC
