File: Motor test module/Motor test module.kicad_pcb (KiCad board)
At the start: 2 copper layers, 16 parts, among them U1 TPS63060, U8 ATmega2560-16AU, U9 MCP2515-EST

Commit message: switching computers - wip
Parts:
- removed C12, C13: 15p, Capacitor_SMD:C_0603_1608Metric
- removed C8, C9: 20p, Capacitor_SMD:C_0603_1608Metric
- added C16: 100n, Capacitor_SMD:C_0603_1608Metric, F.Cu at (212.2, 94.4)
- added C17: 100n, Capacitor_SMD:C_0603_1608Metric, F.Cu at (194.1, 96.2)
- added C18: 100n, Capacitor_SMD:C_0603_1608Metric, F.Cu at (216.0, 91.4)
- added C19: 100n, Capacitor_SMD:C_0603_1608Metric, F.Cu at (213.0, 92.9)
- added C2: 10u, Capacitor_SMD:C_0603_1608Metric, F.Cu at (203.2, 93.9)
- added C20: 100n, Capacitor_SMD:C_0603_1608Metric, F.Cu at (219.9, 86.9)
- added C21: 100n, Capacitor_SMD:C_0603_1608Metric, F.Cu at (209.2, 95.4)
- added C22: 100n, Capacitor_SMD:C_0603_1608Metric, F.Cu at (191.1, 96.2)
- added C23: 100n, Capacitor_SMD:C_0603_1608Metric, F.Cu at (197.1, 96.2)
- added C24: 100n, Capacitor_SMD:C_0603_1608Metric, F.Cu at (200.1, 96.2)
- added C25: 100n, Capacitor_SMD:C_0603_1608Metric, F.Cu at (212.2, 95.9)
- added C26: 100n, Capacitor_SMD:C_0603_1608Metric, F.Cu at (206.2, 93.9)
- added C27: 100n, Capacitor_SMD:C_0603_1608Metric, F.Cu at (203.2, 95.4)
- added C28: 100n, Capacitor_SMD:C_0603_1608Metric, F.Cu at (206.2, 95.4)
- added C29: 100n, Capacitor_SMD:C_0603_1608Metric, F.Cu at (216.9, 86.9)
- added C30: 100n, Capacitor_SMD:C_0603_1608Metric, F.Cu at (209.2, 93.9)
- added J1: Conn_02x04_Counter_Clockwise, Connector_PinHeader_2.54mm:PinHeader_2x04_P2.54mm_Vertical, F.Cu at (210.0, 76.8)
- added J2: Conn_02x04_Counter_Clockwise, Connector_PinHeader_2.54mm:PinHeader_2x04_P2.54mm_Vertical, F.Cu at (203.8, 76.8)
- added J3: Conn_02x04_Counter_Clockwise, Connector_PinHeader_2.54mm:PinHeader_2x04_P2.54mm_Vertical, F.Cu at (197.6, 76.8)
- added J4: Conn_02x04_Counter_Clockwise, Connector_PinHeader_2.54mm:PinHeader_2x04_P2.54mm_Vertical, F.Cu at (216.2, 76.8)
- added J5: Conn_02x04_Counter_Clockwise, Connector_PinHeader_2.54mm:PinHeader_2x04_P2.54mm_Vertical, F.Cu at (191.4, 76.8)
- added J6: Conn_02x04_Counter_Clockwise, Connector_PinHeader_2.54mm:PinHeader_2x04_P2.54mm_Vertical, F.Cu at (222.4, 76.8)
- added L1: XFL4020-102, Inductor_SMD:L_0603_1608Metric, F.Cu at (213.0, 91.4)
- added R1: 1M, Resistor_SMD:R_0603_1608Metric, F.Cu at (222.9, 86.9)
- added R10: 10k, Resistor_SMD:R_0603_1608Metric, F.Cu at (216.9, 88.4)
- added R2: 100k, Resistor_SMD:R_0603_1608Metric, F.Cu at (219.9, 88.4)
- added R3: 1M, Resistor_SMD:R_0603_1608Metric, F.Cu at (222.9, 88.4)
- added R5: 100k, Resistor_SMD:R_0603_1608Metric, F.Cu at (219.0, 90.0)
- added R7: 10k, Resistor_SMD:R_0603_1608Metric, F.Cu at (216.0, 92.9)
- added R8: 10k, Resistor_SMD:R_0603_1608Metric, F.Cu at (215.2, 94.4)
- added U10: ATA6560,1, Package_SO:SO-8_5.3x6.2mm_P1.27mm, F.Cu at (194.5, 89.6)
- added U2: AP1017AEN, Package_SON:SON-8-1EP_3x2mm_P0.5mm_EP1.4x1.6mm, F.Cu at (191.4, 94.2)
- added U3: AP1017AEN, Package_SON:SON-8-1EP_3x2mm_P0.5mm_EP1.4x1.6mm, F.Cu at (195.1, 94.2)
- added U4: AP1017AEN, Package_SON:SON-8-1EP_3x2mm_P0.5mm_EP1.4x1.6mm, F.Cu at (198.7, 94.2)
- added U5: AP1017AEN, Package_SON:SON-8-1EP_3x2mm_P0.5mm_EP1.4x1.6mm, F.Cu at (202.4, 91.9)
- added U6: AP1017AEN, Package_SON:SON-8-1EP_3x2mm_P0.5mm_EP1.4x1.6mm, F.Cu at (206.0, 91.9)
- added U7: AP1017AEN, Package_SON:SON-8-1EP_3x2mm_P0.5mm_EP1.4x1.6mm, F.Cu at (209.7, 91.9)
- added Y1: 16MHz, Crystal:Resonator_SMD_muRata_CSTxExxV-3Pin_3.0x1.1mm, F.Cu at (203.4, 88.4)
- added Y2: 16MHz, Crystal:Resonator_SMD_muRata_CSTxExxV-3Pin_3.0x1.1mm, F.Cu at (211.4, 88.4)
- C1: footprint Diode_THT:D_DO-41_SOD81_P7.62mm_Horizontal -> Capacitor_SMD:C_0603_1608Metric
- moved C11 7.14 mm to (111.4, 104.3), turned to 135 degrees
Routing:
- net GNDREF: track 0.00 -> 0.74 mm
- added copper zone on B.Cu, net (none)
- added copper zone on F.Cu, net GNDREF
Other:
- board outline added: 103.1 x 103.1 mm

Commit message: beginning layout
Parts:
- removed C11: 100n, Capacitor_SMD:C_0603_1608Metric
- U2, U3, U4, U5, U6, U7: footprint Package_SON:SON-8-1EP_3x2mm_P0.5mm_EP1.4x1.6mm -> Package_SON:WSON-8-1EP_2x2mm_P0.5mm_EP0.9x1.6mm
- moved U6 109.9 mm to (96.1, 93.1)
- moved U3 98.9 mm to (96.4, 87.8)
- moved U4 91.6 mm to (107.7, 103.9)
- moved U5 90.9 mm to (112.3, 103.8)
- moved C21 77.8 mm to (139.3, 61.2)
- moved C24 77.8 mm to (130.3, 61.9)
- moved C29 77.8 mm to (147.0, 52.6)
- moved C30 77.8 mm to (139.3, 59.6)
- moved R10 77.8 mm to (147.0, 54.2)
- moved C17 77.8 mm to (124.3, 61.9)
- moved J2 77.8 mm to (134.0, 42.5)
- moved C16 77.8 mm to (142.3, 60.1)
- moved C18 77.8 mm to (146.2, 57.1)
- moved C19 77.8 mm to (143.2, 58.6)
- moved C2 77.8 mm to (133.3, 59.6)
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Routing:
- net +5V: track 0.00 -> 27.8 mm, vias 0 -> 3
- net M2-C: track 0.00 -> 16.1 mm
- net M2+C: track 0.00 -> 14.8 mm
- net +3V3: track 0.00 -> 14.2 mm, vias 0 -> 2
- net M2A-C: track 0.00 -> 11.5 mm
- net M1B-C: track 0.00 -> 9.07 mm
- net M1+C: track 0.00 -> 9.03 mm, vias 0 -> 2
- net M2A+C: track 0.00 -> 8.58 mm
- net M1-C: track 0.00 -> 8.39 mm, vias 0 -> 2
- net M1B+C: track 0.00 -> 6.75 mm

Commit message: First draft of layout
Parts:
- added C11: 100n, Capacitor_SMD:C_0603_1608Metric, F.Cu at (176.0, 66.8)
- moved C25 83.8 mm to (172.5, 139.8)
- moved C21 82.4 mm to (172.7, 136.5)
- moved C30 72.0 mm to (184.6, 115.6)
- moved C19 69.1 mm to (180.3, 116.8)
- moved C17 68.2 mm to (176.8, 105.4), turned to 180 degrees
- moved U6 67.3 mm to (163.1, 86.1)
- moved U8 67.3 mm to (178.6, 81.2)
- moved U3 67.3 mm to (163.3, 80.7)
- moved U4 67.3 mm to (174.6, 96.9)
- moved U5 67.3 mm to (179.2, 96.7)
- moved C18 67.0 mm to (184.9, 111.8)
- moved Y1 66.2 mm to (185.8, 94.7)
- moved C29 65.8 mm to (175.2, 112.1)
- moved C27 65.5 mm to (180.9, 106.2)
- moved C26 64.8 mm to (179.0, 108.3), turned to 180 degrees
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Connections:
- C30 pad 1: +3V3 -> +5V
- U8 pad 10: +3V3 -> +5V
- U8 pad 100: +3V3 -> +5V
- U8 pad 31: +3V3 -> +5V
- U8 pad 61: +3V3 -> +5V
- U8 pad 80: +3V3 -> +5V
Routing:
- net GNDREF: track 0.74 -> 476.8 mm, vias 0 -> 45
- net +5V: track 27.8 -> 338.9 mm, vias 3 -> 20
- net +12V: track 0.00 -> 169.5 mm, vias 0 -> 5
- net +3V3: track 14.2 -> 117.7 mm, vias 2 -> 16
- net M1+: track 0.00 -> 102.9 mm, vias 0 -> 4
- net M1-: track 0.00 -> 101.9 mm, vias 0 -> 4
- net E2: track 0.00 -> 82.4 mm, vias 0 -> 6
- net E1: track 0.00 -> 76.7 mm, vias 0 -> 2
- net M2+: track 0.00 -> 64.3 mm, vias 0 -> 1
- net TX0: track 0.00 -> 63.1 mm, vias 0 -> 2
- net TX1: track 0.00 -> 58.5 mm, vias 0 -> 2
- net SI: track 0.00 -> 55.1 mm, vias 0 -> 2
- net M2-: track 0.00 -> 54.0 mm, vias 0 -> 4
- net M1A+: track 0.00 -> 52.7 mm, vias 0 -> 2
- net Servo1: track 0.00 -> 48.8 mm, vias 0 -> 2
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- removed copper zone on B.Cu, net (none)
- removed copper zone on F.Cu, net GNDREF
Other:
- outline, holes or cut-outs redrawn

Commit message: Second draft of layout
Parts:
- added J7: Conn_01x05_MountingPin, Connector_Molex:Molex_Pico-Clasp_501331-0507_1x05-1MP_P1.00mm_Vertical, F.Cu at (133.6, 108.0)
- added J8: Screw_Terminal_01x02, TerminalBlock:TerminalBlock_bornier-2_P5.08mm, F.Cu at (77.5, 143.6)
- added R4: 10k, Resistor_SMD:R_0603_1608Metric, F.Cu at (108.6, 128.0)
- added SW1: SW_Push, Button_Switch_THT:SW_PUSH_6mm, F.Cu at (116.6, 129.5)
- moved C24 136.5 mm to (53.3, 134.1), turned to 90 degrees
- moved U5 125.2 mm to (55.4, 115.6)
- moved C18 117.2 mm to (68.2, 122.2)
- moved C7 116.7 mm to (56.4, 132.6), turned to 90 degrees
- moved C21 115.8 mm to (56.9, 137.5), turned to 270 degrees
- moved C30 114.6 mm to (70.1, 118.7), turned to 270 degrees
- moved C16 111.3 mm to (73.2, 116.7)
- moved U2 110.8 mm to (55.4, 100.3)
- moved C17 109.7 mm to (68.2, 120.8), turned to 0 degrees
- moved U3 108.9 mm to (55.4, 95.4)
- moved J2 108.3 mm to (47.9, 111.8)
- moved C26 107.9 mm to (71.9, 120.8)
- moved C27 107.7 mm to (73.9, 118.7), turned to 90 degrees
- moved U4 107.5 mm to (68.8, 115.6)
- moved C19 107.5 mm to (72.9, 115.1)
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Connections:
- C30 pad 1: +5V -> +3V3
- U8 pad 10: +5V -> +3V3
- U8 pad 100: +5V -> +3V3
- U8 pad 31: +5V -> +3V3
- U8 pad 61: +5V -> +3V3
- U8 pad 73: Net-(U8-Pad73) -> Vpp
- U8 pad 74: Net-(U8-Pad74) -> Rst
- U8 pad 75: Net-(U8-Pad75) -> Rx
- U8 pad 76: Net-(U8-Pad76) -> Tx
- U8 pad 80: +5V -> +3V3
- U8 pad 94: Net-(U8-Pad94) -> CANL
- U8 pad 95: Net-(U8-Pad95) -> CANH
Routing:
- net GNDREF: track 476.8 -> 0.00 mm, vias 45 -> 1
- net +12V: track 169.5 -> 42.4 mm, vias 5 -> 3
- net M1+: track 102.9 -> 10.3 mm, vias 4 -> 2
- net M1-: track 101.9 -> 15.6 mm, vias 4 -> 2
- net +5V: track 338.9 -> 257.7 mm, vias 20 -> 18
- net E1: track 76.7 -> 156.5 mm, vias 2 -> 0
- net M1-C: track 8.39 -> 80.8 mm
- net M1+C: track 8.71 -> 78.7 mm, vias 2 -> 0
- net +3V3: track 117.7 -> 187.0 mm, vias 16 -> 18
- net M1B+C: track 7.89 -> 66.5 mm
- net E2: track 82.4 -> 140.7 mm, vias 6 -> 0
- net M1B-C: track 10.9 -> 67.9 mm
- net M2+: track 64.3 -> 9.56 mm, vias 1 -> 0
- net M1A-C: track 11.6 -> 63.5 mm
- net M1A+C: track 10.4 -> 61.0 mm
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Other:
- outline, holes or cut-outs redrawn

Commit message: Third draft of layout
Parts:
- J7: value Conn_01x05_MountingPin -> Conn_01x05_Male; footprint Connector_Molex:Molex_Pico-Clasp_501331-0507_1x05-1MP_P1.00mm_Vertical -> Connector_PinHeader_2.54mm:PinHeader_1x05_P2.54mm_Vertical
- moved J8 46.4 mm to (118.2, 121.4)
- moved C1 42.7 mm to (116.9, 104.6)
- moved C19 42.7 mm to (113.7, 102.2)
- moved C23 42.7 mm to (112.5, 81.7)
- moved C28 42.7 mm to (119.8, 104.6)
- moved C4 42.7 mm to (150.3, 93.5)
- moved C5 42.7 mm to (138.4, 118.2)
- moved C6 42.7 mm to (133.6, 116.0)
- moved D1 42.7 mm to (149.1, 67.3)
- moved R10 42.7 mm to (150.3, 78.7)
- moved R3 42.7 mm to (114.8, 81.6)
- moved R5 42.7 mm to (150.1, 64.9)
- moved SW1 42.7 mm to (157.4, 116.7)
- moved U8 42.7 mm to (158.9, 101.5)
- moved C18 42.7 mm to (109.0, 109.3)
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Connections:
- J7 pad 1: GNDREF -> Net-(J7-Pad1)
- J7 pad 2: Tx -> Rst
- J7 pad 4: Rst -> Tx
- J7 pad 5: Vpp -> GNDREF
- R4 pad 2: Net-(R4-Pad2) -> Rst
- SW1 pad 2: Net-(R4-Pad2) -> Rst
- U8 pad 10: +3V3 -> +5V
- U8 pad 100: +3V3 -> +5V
- U8 pad 2: Net-(U8-Pad2) -> Rx
- U8 pad 3: Net-(U8-Pad3) -> Tx
- U8 pad 30: Net-(R4-Pad2) -> Rst
- U8 pad 31: +3V3 -> +5V
- U8 pad 61: +3V3 -> +5V
- U8 pad 73: Vpp -> Net-(U8-Pad73)
- U8 pad 74: Rst -> Net-(U8-Pad74)
- U8 pad 75: Rx -> Net-(U8-Pad75)
- U8 pad 76: Tx -> Net-(U8-Pad76)
- U8 pad 80: +3V3 -> +5V
Routing:
- net +5V: track 257.7 -> 304.2 mm, vias 18 -> 21
- net GNDREF: track 0.00 -> 35.4 mm, vias 1 -> 87
- net +12V: track 42.4 -> 72.4 mm, vias 3 -> 8
- net Rst: track 6.63 -> 32.7 mm, vias 2 -> 1
- net +3V3: track 187.0 -> 162.7 mm
- net Net-(R4-Pad2): track 18.4 -> 0.00 mm, vias 1 -> 0
- net Rx: track 6.66 -> 23.8 mm, vias 2 -> 3
- net Tx: track 12.3 -> 19.4 mm, vias 2 -> 3
- net Vpp: track 6.83 -> 0.00 mm, vias 2 -> 0
- net Net-(J7-PadMP): track 6.60 -> 0.00 mm
- net M1-C: track 80.8 -> 83.9 mm
- net INT: track 28.2 -> 30.0 mm
- net M2A+C: track 50.5 -> 52.3 mm
- net Net-(C4-Pad2): track 36.5 -> 38.2 mm
- net TX2: track 57.2 -> 58.1 mm
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- added copper zone on B.Cu, net GNDREF
- added copper zone on F.Cu, net GNDREF

Commit message: Fourth draft of layout
Parts:
- added D2: D_x2_KCom_AAK, Package_TO_SOT_SMD:SOT-23, F.Cu at (138.4, 106.6)
- added J9: Screw_Terminal_01x02, TerminalBlock:TerminalBlock_bornier-2_P5.08mm, F.Cu at (166.4, 75.7)
- moved C7 73.3 mm to (143.7, 63.1)
- moved C6 53.1 mm to (85.8, 92.8), turned to 270 degrees
- moved C21 48.5 mm to (145.5, 116.4), turned to 180 degrees
- moved C25 39.6 mm to (132.0, 79.9)
- moved C11 38.7 mm to (117.7, 90.6), turned to 0 degrees
- moved C5 36.1 mm to (124.0, 85.2)
- moved C26 31.8 mm to (98.6, 79.5), turned to 90 degrees
- moved C22 30.8 mm to (155.3, 89.9), turned to 270 degrees
- moved C29 30.6 mm to (86.3, 105.3), turned to 270 degrees
- moved C17 29.5 mm to (112.3, 78.6)
- moved C16 25.8 mm to (108.6, 78.7)
- moved C30 24.8 mm to (135.7, 106.4), turned to 90 degrees
- moved C2 20.3 mm to (112.7, 121.4)
- moved C27 17.9 mm to (113.0, 88.1), turned to 270 degrees
- moved C20 13.3 mm to (85.9, 121.9)
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Connections:
- C30 pad 1: +3V3 -> VCC
- U8 pad 10: +5V -> VCC
- U8 pad 100: +5V -> VCC
- U8 pad 31: +5V -> VCC
- U8 pad 61: +5V -> VCC
- U8 pad 80: +5V -> VCC
- U8 pad 94: CANL -> Net-(U8-Pad94)
- U8 pad 95: CANH -> Net-(U8-Pad95)
Routing:
- net VCC: track 0.00 -> 59.3 mm, vias 0 -> 5
- net +3V3: track 162.7 -> 122.4 mm, vias 18 -> 14
- net +5V: track 304.2 -> 281.6 mm, vias 21 -> 23
- net +12V: track 72.4 -> 69.1 mm, vias 8 -> 7
- net GNDREF: track 35.4 -> 38.4 mm, vias 87 -> 33
- net Servo2: track 58.4 -> 60.9 mm, vias 4 -> 2
- net Net-(D2-Pad1): track 0.00 -> 2.38 mm
- net CANL: track 16.4 -> 17.7 mm, vias 0 -> 2
- net M2A-C: track 59.2 -> 60.3 mm
- net M2-: track 11.8 -> 10.6 mm
- net Servo1: track 73.8 -> 72.9 mm
- net TX2: track 58.1 -> 58.9 mm
- net M2+: track 9.56 -> 10.1 mm
- net CANH: track 19.8 -> 19.4 mm, vias 0 -> 2

Commit message: Fifth draft of layout
Parts:
- moved C22 9.94 mm to (164.2, 94.4)
- moved C5 9.94 mm to (132.8, 89.6)
- moved J7 9.94 mm to (148.0, 114.2)
- moved R1 9.94 mm to (159.3, 95.1)
- moved Y2 9.94 mm to (147.4, 80.5)
- moved C3 9.94 mm to (136.9, 115.5)
- moved J9 9.94 mm to (175.3, 80.1)
- moved R2 9.94 mm to (159.3, 96.5)
- moved R7 9.94 mm to (160.3, 74.4)
- moved R8 9.94 mm to (159.3, 93.7)
- moved U10 9.94 mm to (154.7, 86.5)
- moved U9 9.94 mm to (154.7, 76.8)
- moved Y1 9.94 mm to (170.9, 119.0)
- moved C16 9.94 mm to (117.5, 83.1)
- moved C18 9.94 mm to (117.0, 102.8)
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Routing:
- net GNDREF: track 38.4 -> 43.0 mm, vias 33 -> 336
- net +5V: track 281.6 -> 284.7 mm
- net M1A-C: track 64.2 -> 63.4 mm

Commit message: Sixth draft of layout
Parts:
- D1: footprint Diode_THT:D_DO-41_SOD81_P2.54mm_Vertical_AnodeUp -> Diode_SMD:D_0603_1608Metric
- moved C20 88.6 mm to (159.1, 65.4), turned to 0 degrees
- moved C7 81.5 mm to (92.6, 122.7)
- moved J8 70.7 mm to (168.8, 68.7), turned to 270 degrees
- moved R1 28.8 mm to (136.1, 112.2), turned to 0 degrees
- moved R2 27.6 mm to (137.8, 113.9)
- moved C4 27.6 mm to (137.7, 115.3)
- moved C17 22.4 mm to (104.9, 98.6)
- moved C18 11.5 mm to (105.5, 102.6), turned to 180 degrees
- moved Y1 5.27 mm to (165.9, 117.6)
- moved C29 4.21 mm to (94.7, 113.9)
- moved C16 3.61 mm to (121.0, 83.8)
- moved C14 3.57 mm to (164.8, 77.6)
- moved C3 3.36 mm to (134.6, 118.0), turned to 0 degrees
- moved SW1 2.60 mm to (164.6, 123.2)
- moved Y2 1.70 mm to (148.5, 79.2), turned to 270 degrees
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Routing:
- net +12V: track 69.1 -> 201.9 mm, vias 7 -> 10
- net Net-(C4-Pad2): track 37.8 -> 6.47 mm, vias 4 -> 0
- net M1-C: track 83.9 -> 95.2 mm
- net M1+C: track 78.7 -> 89.8 mm
- net GNDREF: track 43.0 -> 31.9 mm, vias 336 -> 457
- net M2+C: track 60.1 -> 69.8 mm
- net M2-C: track 60.7 -> 68.6 mm
- net +5V: track 284.7 -> 279.1 mm, vias 23 -> 21
- net Net-(U8-Pad34): track 9.72 -> 4.57 mm, vias 2 -> 0
- net Net-(U8-Pad33): track 8.64 -> 4.28 mm, vias 2 -> 0
- net Net-(C14-Pad1): track 6.98 -> 11.1 mm
- net +3V3: track 122.4 -> 126.1 mm
- net Net-(U9-Pad8): track 6.78 -> 3.42 mm
- net Rst: track 32.7 -> 29.8 mm, vias 1 -> 2
- net M2B-C: track 61.0 -> 62.6 mm
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Other:
- board text added: "+5V|SERVO1 GND|X +5V|E1 GND|X"
- board text added: "+5V|SERVO2 GND|X +5V|E2 GND|X"
- board text added: "A+ | A- B+ | B- 5V | E1 GND|"
- board text added: "M+|M- X|X +12V|E GND|X"
