File: Motor test module/Motor test module.kicad_pcb (KiCad board)
At the start: 2 copper layers, 103.1 x 103.1 mm, 57 parts, among them J1 Conn_02x04_Counter_Clockwise, J10 ICSP, J2 Conn_02x04_Counter_Clockwise, J3 Conn_02x04_Counter_Clockwise, J4 Conn_02x04_Counter_Clockwise, J5 Conn_02x04_Counter_Clockwise, J6 Conn_02x04_Counter_Clockwise, J7 PROGRAM, J8 Screw_Terminal_01x02, J9 Screw_Terminal_01x02, SW1 SW_Push, U1 TPS63060, U10 ATA6560,1, U2 AP1017AEN, U3 AP1017AEN, U4 AP1017AEN, U5 AP1017AEN, U6 AP1017AEN, U7 AP1017AEN, U8 ATmega2560-16AU, U9 MCP2515-EST, Y1 16MHz, Y2 16MHz

Commit message: fixed stuff
Parts:
- moved G*** 2.84 mm to (133.5, 103.6)
- moved C7 2.54 mm to (152.8, 65.9)
- moved D1 2.54 mm to (158.1, 69.2)
- moved R5 2.54 mm to (159.1, 66.8)
Routing:
- net +5V: track 313.8 -> 309.1 mm, vias 23 -> 21
- net Net-(C14-Pad1): track 6.98 -> 9.46 mm
